File: Kicad/mini/pic8bit.kicad_pcb (KiCad board)
At the start: 2 copper layers, 80 x 100 mm, 85 parts, among them IC201 TLV1117-33, IC202 MICROCHIP-PIC16F1778-ISP, IC301 ONSEMI-CAT4002A-SOT-23, IC302 MICROCHIP-MCP2221A-ISL, K101 PE-450-4X6X-BLACK, K201 *Power & UART, K202 MCU 1, K203 MCU 1, K204 ICSP, K205 MCU 2, K206 MCU 2, K301 HARWIN-254-F-1X08-VERTICAL, K302 HARWIN-254-F-1X06-VERTICAL, P301 PIHER-PT10MV-10K, P302 PIHER-PT10MV-10K

Commit message: Update
Parts:
- added TP203: KEYSTONE-2000-3, tronixio:KEYSTONE-2000-3, F.Cu at (70.5, 90.5)
- moved S201 1.11 mm to (70.5, 98.1)
- moved TP201 0.50 mm to (81.5, 143.5)
- moved TP202 0.50 mm to (132.5, 143.5)
Routing:
- net Net-(IC302-Pad4): track 12.6 -> 11.9 mm
Other:
- board text added: "S"

Commit message: Update Mini
Parts:
- JP301: value EN BCKL -> BCKL
- LED301, LED302: footprint tronixio:FUSE-1206 -> tronixio:LED-1206
- R307: value 2K4 -> 10K
Changed lines of the file:
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@@
     )
   )
-  (footprint "tronixio:FUSE-1206" (layer "F.Cu")
+  (footprint "tronixio:LED-1206" (layer "F.Cu")
     (at 78.5 50.5 90)
     (property "Mouser" "604-APT2012LSECKJ4RV")
@@
     (fp_line (start -0.6 -0.9) (end 0.6 -0.9) (layer "F.SilkS") (width 0.15))
     (fp_line (start -0.6 0.9) (end 0.6 0.9) (layer "F.SilkS") (width 0.15))
-    (fp_rect (start -2.3 1) (end 2.3 -1) (layer "F.CrtYd") (width 0.05) (fill none))
-    (fp_rect (start -1.1 0.8) (end 1.1 -0.8) (layer "F.Fab") (width 0.1) (fill none))
-    (fp_poly (pts
-        (xy 1.1 -0.8)
-        (xy 1.4 -0.8)
-        (xy 1.4 -0.3)
-        (xy 1.1 0)
-        (xy 1.4 0.3)
-        (xy 1.4 0.8)
-        (xy 1.1 0.8)
-      ) (layer "F.Fab") (width 0.1) (fill solid))
     (fp_poly (pts
-        (xy -1.1 0.8)
-        (xy -1.4 0.8)
-        (xy -1.4 0.3)
-        (xy -1.1 0)
-        (xy -1.4 -0.3)
-        (xy -1.4 -0.8)
-        (xy -1.1 -0.8)
-      ) (layer "F.Fab") (width 0.1) (fill solid))
+        (xy 0.5 0.6)
+        (xy 0.3 0.6)
+        (xy 0.3 0.1)
+        (xy -0.5 0.1)
+        (xy -0.5 -0.1)
+        (xy 0.3 -0.1)
+        (xy 0.3 -0.6)
+        (xy 0.5 -0.6)
+      ) (layer "F.SilkS") (width 0.1) (fill solid))
+    (fp_rect (start -2.3 1) (end 2.3 -1) (layer "F.CrtYd") (width 0.05) (fill none))
+    (fp_rect (start -1.5 0.8) (end -1.2 -0.8) (layer "F.Fab") (width 0.1) (fill solid))
+    (fp_rect (start -1.2 0.8) (end 1.2 -0.8) (layer "F.Fab") (width 0.1) (fill none))
     (pad "1" smd roundrect (at -1.5 0 90) (size 1.3 1.75) (layers "F.Cu" "F.Paste" "F.Mask") (roundrect_rratio 0.15)
       (net 18 "Net-(IC302-Pad2)") (pinfunction "K") (pintype "passive") (zone_connect 2))
     (pad "2" smd roundrect (at 1.5 0 90) (size 1.3 1.75) (layers "F.Cu" "F.Paste" "F.Mask") (roundrect_rratio 0.15)
       (net 21 "Net-(LED302-Pad2)") (pinfunction "A") (pintype "passive") (zone_connect 2))
-    (model "${KICAD6_USER_3DMODEL_DIR}/SMD/RESISTOR-1206.wrl"
+    (model "${KICAD6_USER_3DMODEL_DIR}/SMD/LED-1206.wrl"
       (offset (xyz 0 0 0))
       (scale (xyz 1 1 1))
@@
     )
   )
-  (footprint "tronixio:FUSE-1206" (layer "F.Cu")
+  (footprint "tronixio:LED-1206" (layer "F.Cu")
     (at 90.5 50.5 90)
     (property "Mouser" "604-APT2012LSECKJ4RV")
@@
       (effects (font (size 1 1) (thickness 0.15)))
     )
-    (fp_line (start -0.6 0.9) (end 0.6 0.9) (layer "F.SilkS") (width 0.15))
     (fp_line (start -0.6 -0.9) (end 0.6 -0.9) (layer "F.SilkS") (width 0.15))
-    (fp_rect (start -2.3 1) (end 2.3 -1) (layer "F.CrtYd") (width 0.05) (fill none))
-    (fp_rect (start -1.1 0.8) (end 1.1 -0.8) (layer "F.Fab") (width 0.1) (fill none))
-    (fp_poly (pts
-        (xy -1.1 0.8)
-        (xy -1.4 0.8)
-        (xy -1.4 0.3)
-        (xy -1.1 0)
-        (xy -1.4 -0.3)
-        (xy -1.4 -0.8)
-        (xy -1.1 -0.8)
-      ) (layer "F.Fab") (width 0.1) (fill solid))
+    (fp_line (start -0.6 0.9) (end 0.6 0.9) (layer "F.SilkS") (width 0.15))
     (fp_poly (pts
-        (xy 1.1 -0.8)
-        (xy 1.4 -0.8)
-        (xy 1.4 -0.3)
-        (xy 1.1 0)
-        (xy 1.4 0.3)
-        (xy 1.4 0.8)
-        (xy 1.1 0.8)
-      ) (layer "F.Fab") (width 0.1) (fill solid))
+        (xy 0.5 0.6)
+        (xy 0.3 0.6)
+        (xy 0.3 0.1)
+        (xy -0.5 0.1)
+        (xy -0.5 -0.1)
+        (xy 0.3 -0.1)
+        (xy 0.3 -0.6)
+        (xy 0.5 -0.6)
+      ) (layer "F.SilkS") (width 0.1) (fill solid))
+    (fp_rect (start -2.3 1) (end 2.3 -1) (layer "F.CrtYd") (width 0.05) (fill none))
+    (fp_rect (start -1.2 0.8) (end 1.2 -0.8) (layer "F.Fab") (width 0.1) (fill none))
+    (fp_rect (start -1.5 0.8) (end -1.2 -0.8) (layer "F.Fab") (width 0.1) (fill solid))
     (pad "1" smd roundrect (at -1.5 0 90) (size 1.3 1.75) (layers "F.Cu" "F.Paste" "F.Mask") (roundrect_rratio 0.15)
       (net 20 "Net-(IC302-Pad3)") (pinfunction "K") (pintype "passive") (zone_connect 2))
     (pad "2" smd roundrect (at 1.5 0 90) (size 1.3 1.75) (layers "F.Cu" "F.Paste" "F.Mask") (roundrect_rratio 0.15)
       (net 19 "Net-(LED301-Pad2)") (pinfunction "A") (pintype "passive") (zone_connect 2))
-    (model "${KICAD6_USER_3DMODEL_DIR}/SMD/RESISTOR-1206.wrl"
+    (model "${KICAD6_USER_3DMODEL_DIR}/SMD/LED-1206.wrl"
       (offset (xyz 0 0 0))
       (scale (xyz 1 1 1))
@@
     (fp_line (start -3.5 5.3) (end -3.5 2.8) (layer "F.Fab") (width 0.1))
     (fp_arc (start -4 3.3) (mid -4.903738 -1.844892) (end -0.9 -5.2) (layer "F.Fab") (width 0.1))
-    (fp_arc (start 1.5 4.1) (mid 0.923087 4.342349) (end 0.3 4.4) (layer "F.Fab") (width 0.1))
+    (fp_arc (start 1.5 4.1) (mid 0.923087 4.34235) (end 0.3 4.4) (layer "F.Fab") (width 0.1))
     (fp_arc (start -0.3 4.4) (mid -0.923087 4.342349) (end -1.5 4.1) (layer "F.Fab") (width 0.1))
     (fp_arc (start 0.9 -5.2) (mid 4.903738 -1.844893) (end 4 3.3) (layer "F.Fab") (width 0.1))
@@
     (fp_line (start 4 5.3) (end 4 3.3) (layer "F.Fab") (width 0.1))
     (fp_line (start -0.3 2.5) (end -0.3 4.4) (layer "F.Fab") (width 0.1))
-    (fp_arc (start 1.5 4.1) (mid 0.923087 4.342349) (end 0.3 4.4) (layer "F.Fab") (width 0.1))
+    (fp_arc (start 1.5 4.1) (mid 0.923087 4.34235) (end 0.3 4.4) (layer "F.Fab") (width 0.1))
     (fp_arc (start 0.9 -5.2) (mid 4.903738 -1.844893) (end 4 3.3) (layer "F.Fab") (width 0.1))
     (fp_arc (start -4 3.3) (mid -4.903738 -1.844892) (end -0.9 -5.2) (layer "F.Fab") (width 0.1))
@@
       (effects (font (size 1 1) (thickness 0.15)))
     )
-    (fp_text value "EN BCKL" (at 0 5.08) (layer "F.Fab")
+    (fp_text value "BCKL" (at 0 5.08) (layer "F.Fab")
       (effects (font (size 1 1) (thickness 0.15)))
     )
@@
     (at 84.5 58 -90)
     (property "Mouser" "579-MCP2221A-I/SL")
-    (property "Name" "MCP2221A-ISL")
+    (property "Name" "MCP2221A")
     (property "Sheetfile" "pic8bit-hid.kicad_sch")
     (property "Sheetname" "HID")
@@
       (effects (font (size 1 1) (thickness 0.15)) (justify mirror))
     )
-    (fp_text value "2K4" (at 0 -2 90) (layer "B.Fab")
+    (fp_text value "10K" (at 0 -2 90) (layer "B.Fab")
       (effects (font (size 1 1) (thickness 0.15)) (justify mirror))
     )

Commit message: Update Mini
Parts:
- IC301: value ONSEMI-CAT4002A-SOT-23 -> CAT4002A
- IC302: value MICROCHIP-MCP2221A-ISL -> MCP2221A

Commit message: Update
Parts:
- added kibuzzard-627E43A1: G003, kibuzzard-627E43A1, F.Cu at (77.5, 143.5)
- added kibuzzard-627E43A7: G004, kibuzzard-627E43A7, F.Cu at (136.5, 143.5)
- added kibuzzard-627E43EB: G006, kibuzzard-627E43EB, F.Cu at (79.5, 129.5)
- added kibuzzard-627E43EB: G***, kibuzzard-627E43EB, F.Cu at (134.8, 118.2)
- added kibuzzard-627E43EB: G008, kibuzzard-627E43EB, F.Cu at (72.8, 90.5)
- added kibuzzard-627E4456: G007, kibuzzard-627E4456, F.Cu at (79.5, 123.0)
- added kibuzzard-627E464E: G***, kibuzzard-627E464E, F.Cu at (94.5, 52.5)
- added kibuzzard-627E4655: G***, kibuzzard-627E4655, F.Cu at (97.0, 53.6)
- K203, K206: footprint tronixio:zzHARWIN-M20-782144x -> tronixio:HARWIN-M20-782144x
Routing:
- net /HID/UTX: track 70.9 -> 71.5 mm
- net Net-(C301-Pad1): track 6.40 -> 6.90 mm
Other:
- board text removed: "+3V3"
- board text removed: "+5V IN"
