File: Kicad/mini/pic8bit.kicad_pcb (KiCad board)
At the start: 2 copper layers, 80 x 100 mm, 94 parts, among them IC201 TLV1117-33, IC202 MICROCHIP-PIC16F1778-ISP, IC301 CAT4002A, IC302 MCP2221A, K101 PE-450-4X6X-BLACK, K201 *Power & UART, K202 MCU 1, K203 MCU 1, K204 ICSP, K205 MCU 2, K206 MCU 2, K301 HARWIN-254-F-1X08-VERTICAL, K302 HARWIN-254-F-1X06-VERTICAL, P301 PIHER-PT10MV-10K, P302 PIHER-PT10MV-10K

Commit message: Update pic8bit.kicad_pcb
Routing:
- net +3V3: vias 20 -> 18
Changed lines of the file:
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@@
     (fp_arc (start -4 3.3) (mid -4.903738 -1.844892) (end -0.9 -5.2) (layer "F.Fab") (width 0.1))
     (fp_arc (start -0.3 4.4) (mid -0.923087 4.342349) (end -1.5 4.1) (layer "F.Fab") (width 0.1))
-    (fp_arc (start 1.5 4.1) (mid 0.923087 4.34235) (end 0.3 4.4) (layer "F.Fab") (width 0.1))
+    (fp_arc (start 1.5 4.1) (mid 0.923087 4.342349) (end 0.3 4.4) (layer "F.Fab") (width 0.1))
     (fp_circle (center -2.5 5.3) (end -1.5 5.3) (layer "F.Fab") (width 0.1) (fill none))
     (fp_circle (center 2.5 5.3) (end 3.5 5.3) (layer "F.Fab") (width 0.1) (fill none))
@@
     (fp_arc (start 0.9 -5.2) (mid 4.903738 -1.844893) (end 4 3.3) (layer "F.Fab") (width 0.1))
     (fp_arc (start -4 3.3) (mid -4.903738 -1.844892) (end -0.9 -5.2) (layer "F.Fab") (width 0.1))
-    (fp_arc (start 1.5 4.1) (mid 0.923087 4.34235) (end 0.3 4.4) (layer "F.Fab") (width 0.1))
+    (fp_arc (start 1.5 4.1) (mid 0.923087 4.342349) (end 0.3 4.4) (layer "F.Fab") (width 0.1))
     (fp_arc (start -0.3 4.4) (mid -0.923087 4.342349) (end -1.5 4.1) (layer "F.Fab") (width 0.1))
     (fp_circle (center 0 -4.7) (end 1 -4.7) (layer "F.Fab") (width 0.1) (fill none))
@@
   (gr_line (start 137.25 48) (end 137.25 57.5) (layer "F.SilkS") (width 0.2))
   (gr_rect (start 105.5 57.5) (end 120 48.5) (layer "B.Mask") (width 0.1) (fill solid))
-  (gr_rect (start 109 57.75) (end 120 48.25) (layer "F.Mask") (width 0.1) (fill solid))
+  (gr_rect (start 109 57.5) (end 120 48.5) (layer "F.Mask") (width 0.1) (fill solid))
   (gr_line (start 57 47) (end 56.5 47) (layer "Dwgs.User") (width 0.05))
   (gr_line (start 57 49.5) (end 57 44.5) (layer "Dwgs.User") (width 0.05))
@@
   (via (at 104.5 52) (size 0.6) (drill 0.3) (layers "F.Cu" "B.Cu") (net 3))
   (via (at 73 124) (size 0.6) (drill 0.3) (layers "F.Cu" "B.Cu") (net 3))
-  (via (at 111 57) (size 1) (drill 0.5) (layers "F.Cu" "B.Cu") (free) (net 3))
-  (via (at 113 49) (size 1) (drill 0.5) (layers "F.Cu" "B.Cu") (free) (net 3))
-  (via (at 115 57) (size 1) (drill 0.5) (layers "F.Cu" "B.Cu") (free) (net 3))
+  (via (at 113 49.25) (size 1) (drill 0.5) (layers "F.Cu" "B.Cu") (free) (net 3))
+  (via (at 115 56.75) (size 1) (drill 0.5) (layers "F.Cu" "B.Cu") (free) (net 3))
   (via (at 84.5 107) (size 0.6) (drill 0.3) (layers "F.Cu" "B.Cu") (net 3))
-  (via (at 115 49) (size 1) (drill 0.5) (layers "F.Cu" "B.Cu") (free) (net 3))
-  (via (at 113 57) (size 1) (drill 0.5) (layers "F.Cu" "B.Cu") (free) (net 3))
-  (via (at 119 49) (size 1) (drill 0.5) (layers "F.Cu" "B.Cu") (free) (net 3))
+  (via (at 115 49.25) (size 1) (drill 0.5) (layers "F.Cu" "B.Cu") (free) (net 3))
+  (via (at 113 56.75) (size 1) (drill 0.5) (layers "F.Cu" "B.Cu") (free) (net 3))
+  (via (at 119 49.25) (size 1) (drill 0.5) (layers "F.Cu" "B.Cu") (free) (net 3))
   (via (at 73 136) (size 0.6) (drill 0.3) (layers "F.Cu" "B.Cu") (net 3))
   (via (at 87.5 76.5) (size 0.6) (drill 0.3) (layers "F.Cu" "B.Cu") (net 3))
   (via (at 119 53) (size 1) (drill 0.5) (layers "F.Cu" "B.Cu") (free) (net 3))
-  (via (at 117 49) (size 1) (drill 0.5) (layers "F.Cu" "B.Cu") (free) (net 3))
+  (via (at 117 49.25) (size 1) (drill 0.5) (layers "F.Cu" "B.Cu") (free) (net 3))
   (via (at 137.25 134) (size 0.6) (drill 0.3) (layers "F.Cu" "B.Cu") (net 3))
   (via (at 113 76.5) (size 0.6) (drill 0.3) (layers "F.Cu" "B.Cu") (net 3))
   (via (at 119 55) (size 1) (drill 0.5) (layers "F.Cu" "B.Cu") (free) (net 3))
-  (via (at 111 49) (size 1) (drill 0.5) (layers "F.Cu" "B.Cu") (free) (net 3))
-  (via (at 119 57) (size 1) (drill 0.5) (layers "F.Cu" "B.Cu") (free) (net 3))
-  (via (at 117 57) (size 1) (drill 0.5) (layers "F.Cu" "B.Cu") (free) (net 3))
+  (via (at 119 56.75) (size 1) (drill 0.5) (layers "F.Cu" "B.Cu") (free) (net 3))
+  (via (at 117 56.75) (size 1) (drill 0.5) (layers "F.Cu" "B.Cu") (free) (net 3))
   (segment (start 110.82 100.9) (end 110.82 103.75) (width 0.4) (layer "B.Cu") (net 3))
   (segment (start 87.5 76.5) (end 84.5 73.5) (width 0.5) (layer "B.Cu") (net 3))
@@
     (polygon
       (pts
-        (xy 120 57.75)
-        (xy 109 57.75)
-        (xy 109 48.25)
-        (xy 120 48.25)
+        (xy 120 57.5)
+        (xy 109 57.5)
+        (xy 109 48.5)
+        (xy 120 48.5)
       )
     )

Commit message: Up
Parts:
- removed IC201: TLV1117-33, tronixio:SOT-223-3
- removed IC202: MICROCHIP-PIC16F1778-ISP, tronixio:DIP-28-W762-SOCKET
- removed IC301: CAT4002A, tronixio:SOT-23-6
- removed IC302: MCP2221A, tronixio:SOIC-SL-14
- added U201: TLV1117-33, tronixio:SOT-223-3, F.Cu at (110.0, 53.0)
- added U202: MICROCHIP-PIC16F1778-ISP, tronixio:DIP-28-W762, F.Cu at (90.5, 96.8)
- added U301: CAT4002A, tronixio:SOT-23-6, B.Cu at (75.0, 65.7)
- added U302: MCP2221A, tronixio:SOIC-SL-14, B.Cu at (84.5, 58.0)

Commit message: Update
Parts:
- S303: footprint tronixio:BOURNS-PEC12R -> tronixio:BOURNS-PEC12R-SWITCH
Changed lines of the file:
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@@
     (at 90.5 96.75 90)
     (property "Mouser" "579-PIC16F1778-I/SP")
-    (property "Name" "PIC16F1778-ISP")
+    (property "Name" "PIC16F/PIC18F")
     (property "Sheetfile" "pic8bit-mcu.kicad_sch")
     (property "Sheetname" "MCU")
@@
     (fp_arc (start -4 3.3) (mid -4.903738 -1.844892) (end -0.9 -5.2) (layer "F.Fab") (width 0.1))
     (fp_arc (start -0.3 4.4) (mid -0.923087 4.342349) (end -1.5 4.1) (layer "F.Fab") (width 0.1))
-    (fp_arc (start 1.5 4.1) (mid 0.923087 4.342349) (end 0.3 4.4) (layer "F.Fab") (width 0.1))
+    (fp_arc (start 1.5 4.1) (mid 0.923087 4.34235) (end 0.3 4.4) (layer "F.Fab") (width 0.1))
     (fp_circle (center -2.5 5.3) (end -1.5 5.3) (layer "F.Fab") (width 0.1) (fill none))
     (fp_circle (center 2.5 5.3) (end 3.5 5.3) (layer "F.Fab") (width 0.1) (fill none))
@@
     (fp_arc (start 0.9 -5.2) (mid 4.903738 -1.844893) (end 4 3.3) (layer "F.Fab") (width 0.1))
     (fp_arc (start -4 3.3) (mid -4.903738 -1.844892) (end -0.9 -5.2) (layer "F.Fab") (width 0.1))
-    (fp_arc (start 1.5 4.1) (mid 0.923087 4.342349) (end 0.3 4.4) (layer "F.Fab") (width 0.1))
+    (fp_arc (start 1.5 4.1) (mid 0.923087 4.34235) (end 0.3 4.4) (layer "F.Fab") (width 0.1))
     (fp_arc (start -0.3 4.4) (mid -0.923087 4.342349) (end -1.5 4.1) (layer "F.Fab") (width 0.1))
     (fp_circle (center 0 -4.7) (end 1 -4.7) (layer "F.Fab") (width 0.1) (fill none))
@@
     )
   )
-  (footprint "tronixio:BOURNS-PEC12R" (layer "F.Cu")
+  (footprint "tronixio:BOURNS-PEC12R-SWITCH" (layer "F.Cu")
     (at 138.5 131)
     (property "Mouser" "652-PEC12R-4215F-S24")
@@
     (property "Sheetname" "HID")
     (attr through_hole)
-    (fp_text reference "S303" (at 0 -8) (layer "F.Fab")
-      (effects (font (size 1 1) (thickness 0.15)))
-    )
-    (fp_text value "BOURNS-PEC12R-24DENTS" (at -7.5 0.5 90) (layer "F.Fab")
+    (fp_text reference "S303" (at 0 -10.16) (layer "F.Fab")
+      (effects (font (size 1 1) (thickness 0.15)))
+    )
+    (fp_text value "BOURNS-PEC12R-24DENTS" (at 0 10.16) (layer "F.Fab")
       (effects (font (size 1 1) (thickness 0.15)))
     )
     (fp_line (start -6.2 -6.7) (end -3.6 -6.7) (layer "F.SilkS") (width 0.12))
-    (fp_line (start 3.6 -6.7) (end 6.2 -6.7) (layer "F.SilkS") (width 0.12))
-    (fp_line (start 6.2 1.9) (end 6.2 6.7) (layer "F.SilkS") (width 0.12))
-    (fp_line (start 6.2 -6.7) (end 6.2 -1.9) (layer "F.SilkS") (width 0.12))
     (fp_line (start -6.2 1.9) (end -6.2 6.7) (layer "F.SilkS") (width 0.12))
-    (fp_line (start -6.2 6.7) (end -3.6 6.7) (layer "F.SilkS") (width 0.12))
-    (fp_line (start -1.3 -6.7) (end 1.3 -6.7) (layer "F.SilkS") (width 0.12))
     (fp_line (start 3.6 6.7) (end 6.2 6.7) (layer "F.SilkS") (width 0.12))
     (fp_line (start -6.2 -6.7) (end -6.2 -1.9) (layer "F.SilkS") (width 0.12))
+    (fp_line (start 6.2 1.9) (end 6.2 6.7) (layer "F.SilkS") (width 0.12))
+    (fp_line (start -1.3 -6.7) (end 1.3 -6.7) (layer "F.SilkS") (width 0.12))
+    (fp_line (start 3.6 -6.7) (end 6.2 -6.7) (layer "F.SilkS") (width 0.12))
+    (fp_line (start -6.2 6.7) (end -3.6 6.7) (layer "F.SilkS") (width 0.12))
+    (fp_line (start 6.2 -6.7) (end 6.2 -1.9) (layer "F.SilkS") (width 0.12))
     (fp_rect (start -7.7 8.6) (end 7.7 -8.1) (layer "F.CrtYd") (width 0.05) (fill none))
     (fp_line (start -2 1.5) (end -1.8 1) (layer "F.Fab") (width 0.1))
@@
     (fp_line (start 2 1.5) (end 1.8 1) (layer "F.Fab") (width 0.1))
     (fp_line (start -2 1.5) (end 2 1.5) (layer "F.Fab") (width 0.1))
-    (fp_rect (start -0.5 7.1) (end 0.5 6.7) (layer "F.Fab") (width 0.1) (fill solid))
+    (fp_rect (start -6.2 6.7) (end 6.2 -6.7) (layer "F.Fab") (width 0.1) (fill none))
+    (fp_rect (start 2 -6.7) (end 3 -7.1) (layer "F.Fab") (width 0.1) (fill solid))
+    (fp_rect (start -3 -6.7) (end -2 -7.1) (layer "F.Fab") (width 0.1) (fill solid))
     (fp_rect (start -7 1.25) (end -6.2 -1.25) (layer "F.Fab") (width 0.1) (fill solid))
     (fp_rect (start -3 7.1) (end -2 6.7) (layer "F.Fab") (width 0.1) (fill solid))
-    (fp_rect (start 2 -6.7) (end 3 -7.1) (layer "F.Fab") (width 0.1) (fill solid))
-    (fp_rect (start -3 -6.7) (end -2 -7.1) (layer "F.Fab") (width 0.1) (fill solid))
+    (fp_rect (start -0.5 7.1) (end 0.5 6.7) (layer "F.Fab") (width 0.1) (fill solid))
+    (fp_rect (start 6.2 1.25) (end 7 -1.25) (layer "F.Fab") (width 0.1) (fill solid))
     (fp_rect (start 2 7.1) (end 3 6.7) (layer "F.Fab") (width 0.1) (fill solid))
-    (fp_rect (start -6.2 6.7) (end 6.2 -6.7) (layer "F.Fab") (width 0.1) (fill none))
-    (fp_rect (start 6.2 1.25) (end 7 -1.25) (layer "F.Fab") (width 0.1) (fill solid))
     (fp_arc (start -1.8 1) (mid 0 -2.046667) (end 1.8 1) (layer "F.Fab") (width 0.1))
+    (fp_circle (center 0 0) (end 2.5 0) (layer "F.Fab") (width 0.1) (fill none))
+    (fp_circle (center 0 0) (end 3.5 0) (layer "F.Fab") (width 0.1) (fill none))
+    (fp_circle (center -5.3 6) (end -5 6) (layer "F.Fab") (width 0.1) (fill none))
     (fp_circle (center 5.3 6) (end 5.6 6) (layer "F.Fab") (width 0.1) (fill none))
     (fp_circle (center -5.3 -5.5) (end -5 -5.5) (layer "F.Fab") (width 0.1) (fill none))
-    (fp_circle (center -5.3 6) (end -5 6) (layer "F.Fab") (width 0.1) (fill none))
-    (fp_circle (center 0 0) (end 3.5 0) (layer "F.Fab") (width 0.1) (fill none))
     (fp_circle (center 5.3 -5.5) (end 5.6 -5.5) (layer "F.Fab") (width 0.1) (fill none))
-    (fp_circle (center 0 0) (end 2.5 0) (layer "F.Fab") (width 0.1) (fill none))
     (pad "1" thru_hole circle (at -2.5 7.5) (size 1.8 1.8) (drill 1) (layers *.Cu *.Mask)
       (net 9 "Net-(C305-Pad1)") (pinfunction "A") (pintype "passive"))
+    (pad "2" thru_hole rect (at 6.5 0) (size 2 3.2) (drill oval 1 2.4) (layers *.Cu *.Mask)
+      (net 2 "GND") (pintype "passive"))
     (pad "2" thru_hole circle (at 0 7.5) (size 1.8 1.8) (drill 1) (layers *.Cu *.Mask)
-      (net 2 "GND") (pinfunction "C") (pintype "passive"))
-    (pad "2" thru_hole rect (at 6.5 0) (size 2 3.2) (drill oval 1 2.4) (layers *.Cu *.Mask)
-      (net 2 "GND") (pinfunction "C") (pintype "passive"))
+      (net 2 "GND") (pintype "passive"))
     (pad "2" thru_hole rect (at -6.5 0) (size 2 3.2) (drill oval 1 2.4) (layers *.Cu *.Mask)
-      (net 2 "GND") (pinfunction "C") (pintype "passive"))
+      (net 2 "GND") (pintype "passive"))
     (pad "3" thru_hole circle (at 2.5 7.5) (size 1.8 1.8) (drill 1) (layers *.Cu *.Mask)
       (net 10 "Net-(C307-Pad1)") (pinfunction "B") (pintype "passive"))
     (pad "4" thru_hole circle (at 2.5 -7) (size 1.8 1.8) (drill 1) (layers *.Cu *.Mask)
-      (net 2 "GND") (pinfunction "2") (pintype "passive"))
+      (net 2 "GND") (pintype "passive"))
     (pad "5" thru_hole circle (at -2.5 -7) (size 1.8 1.8) (drill 1) (layers *.Cu *.Mask)
-      (net 8 "Net-(R309-Pad2)") (pinfunction "1") (pintype "passive"))
+      (net 8 "Net-(R309-Pad2)") (pintype "passive"))
     (model "${KICAD6_USER_3DMODEL_DIR}/Discret/BOURNS-PEC12R.step"
       (offset (xyz 0 0 0))

Commit message: Update
Parts:
- F201: value F050 -> 500mA; footprint tronixio:FUSE-1206 -> tronixio:FUSE-0805
- JP201: value *Power IN -> Power IN
- K203: value MCU 1 -> MCU 2
- K205: value MCU 2 -> MCU 1
- K302: footprint tronixio:zzHARWIN-M20-782064x -> tronixio:HARWIN-M20-782064x
- P301, P302: value PIHER-PT10MV-10K -> 10K
- R315: value 10K -> 1K
- S303: value BOURNS-PEC12R-24DENTS -> BOURNS-PEC12R-24DENTS-SWITCH
- U202: value MICROCHIP-PIC16F1778-ISP -> PIC16F/PIC18F
- U302: value MCP2221A -> MCP2221A-ISL; footprint tronixio:SOIC-SL-14 -> tronixio:SOIC-14

Commit message: Update
Parts:
- K203: value MCU 2 -> MCU 1
- K205: value MCU 1 -> MCU 2
- U202: footprint tronixio:DIP-28-W762 -> tronixio:DIP-28-W762-SOCKET

Commit message: Update
Parts:
- C201, C202, C203, C205, C301, C302, C303, C304, C305, C306, C307: footprint tronixio:CAPACITOR-1206 -> tronixio:CAPACITOR-SMD-1206
- F201: footprint tronixio:FUSE-0805 -> tronixio:FUSE-SMD-1206
- LED201, LED301, LED302: footprint tronixio:LED-1206 -> tronixio:LED-SMD-1206
- R201, R202, R203, R204, R205, R301, R302, R303, R304, R305, R306, R307, R308, R309, R310, R311, R312, R313, R314, R315, R316, R317, R318, R319, R320: footprint tronixio:RESISTOR-1206 -> tronixio:RESISTOR-SMD-1206
- U202: footprint tronixio:DIP-28-W762-SOCKET -> tronixio:DIP-28-W762
