File: Kicad/mini/pic8bit.kicad_pcb (KiCad board)
At the start: 2 copper layers, 80 x 100 mm, 94 parts, among them K101 PE-450-4X6X-BLACK, K201 *Power & UART, K202 MCU 1, K203 MCU 1, K204 ICSP, K205 MCU 2, K206 MCU 2, K301 HARWIN-254-F-1X08-VERTICAL, K302 HARWIN-254-F-1X06-VERTICAL, P301 10K, P302 10K, U201 TLV1117-33, U202 PIC16F/PIC18F, U301 CAT4002A, U302 MCP2221A-ISL

Commit message: Update
Parts:
- U301: footprint tronixio:SOT-23-6 -> tronixioZZZ:SC-70-6
- U302: value MCP2221A-ISL -> MCP2221A
- moved U301 0.30 mm to (75.0, 65.4)
Routing:
- net GND: track 108.5 -> 113.3 mm
- net +5V: track 63.5 -> 64.3 mm
Changed lines of the file:
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@@
     )
   )
-  (footprint "tronixio:SOT-23-6" (layer "B.Cu")
-    (at 75 65.7 180)
-    (property "Mouser" "863-CAT4002ATD-GT3")
-    (property "Name" "ONSEMI-CAT4002A-SOT-23")
+  (footprint "tronixioZZZ:SC-70-6" (layer "B.Cu")
+    (at 75 65.4 180)
+    (property "Mouser" "863-CAT4002ASD-GT3")
+    (property "Name" "ONSEMI-CAT4002A-SC-70")
     (property "Sheetfile" "pic8bit-hid.kicad_sch")
     (property "Sheetname" "HID")
@@
       (effects (font (size 1 1) (thickness 0.15)) (justify mirror))
     )
-    (fp_rect (start -2.1 -1.7) (end 2.1 1.7) (layer "B.CrtYd") (width 0.05) (fill none))
-    (fp_rect (start 1 1.2) (end 1.2 0.7) (layer "B.Fab") (width 0.1) (fill solid))
-    (fp_rect (start -1.2 1.2) (end -1 0.7) (layer "B.Fab") (width 0.1) (fill solid))
-    (fp_rect (start -1.2 0.25) (end -1 -0.25) (layer "B.Fab") (width 0.1) (fill solid))
-    (fp_rect (start 1 0.25) (end 1.2 -0.25) (layer "B.Fab") (width 0.1) (fill solid))
-    (fp_rect (start -1.2 -0.7) (end -1 -1.2) (layer "B.Fab") (width 0.1) (fill solid))
-    (fp_rect (start 1 -0.7) (end 1.2 -1.2) (layer "B.Fab") (width 0.1) (fill solid))
-    (fp_rect (start -1 -1.5) (end 1 1.5) (layer "B.Fab") (width 0.1) (fill none))
-    (fp_circle (center -0.5 1) (end -0.35 1) (layer "B.Fab") (width 0.1) (fill solid))
-    (pad "1" smd roundrect (at -1.3 0.95 180) (size 1.2 0.6) (layers "B.Cu" "B.Paste" "B.Mask") (roundrect_rratio 0.15)
+    (fp_rect (start -1.5 -1.2) (end 1.5 1.2) (layer "B.CrtYd") (width 0.05) (fill none))
+    (fp_rect (start 0.9 0.5) (end 0.6 0.8) (layer "B.Fab") (width 0.1) (fill solid))
+    (fp_rect (start -0.6 -0.15) (end -0.9 0.15) (layer "B.Fab") (width 0.1) (fill solid))
+    (fp_rect (start -0.6 0.5) (end -0.9 0.8) (layer "B.Fab") (width 0.1) (fill solid))
+    (fp_rect (start 0.9 -0.15) (end 0.6 0.15) (layer "B.Fab") (width 0.1) (fill solid))
+    (fp_rect (start -0.6 -1) (end 0.6 1) (layer "B.Fab") (width 0.1) (fill none))
+    (fp_rect (start -0.6 -0.8) (end -0.9 -0.5) (layer "B.Fab") (width 0.1) (fill solid))
+    (fp_rect (start 0.9 -0.8) (end 0.6 -0.5) (layer "B.Fab") (width 0.1) (fill solid))
+    (fp_circle (center -0.3 0.7) (end -0.2 0.7) (layer "B.Fab") (width 0.1) (fill solid))
+    (pad "1" smd roundrect (at -0.95 0.65 180) (size 0.7 0.4) (layers "B.Cu" "B.Paste" "B.Mask") (roundrect_rratio 0.1)
       (net 62 "Net-(JP301-Pad2)") (pinfunction "EN") (pintype "input"))
-    (pad "2" smd roundrect (at -1.3 0 180) (size 1.2 0.6) (layers "B.Cu" "B.Paste" "B.Mask") (roundrect_rratio 0.15)
+    (pad "2" smd roundrect (at -0.95 0 180) (size 0.7 0.4) (layers "B.Cu" "B.Paste" "B.Mask") (roundrect_rratio 0.1)
       (net 2 "GND") (pinfunction "GND") (pintype "power_in"))
-    (pad "3" smd roundrect (at -1.3 -0.95 180) (size 1.2 0.6) (layers "B.Cu" "B.Paste" "B.Mask") (roundrect_rratio 0.15)
+    (pad "3" smd roundrect (at -0.95 -0.65 180) (size 0.7 0.4) (layers "B.Cu" "B.Paste" "B.Mask") (roundrect_rratio 0.1)
       (net 1 "+5V") (pinfunction "VIN") (pintype "power_in"))
-    (pad "4" smd roundrect (at 1.3 -0.95 180) (size 1.2 0.6) (layers "B.Cu" "B.Paste" "B.Mask") (roundrect_rratio 0.15)
+    (pad "4" smd roundrect (at 0.95 -0.65 180) (size 0.7 0.4) (layers "B.Cu" "B.Paste" "B.Mask") (roundrect_rratio 0.1)
       (net 64 "unconnected-(U301-Pad4)") (pinfunction "LED2") (pintype "output+no_connect"))
-    (pad "5" smd roundrect (at 1.3 0 180) (size 1.2 0.6) (layers "B.Cu" "B.Paste" "B.Mask") (roundrect_rratio 0.15)
+    (pad "5" smd roundrect (at 0.95 0 180) (size 0.7 0.4) (layers "B.Cu" "B.Paste" "B.Mask") (roundrect_rratio 0.1)
       (net 63 "Net-(R308-Pad1)") (pinfunction "RSET") (pintype "passive"))
-    (pad "6" smd roundrect (at 1.3 0.95 180) (size 1.2 0.6) (layers "B.Cu" "B.Paste" "B.Mask") (roundrect_rratio 0.15)
+    (pad "6" smd roundrect (at 0.95 0.65 180) (size 0.7 0.4) (layers "B.Cu" "B.Paste" "B.Mask") (roundrect_rratio 0.1)
       (net 27 "BCKL") (pinfunction "LED1") (pintype "output"))
-    (model "${KICAD6_USER_3DMODEL_DIR}/SMD/SOT-23-6.wrl"
+    (model "${KICAD6_USER_3DMODEL_DIR}/SMD/SC-70-6.wrl"
       (offset (xyz 0 0 0))
       (scale (xyz 1 1 1))
@@
       (effects (font (size 1 1) (thickness 0.15)) (justify mirror))
     )
-    (fp_text value "MCP2221A-ISL" (at 0 -5.5 90) (layer "B.Fab")
+    (fp_text value "MCP2221A" (at 0 -5.5 90) (layer "B.Fab")
       (effects (font (size 1 1) (thickness 0.15)) (justify mirror))
     )
@@
   )
   (gr_circle (center 79.75 55.5) (end 79.95 55.5) (layer "B.SilkS") (width 0.1) (fill solid))
-  (gr_circle (center 76 63.5) (end 76.2 63.5) (layer "B.SilkS") (width 0.1) (fill solid))
+  (gr_circle (center 76 63.75) (end 76.2 63.75) (layer "B.SilkS") (width 0.1) (fill solid))
   (gr_line (start 88.5 100) (end 88.5 105) (layer "F.SilkS") (width 0.2))
   (gr_line (start 125.5 141) (end 125.5 146) (layer "F.SilkS") (width 0.2))
@@
   (segment (start 70.45 82.23) (end 70.45 73.25) (width 0.5) (layer "B.Cu") (net 1))
   (segment (start 83 69) (end 77.5 69) (width 0.5) (layer "B.Cu") (net 1))
-  (segment (start 76.3 66.65) (end 77.15 66.65) (width 0.5) (layer "B.Cu") (net 1))
   (segment (start 70.45 73.25) (end 70.45 71.05) (width 0.5) (layer "B.Cu") (net 1))
+  (segment (start 77.5 66.75) (end 76.8 66.05) (width 0.4) (layer "B.Cu") (net 1))
   (segment (start 70.45 71.05) (end 71 70.5) (width 0.5) (layer "B.Cu") (net 1))
-  (segment (start 77.15 66.65) (end 77.5 67) (width 0.5) (layer "B.Cu") (net 1))
   (segment (start 77.5 70) (end 77.5 69) (width 0.5) (layer "B.Cu") (net 1))
+  (segment (start 77.5 69) (end 77.5 66.75) (width 0.4) (layer "B.Cu") (net 1))
   (segment (start 102.3 60.2) (end 104.5 58) (width 0.5) (layer "B.Cu") (net 1))
   (segment (start 96.5 62) (end 96.5 60.2) (width 0.5) (layer "B.Cu") (net 1))
@@
   (segment (start 100.5 60.2) (end 102.3 60.2) (width 0.5) (layer "B.Cu") (net 1))
   (segment (start 77 70.5) (end 77.5 70) (width 0.5) (layer "B.Cu") (net 1))
-  (segment (start 77.5 67) (end 77.5 69) (width 0.5) (layer "B.Cu") (net 1))
+  (segment (start 76.8 66.05) (end 75.95 66.05) (width 0.4) (layer "B.Cu") (net 1))
   (segment (start 104.5 50.25) (end 104.95 50.7) (width 0.8) (layer "F.Cu") (net 2))
   (segment (start 104.95 50.7) (end 106.85 50.7) (width 0.8) (layer "F.Cu") (net 2))
@@
   (via (at 69.4 98.105) (size 0.6) (drill 0.3) (layers "F.Cu" "B.Cu") (net 2))
   (via (at 101.5 54) (size 0.6) (drill 0.3) (layers "F.Cu" "B.Cu") (net 2))
+  (segment (start 78.9 65.4) (end 79.5 66) (width 0.4) (layer "B.Cu") (net 2))
   (segment (start 113.355 99.375) (end 114.625 98.105) (width 0.4) (layer "B.Cu") (net 2))
   (segment (start 108.28 145.1) (end 108.28 142.25) (width 0.5) (layer "B.Cu") (net 2))
+  (segment (start 79.5 66) (end 79.5 67) (width 0.4) (layer "B.Cu") (net 2))
   (segment (start 107.005 104.455) (end 107.005 106.36) (width 0.5) (layer "B.Cu") (net 2))
   (segment (start 113.36 100.9) (end 113.36 99.38) (width 0.4) (layer "B.Cu") (net 2))
@@
   (segment (start 113.36 103.75) (end 113.36 100.9) (width 0.4) (layer "B.Cu") (net 2))
   (segment (start 113.36 99.38) (end 113.355 99.375) (width 0.4) (layer "B.Cu") (net 2))
+  (segment (start 75.95 65.4) (end 78.9 65.4) (width 0.4) (layer "B.Cu") (net 2))
   (segment (start 142.25 132.5) (end 142.25 130) (width 0.5) (layer "B.Cu") (net 2))
   (segment (start 107.005 100.01) (end 107.005 104.46) (width 0.2) (layer "B.Cu") (net 2))
@@
   (segment (start 131.4 106.5) (end 136.4 111.5) (width 0.5) (layer "B.Cu") (net 26))
   (segment (start 136.4 111.5) (end 139.5 111.5) (width 0.5) (layer "B.Cu") (net 26))
-  (segment (start 70.45 64.75) (end 73.7 64.75) (width 0.5) (layer "B.Cu") (net 27))
+  (segment (start 74.05 64.75) (end 70.45 64.75) (width 0.4) (layer "B.Cu") (net 27))
   (segment (start 71.6 98.105) (end 71.6 96.005) (width 0.5) (layer "F.Cu") (net 28))
   (segment (start 71.6 100.205) (end 71.6 98.105) (width 0.5) (layer "F.Cu") (net 28))
@@
   (segment (start 122.245 93.66) (end 122.245 98.105) (width 0.4) (layer "B.Cu") (net 61))
   (segment (start 120.98 103.75) (end 120.98 100.9) (width 0.4) (layer "B.Cu") (net 61))
-  (segment (start 70.45 84.77) (end 75 80.22) (width 0.5) (layer "F.Cu") (net 62))
-  (segment (start 75 80.22) (end 75 64.75) (width 0.5) (layer "F.Cu") (net 62))
+  (segment (start 75 64.75) (end 75 80.22) (width 0.5) (layer "F.Cu") (net 62))
+  (segment (start 75 80.22) (end 70.45 84.77) (width 0.5) (layer "F.Cu") (net 62))
   (via (at 75 64.75) (size 0.6) (drill 0.3) (layers "F.Cu" "B.Cu") (net 62))
-  (segment (start 77.25 64.75) (end 78 64) (width 0.5) (layer "B.Cu") (net 62))
-  (segment (start 78 64) (end 79.5 64) (width 0.5) (layer "B.Cu") (net 62))
-  (segment (start 76.3 64.75) (end 77.25 64.75) (width 0.5) (layer "B.Cu") (net 62))
-  (segment (start 76.3 64.75) (end 75 64.75) (width 0.5) (layer "B.Cu") (net 62))
-  (segment (start 75 66) (end 75 69) (width 0.5) (layer "B.Cu") (net 63))
-  (segment (start 73.7 65.7) (end 74.7 65.7) (width 0.5) (layer "B.Cu") (net 63))
-  (segment (start 74.7 65.7) (end 75 66) (width 0.5) (layer "B.Cu") (net 63))
+  (segment (start 77.675 64) (end 79.5 64) (width 0.4) (layer "B.Cu") (net 62))
+  (segment (start 76.925 64.75) (end 77.675 64) (width 0.4) (layer "B.Cu") (net 62))
+  (segment (start 75.95 64.75) (end 75 64.75) (width 0.4) (layer "B.Cu") (net 62))
+  (segment (start 75.95 64.75) (end 76.925 64.75) (width 0.4) (layer "B.Cu") (net 62))
+  (segment (start 74.65 65.4) (end 75 65.75) (width 0.3) (layer "B.Cu") (net 63))
+  (segment (start 75 65.75) (end 75 69) (width 0.3) (layer "B.Cu") (net 63))
+  (segment (start 74.05 65.4) (end 74.65 65.4) (width 0.3) (layer "B.Cu") (net 63))
   (segment (start 80 81) (end 78.5 82.5) (width 0.5) (layer "F.Cu") (net 65))
   (segment (start 80 64) (end 80 81) (width 0.5) (layer "F.Cu") (net 65))

Commit message: Update Mini
Parts:
- U301: footprint tronixioZZZ:SC-70-6 -> tronixio:SC-70-6
