File: Kicad/mini/pic8bit.kicad_pcb (KiCad board)
At the start: 2 copper layers, 80 x 100 mm, 96 parts, among them K101 PE-450-4X6X-BLACK, K201 *Power & UART, K202 MCU 1, K203 MCU 1, K204 ICSP, K205 MCU 2, K206 MCU 2, K301 HARWIN-254-F-1X08-VERTICAL, K302 HARWIN-254-F-1X06-VERTICAL, P301 10K, P302 10K, U201 TLV1117-33, U202 PIC16F/PIC18F, U301 CAT4002A, U302 MCP2221A

Commit message: Up
Parts:
- C204: footprint tronixio:KEMET-C322 -> tronixio:CAPACITOR-SMD-1206
- K201: footprint tronixio:FCI-USB-TYPE-B-MICRO-THT -> tronixio:USB-TYPE-B-MICRO-TH
- P301, P302, R201, R301, R303, R304, R307, R310, R311, R312, R313, R314, R316, R317: value 10K -> 10k
- R202, R302, R305, R306, R309, R320: value 1K -> 1k
- R203, R204, R205, R318, R319: value 4K7 -> 4k7
- R308: value 2K4 -> 2k4
- R315: value 1K -> 10k
- U202: footprint tronixio:DIP-28-W762 -> tronixio:DIP-28-W762-SOCKET
- moved JP203 1.00 mm to (132.0, 94.5)
- turned S303 to 180 degrees
Connections:
- S303 pad 4: GND -> Net-(R309-Pad2)
- S303 pad 5: Net-(R309-Pad2) -> GND
Routing:
- net Net-(C204-Pad1): track 5.03 -> 3.60 mm
- net GND: track 113.3 -> 114.6 mm, vias 4 -> 5
- net Net-(K202-Pin_6): track 83.6 -> 82.5 mm

Commit message: Up
Parts:
- C204: moved to B.Cu
- moved C204 3.50 mm to (132.0, 93.2)
- moved JP203 3.50 mm to (128.5, 94.5)
Routing:
- net Net-(K202-Pin_6): track 82.5 -> 79.1 mm
- net GND: track 114.6 -> 113.3 mm, vias 5 -> 4

Commit message: Up
Parts:
- H101, H102, H103, H104: value KEYSTONE-9055 -> 9055
- TP201, TP202: value KEYSTONE-5006 -> 5006
- TP203: value KEYSTONE-2000-3 -> 2000-3
Changed lines of the file:
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@@
     (fp_arc (start 0.9 -5.2) (mid 4.903738 -1.844893) (end 4 3.3)
       (stroke (width 0.1) (type solid)) (layer "F.Fab"))
-    (fp_arc (start 1.5 4.1) (mid 0.923087 4.34235) (end 0.3 4.4)
+    (fp_arc (start 1.5 4.1) (mid 0.923087 4.342349) (end 0.3 4.4)
       (stroke (width 0.1) (type solid)) (layer "F.Fab"))
     (fp_circle (center -2.5 5.3) (end -1.5 5.3)
@@
         (effects (font (size 1 1) (thickness 0.15)))
     )
-    (fp_text value "KEYSTONE-5006" (at 0 2.5 90) (layer "F.Fab")
+    (fp_text value "5006" (at 0 2.5 90) (layer "F.Fab")
         (effects (font (size 1 1) (thickness 0.15)))
     )
@@
         (effects (font (size 1 1) (thickness 0.15)))
     )
-    (fp_text value "KEYSTONE-9055" (at 0 3.5) (layer "F.Fab") hide
+    (fp_text value "9055" (at 0 3.5) (layer "F.Fab") hide
         (effects (font (size 1 1) (thickness 0.15)))
     )
@@
         (effects (font (size 1 1) (thickness 0.15)))
     )
-    (fp_text value "KEYSTONE-5006" (at 0 2.5 90) (layer "F.Fab")
+    (fp_text value "5006" (at 0 2.5 90) (layer "F.Fab")
         (effects (font (size 1 1) (thickness 0.15)))
     )
@@
         (effects (font (size 1 1) (thickness 0.15)))
     )
-    (fp_text value "KEYSTONE-9055" (at 0 3.5) (layer "F.Fab") hide
+    (fp_text value "9055" (at 0 3.5) (layer "F.Fab") hide
         (effects (font (size 1 1) (thickness 0.15)))
     )
@@
     (fp_arc (start 0.9 -5.2) (mid 4.903738 -1.844893) (end 4 3.3)
       (stroke (width 0.1) (type solid)) (layer "F.Fab"))
-    (fp_arc (start 1.5 4.1) (mid 0.923087 4.34235) (end 0.3 4.4)
+    (fp_arc (start 1.5 4.1) (mid 0.923087 4.342349) (end 0.3 4.4)
       (stroke (width 0.1) (type solid)) (layer "F.Fab"))
     (fp_circle (center -2.5 5.3) (end -1.5 5.3)
@@
         (effects (font (size 1 1) (thickness 0.15)))
     )
-    (fp_text value "KEYSTONE-2000-3" (at 0 2) (layer "F.Fab")
+    (fp_text value "2000-3" (at 0 2) (layer "F.Fab")
         (effects (font (size 1 1) (thickness 0.15)))
     )
@@
         (effects (font (size 1 1) (thickness 0.15)))
     )
-    (fp_text value "KEYSTONE-9055" (at 0 3.5) (layer "F.Fab") hide
+    (fp_text value "9055" (at 0 3.5) (layer "F.Fab") hide
         (effects (font (size 1 1) (thickness 0.15)))
     )
@@
       (net 3 "+3V3") (pinfunction "Pin_9") (pintype "passive"))
     (pad "10" thru_hole roundrect (at 0 22.86 90) (size 1.8 1.6) (drill 0.7) (layers "*.Cu" "*.Mask") (roundrect_rratio 0.1)
-      (net 2 "GND") (pinfunction "Pin_10") (pintype "passive") (zone_connect 2))
+      (net 2 "GND") (pinfunction "Pin_10") (pintype "passive"))
     (pad "11" thru_hole roundrect (at 0 25.4 90) (size 1.8 1.6) (drill 0.7) (layers "*.Cu" "*.Mask") (roundrect_rratio 0.1)
       (net 48 "/HID/URX") (pinfunction "Pin_11") (pintype "passive"))
@@
         (effects (font (size 1 1) (thickness 0.15)))
     )
-    (fp_text value "KEYSTONE-9055" (at 0 3.5) (layer "F.Fab") hide
+    (fp_text value "9055" (at 0 3.5) (layer "F.Fab") hide
         (effects (font (size 1 1) (thickness 0.15)))
     )
@@
       (net 10 "Net-(S303-A)") (pintype "passive"))
     (pad "2" smd roundrect (at 1.5 0 90) (size 1.3 1.75) (layers "B.Cu" "B.Paste" "B.Mask") (roundrect_rratio 0.1)
-      (net 2 "GND") (pintype "passive") (zone_connect 2))
+      (net 2 "GND") (pintype "passive"))
     (model "${KICAD_USER_3DMODEL_DIR}/SMD/CAPACITOR-1206.wrl"
       (offset (xyz 0 0 0))
@@
   )
   (zone (net 2) (net_name "GND") (layer "B.Cu") (name "GND") (hatch none 0.5)
-    (connect_pads (clearance 0.5))
+    (connect_pads yes (clearance 0.5))
     (min_thickness 0.3) (filled_areas_thickness no)
     (fill yes (thermal_gap 0.5) (thermal_bridge_width 0.5))
