File: Kicad/mini/pic8bit-hid.kicad_sch (KiCad schematic)
At the start: 43 parts, among them K301 HARWIN-254-F-1X08-VERTICAL, K302 HARWIN-254-F-1X06-VERTICAL, P301 PIHER-PT10MV-10K, P302 PIHER-PT10MV-10K, U301 CAT4002A, U302 MCP2221A

Commit message: Update
Parts:
- C301, C305, C307: symbol tronixio:C-0805 -> tronixio:CAPACITOR-1206-10N; Mouser (none) -> 80-C1206C103M5R; Name (none) -> CAPACITOR-1206-10N; Tolerance (none) -> 20%; Voltage (none) -> 50V
- C306: symbol tronixio:C-0805 -> tronixio:CAPACITOR-1206-100N; Mouser (none) -> 80-C1206C104M5R; Name (none) -> CAPACITOR-1206-100N; Tolerance (none) -> 20%; Voltage (none) -> 50V
- R301, R303, R304, R307, R310, R311, R312, R313, R314, R316, R317: symbol tronixio:R-0805 -> tronixio:RESISTOR-1206-10K; Mouser (none) -> 660-RK73B2BTTDD103J; Name (none) -> RESISTOR-1206-10K; Tolerance (none) -> 5%
- R302, R305, R306, R309, R320: symbol tronixio:R-0805 -> tronixio:RESISTOR-1206-1K; Mouser (none) -> 660-RK73B2BTTDD102J; Name (none) -> RESISTOR-1206-1K; Tolerance (none) -> 5%
- R308: symbol tronixio:R-0805 -> tronixio:RESISTOR-1206-2K4; Mouser (none) -> 660-RK73B2BTTD242J; Name (none) -> RESISTOR-1206-2K4; Tolerance (none) -> 5%
- R315: value 10K -> 1K; symbol tronixio:R-0805 -> tronixio:RESISTOR-1206-10K; Mouser (none) -> 660-RK73B2BTTDD103J; Name (none) -> RESISTOR-1206-10K; Tolerance (none) -> 5%
- R318, R319: symbol tronixio:R-0805 -> tronixio:RESISTOR-1206-4K7; Mouser (none) -> 660-RK73B2BTTDD472J; Name (none) -> RESISTOR-1206-4K7; Tolerance (none) -> 5%

Commit message: Update
Parts:
- JP301, JP302, JP303: Name (none) -> HARWIN-254-M-1X02-JUMPER-VERTICAL
- LED301, LED302: symbol tronixio:LED-0805-ORANGE -> tronixio:KINGBRIGHT-LED-1206-BLUE; Mouser 604-APT2012LSECKJ4RV -> 604-APT3216LVBCD; Name (none) -> KINGBRIGHT-LED-1206-BLUE
Changed lines of the file:
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@@
     (pin "2")
   )
-  (symbol (lib_id "tronixio:HARWIN-254-M-1X02-JUMPER-VERTICAL") (at 226.06 55.88 90) (unit 1)
+  (symbol (lib_name "HARWIN-254-M-1X02-JUMPER-VERTICAL_2") (lib_id "tronixio:HARWIN-254-M-1X02-JUMPER-VERTICAL") (at 226.06 55.88 90) (unit 1)
     (in_bom yes) (on_board yes)
     (property "Reference" "JP303" (id 0) (at 230.505 54.61 90)
@@
       (effects (font (size 1.15 1.15)) (justify left))
     )
-    (property "Footprint" "tronixio:HARWIN-M20-999024x" (id 2) (at 238.76 55.88 0)
-      (effects (font (size 1 1)) hide)
-    )
-    (property "Datasheet" "https://www.harwin.com/products/M20-9990846/" (id 3) (at 241.3 55.88 0)
-      (effects (font (size 1 1)) hide)
-    )
-    (property "Mouser" "855-M20-999024" (id 4) (at 243.84 55.88 0)
+    (property "Footprint" "tronixio:HARWIN-M20-999024x" (id 2) (at 241.3 55.88 0)
+      (effects (font (size 1 1)) hide)
+    )
+    (property "Datasheet" "https://www.harwin.com/products/M20-9990846/" (id 3) (at 243.84 55.88 0)
+      (effects (font (size 1 1)) hide)
+    )
+    (property "Mouser" "855-M20-999024" (id 4) (at 246.38 55.88 0)
+      (effects (font (size 1 1)) hide)
+    )
+    (property "Name" "HARWIN-254-M-1X02-JUMPER-VERTICAL" (id 5) (at 238.76 55.88 0)
       (effects (font (size 1 1)) hide)
     )
@@
       (effects (font (size 1.15 1.15)) (justify left))
     )
-    (property "Footprint" "tronixio:HARWIN-M20-999024x" (id 2) (at 238.76 53.34 0)
-      (effects (font (size 1 1)) hide)
-    )
-    (property "Datasheet" "https://www.harwin.com/products/M20-9990846/" (id 3) (at 241.3 53.34 0)
-      (effects (font (size 1 1)) hide)
-    )
-    (property "Mouser" "855-M20-999024" (id 4) (at 243.84 53.34 0)
+    (property "Footprint" "tronixio:HARWIN-M20-999024x" (id 2) (at 241.3 53.34 0)
+      (effects (font (size 1 1)) hide)
+    )
+    (property "Datasheet" "https://www.harwin.com/products/M20-9990846/" (id 3) (at 243.84 53.34 0)
+      (effects (font (size 1 1)) hide)
+    )
+    (property "Mouser" "855-M20-999024" (id 4) (at 246.38 53.34 0)
+      (effects (font (size 1 1)) hide)
+    )
+    (property "Name" "HARWIN-254-M-1X02-JUMPER-VERTICAL" (id 5) (at 238.76 53.34 0)
       (effects (font (size 1 1)) hide)
     )
@@
     (pin "2")
   )
-  (symbol (lib_id "tronixio:LED-0805-ORANGE") (at 218.44 66.04 270) (mirror x) (unit 1)
+  (symbol (lib_id "tronixio:KINGBRIGHT-LED-1206-BLUE") (at 218.44 66.04 270) (mirror x) (unit 1)
     (in_bom yes) (on_board yes)
     (property "Reference" "LED302" (id 0) (at 219.075 63.5 90)
@@
       (effects (font (size 1.15 1.15)) (justify left))
     )
-    (property "Footprint" "tronixio:LED-1206" (id 2) (at 210.82 66.04 0)
-      (effects (font (size 1 1)) hide)
-    )
-    (property "Datasheet" "http://www.kingbrightusa.com/images/catalog/SPEC/APT2012LSECK-J4-PRV.pdf" (id 3) (at 208.28 66.04 0)
-      (effects (font (size 1 1)) hide)
-    )
-    (property "Mouser" "604-APT2012LSECKJ4RV" (id 4) (at 205.74 66.04 0)
+    (property "Footprint" "tronixio:LED-1206" (id 2) (at 208.28 66.04 0)
+      (effects (font (size 1 1)) hide)
+    )
+    (property "Datasheet" "http://www.kingbrightusa.com/images/catalog/SPEC/APT3216LVBC-D.pdf" (id 3) (at 205.74 66.04 0)
+      (effects (font (size 1 1)) hide)
+    )
+    (property "Mouser" "604-APT3216LVBCD" (id 4) (at 203.2 66.04 0)
+      (effects (font (size 1 1)) hide)
+    )
+    (property "Name" "KINGBRIGHT-LED-1206-BLUE" (id 5) (at 210.82 66.04 0)
       (effects (font (size 1 1)) hide)
     )
@@
     (pin "2")
   )
-  (symbol (lib_id "tronixio:LED-0805-ORANGE") (at 213.36 66.04 270) (mirror x) (unit 1)
+  (symbol (lib_id "tronixio:KINGBRIGHT-LED-1206-BLUE") (at 213.36 66.04 270) (mirror x) (unit 1)
     (in_bom yes) (on_board yes)
     (property "Reference" "LED301" (id 0) (at 212.725 63.5 90)
@@
       (effects (font (size 1.15 1.15)) (justify right))
     )
-    (property "Footprint" "tronixio:LED-1206" (id 2) (at 205.74 66.04 0)
-      (effects (font (size 1 1)) hide)
-    )
-    (property "Datasheet" "http://www.kingbrightusa.com/images/catalog/SPEC/APT2012LSECK-J4-PRV.pdf" (id 3) (at 203.2 66.04 0)
-      (effects (font (size 1 1)) hide)
-    )
-    (property "Mouser" "604-APT2012LSECKJ4RV" (id 4) (at 200.66 66.04 0)
+    (property "Footprint" "tronixio:LED-1206" (id 2) (at 203.2 66.04 0)
+      (effects (font (size 1 1)) hide)
+    )
+    (property "Datasheet" "http://www.kingbrightusa.com/images/catalog/SPEC/APT3216LVBC-D.pdf" (id 3) (at 200.66 66.04 0)
+      (effects (font (size 1 1)) hide)
+    )
+    (property "Mouser" "604-APT3216LVBCD" (id 4) (at 198.12 66.04 0)
+      (effects (font (size 1 1)) hide)
+    )
+    (property "Name" "KINGBRIGHT-LED-1206-BLUE" (id 5) (at 205.74 66.04 0)
       (effects (font (size 1 1)) hide)
     )
@@
     (pin "1")
   )
-  (symbol (lib_id "tronixio:HARWIN-254-M-1X02-JUMPER-VERTICAL") (at 109.22 55.88 0) (mirror y) (unit 1)
+  (symbol (lib_name "HARWIN-254-M-1X02-JUMPER-VERTICAL_1") (lib_id "tronixio:HARWIN-254-M-1X02-JUMPER-VERTICAL") (at 109.22 55.88 0) (mirror y) (unit 1)
     (in_bom yes) (on_board yes)
     (property "Reference" "JP301" (id 0) (at 108.585 53.34 0)
@@
       (effects (font (size 1.15 1.15)) (justify left))
     )
-    (property "Footprint" "tronixio:HARWIN-M20-999024x" (id 2) (at 109.22 68.58 0)
-      (effects (font (size 1 1)) hide)
-    )
-    (property "Datasheet" "https://www.harwin.com/products/M20-9990846/" (id 3) (at 109.22 71.12 0)
-      (effects (font (size 1 1)) hide)
-    )
-    (property "Mouser" "855-M20-999024" (id 4) (at 109.22 73.66 0)
-      (effects (font (size 1 1)) hide)
-    )
+    (property "Footprint" "tronixio:HARWIN-M20-999024x" (id 2) (at 109.22 71.12 0)
+      (effects (font (size 1 1)) hide)
+    )
+    (property "Datasheet" "https://www.harwin.com/products/M20-9990846/" (id 3) (at 109.22 73.66 0)
+      (effects (font (size 1 1)) hide)
+    )
+    (property "Mouser" "855-M20-999024" (id 4) (at 109.22 76.2 0)
+      (effects (font (size 1 1)) hide)
+    )
+    (property "Name" "HARWIN-254-M-1X02-JUMPER-VERTICAL" (id 5) (at 109.22 68.58 0)
+      (effects (font (size 1 1)) hide)
+    )

Commit message: Update
Parts:
- C302, C303, C304: symbol tronixio:C-0805 -> tronixio:CAPACITOR-1206-1U; Mouser (none) -> C1206C105M5RACTU; Name (none) -> CAPACITOR-1206-1U; Tolerance (none) -> 20%; Voltage (none) -> 50V
- K301: Name (none) -> HARWIN-254-F-1X06-VERTICAL
- K302: footprint tronixio:zzHARWIN-M20-782064x -> tronixio:HARWIN-M20-782064x; Name (none) -> HARWIN-254-F-1X06-VERTICAL
- P301, P302: value PIHER-PT10MV-10K -> 10K; Name 10K -> PIHER-PT10MV-10K; Tolerance (none) -> 20%
- S301, S302: Name (none) -> CK-KSA
- S303: value BOURNS-PEC12R-24DENTS -> BOURNS-PEC12R-24DENTS-SWITCH; symbol tronixio:BOURNS-PEC12R-24DENTS-SWITCH-15MM -> tronixio:BOURNS-PEC12R-24DENTS-SWITCH; Name (none) -> BOURNS-PEC12R-24DENTS-SWITCH
- U301: Name CAT4002A -> ONSEMI-CAT4002A-SOT-23
- U302: value MCP2221A -> MCP2221A-ISL; footprint tronixio:SOIC-SL-14 -> tronixio:SOIC-14; Name MCP2221A-ISL -> MICROCHIP-MCP2221A-ISL

Commit message: Update
Parts:
- C301, C302, C303, C304, C305, C306, C307: footprint tronixio:CAPACITOR-1206 -> tronixio:CAPACITOR-SMD-1206
- LED301, LED302: footprint tronixio:LED-1206 -> tronixio:LED-SMD-1206
- R301, R302, R303, R304, R305, R306, R307, R308, R309, R310, R311, R312, R313, R314, R315, R316, R317, R318, R319, R320: footprint tronixio:RESISTOR-1206 -> tronixio:RESISTOR-SMD-1206

Commit message: Update
Parts:
- U301: footprint tronixio:SOT-23-6 -> tronixioZZZ:SC-70-6; symbol tronixio:ONSEMI-CAT4002A-SOT-23 -> tronixio:ONSEMI-CAT4002A-SC-70; Mouser 863-CAT4002ATD-GT3 -> 863-CAT4002ASD-GT3; Name ONSEMI-CAT4002A-SOT-23 -> ONSEMI-CAT4002A-SC-70
- U302: value MCP2221A-ISL -> MCP2221A
Changed lines of the file:
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@@
     (effects (font (size 1.2 1.2)) (justify left))
   )
-  (hierarchical_label "SCL" (shape input) (at 48.26 55.88 180)
+  (hierarchical_label "SCL" (shape bidirectional) (at 48.26 55.88 180)
     (effects (font (size 1.2 1.2)) (justify right))
   )
@@
     (effects (font (size 1.2 1.2)) (justify right))
   )
-  (hierarchical_label "SCL" (shape output) (at 238.76 58.42 0)
+  (hierarchical_label "SCL" (shape bidirectional) (at 238.76 58.42 0)
     (effects (font (size 1.2 1.2)) (justify left))
   )
@@
   (symbol (lib_id "tronixio:MICROCHIP-MCP2221A-ISL") (at 180.34 53.34 0) (unit 1)
     (in_bom yes) (on_board yes)
-    (property "Reference" "U302" (id 0) (at 190.5 49.53 0)
-      (effects (font (size 1.15 1.15)))
-    )
-    (property "Value" "MCP2221A-ISL" (id 1) (at 190.5 77.47 0)
-      (effects (font (size 1.15 1.15)))
+    (property "Reference" "U302" (id 0) (at 182.88 49.53 0)
+      (effects (font (size 1.15 1.15)) (justify left))
+    )
+    (property "Value" "MCP2221A" (id 1) (at 198.12 49.53 0)
+      (effects (font (size 1.15 1.15)) (justify right))
     )
     (property "Footprint" "tronixio:SOIC-14" (id 2) (at 190.5 83.82 0)
@@
     (pin "2")
   )
-  (symbol (lib_id "tronixio:ONSEMI-CAT4002A-SOT-23") (at 124.46 63.5 0) (unit 1)
+  (symbol (lib_id "tronixio:ONSEMI-CAT4002A-SC-70") (at 124.46 63.5 0) (unit 1)
     (in_bom yes) (on_board yes)
     (property "Reference" "U301" (id 0) (at 132.08 59.69 0)
@@
       (effects (font (size 1.15 1.15)))
     )
-    (property "Footprint" "tronixio:SOT-23-6" (id 2) (at 132.08 78.74 0)
+    (property "Footprint" "tronixioZZZ:SC-70-6" (id 2) (at 132.08 78.74 0)
       (effects (font (size 1 1)) hide)
     )
@@
       (effects (font (size 1 1)) hide)
     )
-    (property "Name" "ONSEMI-CAT4002A-SOT-23" (id 4) (at 132.08 76.2 0)
-      (effects (font (size 1 1)) hide)
-    )
-    (property "Mouser" "863-CAT4002ATD-GT3" (id 5) (at 132.08 83.82 0)
-      (effects (font (size 1 1)) hide)
-    )
+    (property "Name" "ONSEMI-CAT4002A-SC-70" (id 4) (at 132.08 76.2 0)
+      (effects (font (size 1 1)) hide)
+    )
+    (property "Mouser" "863-CAT4002ASD-GT3" (id 5) (at 132.08 83.82 0)
+      (effects (font (size 1 1)) hide)
+    )

Commit message: Update Mini
Parts:
- C301, C305, C307: symbol tronixio:CAPACITOR-1206-10N -> tronixio:KEMET-X7R-1206-10N-50V-20P; Name CAPACITOR-1206-10N -> (none)
- C302, C303, C304: symbol tronixio:CAPACITOR-1206-1U -> tronixio:KEMET-X7R-1206-1U-50V-20P; Mouser C1206C105M5RACTU -> 80-C1206C105M5R; Name CAPACITOR-1206-1U -> (none)
- C306: symbol tronixio:CAPACITOR-1206-100N -> tronixio:KEMET-X7R-1206-100N-50V-20P; Name CAPACITOR-1206-100N -> (none)
- JP301, JP302, JP303: Name HARWIN-254-M-1X02-JUMPER-VERTICAL -> (none)
- K301, K302: Name HARWIN-254-F-1X06-VERTICAL -> (none)
- LED301, LED302: Name KINGBRIGHT-LED-1206-BLUE -> (none)
- P301, P302: Name PIHER-PT10MV-10K -> (none)
- R301, R303, R304, R307, R310, R311, R312, R313, R314, R315, R316, R317: symbol tronixio:RESISTOR-1206-10K -> tronixio:KOASPEER-RK73B-1206-10K-5P; Name RESISTOR-1206-10K -> (none)
- R302, R305, R306, R309, R320: symbol tronixio:RESISTOR-1206-1K -> tronixio:KOASPEER-RK73B-1206-1K-5P; Name RESISTOR-1206-1K -> (none)
- R308: symbol tronixio:RESISTOR-1206-2K4 -> tronixio:KOASPEER-RK73B-1206-2K4-5P; Mouser 660-RK73B2BTTD242J -> 660-RK73B2BTTDD242J; Name RESISTOR-1206-2K4 -> (none)
- R318, R319: symbol tronixio:RESISTOR-1206-4K7 -> tronixio:KOASPEER-RK73B-1206-4K7-5P; Name RESISTOR-1206-4K7 -> (none)
- S301, S302: Name CK-KSA -> (none)
- S303: Name BOURNS-PEC12R-24DENTS-SWITCH -> (none)
- U301: footprint tronixioZZZ:SC-70-6 -> tronixio:SC-70-6; Name ONSEMI-CAT4002A-SC-70 -> (none)
- U302: Name MICROCHIP-MCP2221A-ISL -> (none)
Other:
- moved on the sheet: JP301, JP302, JP303

Commit message: Update Mini
Parts:
- C302, C303, C304: symbol tronixio:KEMET-X7R-1206-1U-50V-20P -> tronixio:KEMET-X7R-1206-1U-16V-20P; Mouser 80-C1206C105M5R -> 80-C1206C105M4R; Voltage 50V -> 16V
