File: Kicad/mini/pic8bit.kicad_sch (KiCad schematic)
At the start: 11 parts, among them K101 PE-450-4X6X-BLACK

Commit message: Update Mini
Parts:
- H101, H102, H103, H104: MOUSER 534-9055 -> (none); Mouser (none) -> 534-9055
- JP101, JP102, JP103, JP104, JP105, JP106: MOUSER 855-M7582 -> (none); Mouser (none) -> 855-M7582
- K101: MOUSER 450-476 -> (none); Mouser (none) -> 450-476
Changed lines of the file:
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@@
       (effects (font (size 1 1)) hide)
     )
-    (property "MOUSER" "855-M7582" (id 4) (at 261.62 182.88 0)
+    (property "Mouser" "855-M7582" (id 4) (at 261.62 182.88 0)
       (effects (font (size 1 1)) hide)
     )
@@
       (effects (font (size 1 1)) hide)
     )
-    (property "MOUSER" "855-M7582" (id 4) (at 251.46 182.88 0)
+    (property "Mouser" "855-M7582" (id 4) (at 251.46 182.88 0)
       (effects (font (size 1 1)) hide)
     )
@@
       (effects (font (size 1 1)) hide)
     )
-    (property "MOUSER" "450-476" (id 4) (at 251.46 177.8 0)
+    (property "Mouser" "450-476" (id 4) (at 251.46 177.8 0)
       (effects (font (size 1 1)) hide)
     )
@@
       (effects (font (size 1 1)) hide)
     )
-    (property "MOUSER" "855-M7582" (id 4) (at 276.86 182.88 0)
+    (property "Mouser" "855-M7582" (id 4) (at 276.86 182.88 0)
       (effects (font (size 1 1)) hide)
     )
@@
       (effects (font (size 1 1)) hide)
     )
-    (property "MOUSER" "534-9055" (id 4) (at 271.78 177.8 0)
+    (property "Mouser" "534-9055" (id 4) (at 271.78 177.8 0)
       (effects (font (size 1 1)) hide)
     )
@@
       (effects (font (size 1 1)) hide)
     )
-    (property "MOUSER" "855-M7582" (id 4) (at 256.54 182.88 0)
+    (property "Mouser" "855-M7582" (id 4) (at 256.54 182.88 0)
       (effects (font (size 1 1)) hide)
     )
@@
       (effects (font (size 1 1)) hide)
     )
-    (property "MOUSER" "534-9055" (id 4) (at 261.62 177.8 0)
+    (property "Mouser" "534-9055" (id 4) (at 261.62 177.8 0)
       (effects (font (size 1 1)) hide)
     )
@@
       (effects (font (size 1 1)) hide)
     )
-    (property "MOUSER" "855-M7582" (id 4) (at 271.78 182.88 0)
+    (property "Mouser" "855-M7582" (id 4) (at 271.78 182.88 0)
       (effects (font (size 1 1)) hide)
     )
@@
       (effects (font (size 1 1)) hide)
     )
-    (property "MOUSER" "855-M7582" (id 4) (at 266.7 182.88 0)
+    (property "Mouser" "855-M7582" (id 4) (at 266.7 182.88 0)
       (effects (font (size 1 1)) hide)
     )
@@
       (effects (font (size 1 1)) hide)
     )
-    (property "MOUSER" "534-9055" (id 4) (at 266.7 177.8 0)
+    (property "Mouser" "534-9055" (id 4) (at 266.7 177.8 0)
       (effects (font (size 1 1)) hide)
     )
@@
       (effects (font (size 1 1)) hide)
     )
-    (property "MOUSER" "534-9055" (id 4) (at 276.86 177.8 0)
+    (property "Mouser" "534-9055" (id 4) (at 276.86 177.8 0)
       (effects (font (size 1 1)) hide)
     )
@@
       (reference "IC202") (unit 1) (value "MICROCHIP-PIC16F1778-ISP") (footprint "tronixio:DIP-28-W762-SOCKET")
     )
-    (path "/8cdf8b92-b881-481d-a85a-c0055e9a856b/253151d6-cdc9-4c0d-9799-515e8cbda321"
-      (reference "IC301") (unit 1) (value "CAT4002A") (footprint "tronixio:SOT-23-6")
-    )
-    (path "/8cdf8b92-b881-481d-a85a-c0055e9a856b/20f9a251-d03b-4c79-a0b6-ede074b32619"
-      (reference "IC302") (unit 1) (value "MCP2221A") (footprint "tronixio:SOIC-SL-14")
+    (path "/8cdf8b92-b881-481d-a85a-c0055e9a856b/aaac6ca3-9aba-4f82-b45d-8eb04e78b4e9"
+      (reference "IC301") (unit 1) (value "ONSEMI-CAT4002A-SOT-23") (footprint "tronixio:SOT-23-6")
+    )
+    (path "/8cdf8b92-b881-481d-a85a-c0055e9a856b/62241e61-fae0-4fcf-92ee-1276a4ab7387"
+      (reference "IC302") (unit 1) (value "MICROCHIP-MCP2221A-ISL") (footprint "tronixio:SOIC-SL-14")
     )
     (path "/55795f44-b358-4de2-a286-91a0aa0ebc8a"
@@
     )
     (path "/8cdf8b92-b881-481d-a85a-c0055e9a856b/d8dfe39a-4c2d-4583-9a29-5f6578ad8af3"
-      (reference "K301") (unit 1) (value "HARWIN-254-F-1X08-VERTICAL") (footprint "tronixio:zzHARWIN-M20-782084x")
+      (reference "K301") (unit 1) (value "HARWIN-254-F-1X08-VERTICAL") (footprint "tronixio:HARWIN-M20-782084x")
     )
     (path "/8cdf8b92-b881-481d-a85a-c0055e9a856b/50151c1d-c91d-453c-a0af-92c029bb2229"
@@
     )
     (path "/8cdf8b92-b881-481d-a85a-c0055e9a856b/aebba99c-334c-4929-a5a1-891c48d14b31"
-      (reference "LED301") (unit 1) (value "URX") (footprint "tronixio:LED-1206")
+      (reference "LED301") (unit 1) (value "URX") (footprint "tronixio:FUSE-1206")
     )
     (path "/8cdf8b92-b881-481d-a85a-c0055e9a856b/8b71b4b0-c289-4468-a7ee-4a6409128d8d"
-      (reference "LED302") (unit 1) (value "UTX") (footprint "tronixio:LED-1206")
+      (reference "LED302") (unit 1) (value "UTX") (footprint "tronixio:FUSE-1206")
     )
     (path "/8cdf8b92-b881-481d-a85a-c0055e9a856b/f08bf669-a7e1-403b-a155-13b894bbc40b"

Commit message: Update
Changed lines of the file:
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@@
-      (effects (font (size 1.27 1.27)) (justify right))
-    )
-    (pin "SCL" input (at 124.46 96.52 0)
       (effects (font (size 1.27 1.27)) (justify right))
     )
@@
       (effects (font (size 1.27 1.27)) (justify right))
     )
-    (pin "URX" input (at 124.46 104.14 0)
-      (effects (font (size 1.27 1.27)) (justify right))
-    )
-    (pin "UTX" output (at 124.46 106.68 0)
+    (pin "SCL" output (at 124.46 96.52 0)
+      (effects (font (size 1.27 1.27)) (justify right))
+    )
+    (pin "URX" input (at 124.46 106.68 0)
+      (effects (font (size 1.27 1.27)) (justify right))
+    )
+    (pin "UTX" output (at 124.46 104.14 0)
       (effects (font (size 1.27 1.27)) (justify right))
     )
@@
       (effects (font (size 1.27 1.27)) (justify left))
     )
-    (pin "UTX" output (at 165.1 106.68 180)
-      (effects (font (size 1.27 1.27)) (justify left))
-    )
-    (pin "URX" input (at 165.1 104.14 180)
+    (pin "UTX" input (at 165.1 104.14 180)
+      (effects (font (size 1.27 1.27)) (justify left))
+    )
+    (pin "URX" output (at 165.1 106.68 180)
       (effects (font (size 1.27 1.27)) (justify left))
     )
@@
       (reference "#PWR0337") (unit 1) (value "POWER-GND") (footprint "")
     )
+    (path "/64edc06d-d6ae-4dac-9759-3f1fbed6457d/5e25d914-20d1-414a-a128-b79a39469e2d"
+      (reference "#PWR?") (unit 1) (value "POWER-GND") (footprint "")
+    )
     (path "/8cdf8b92-b881-481d-a85a-c0055e9a856b/36380bba-c7ac-4db6-bbd7-e4b4cc9c6541"
       (reference "BB301") (unit 1) (value "BREADBOARD-170") (footprint "tronixio:BREADBOARD-170")
@@
       (reference "TP202") (unit 1) (value "KEYSTONE-5006") (footprint "tronixio:KEYSTONE-5006")
     )
+    (path "/64edc06d-d6ae-4dac-9759-3f1fbed6457d/721ae374-0abc-463c-874b-568f793edc13"
+      (reference "TP203") (unit 1) (value "KEYSTONE-2000-3") (footprint "tronixio:KEYSTONE-2000-3")
+    )
   )

Commit message: Update
Other:
- title: Diagram -> Connections
