File: Kicad/mini/pic8bit.kicad_sch (KiCad schematic)
At the start: 11 parts, among them K101 PE-450-4X6X-BLACK

Commit message: Update
Changed lines of the file:
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@@
       (effects (font (size 1.27 1.27)) (justify left))
     )
-    (pin "SCL" input (at 165.1 96.52 180)
+    (pin "SCL" bidirectional (at 165.1 96.52 180)
       (effects (font (size 1.27 1.27)) (justify left))
     )
@@
     )
     (path "/8cdf8b92-b881-481d-a85a-c0055e9a856b/aaac6ca3-9aba-4f82-b45d-8eb04e78b4e9"
-      (reference "U301") (unit 1) (value "CAT4002A") (footprint "tronixio:SOT-23-6")
+      (reference "U301") (unit 1) (value "CAT4002A") (footprint "tronixioZZZ:SC-70-6")
     )
     (path "/8cdf8b92-b881-481d-a85a-c0055e9a856b/62241e61-fae0-4fcf-92ee-1276a4ab7387"
-      (reference "U302") (unit 1) (value "MCP2221A-ISL") (footprint "tronixio:SOIC-14")
+      (reference "U302") (unit 1) (value "MCP2221A") (footprint "tronixio:SOIC-14")
     )
   )
