File: Kicad/mini/pic8bit-mcu.kicad_sch (KiCad schematic)
At the start: 29 parts, among them IC201 TLV1117-33, IC202 MICROCHIP-PIC16F1778-ISP, K201 *Power & UART, K202 MCU 1, K203 MCU 1, K204 ICSP, K205 MCU 2, K206 MCU 2

Commit message: Update Mini
Connections:
- no-connect marks 2 -> 1
Changed lines of the file:
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@@
   )
   (no_connect (at 43.18 177.8))
-  (no_connect (at 147.32 125.73))
   (wire (pts (xy 190.5 78.74) (xy 190.5 123.19))
     (stroke (width 0) (type solid) (color 0 0 0 0))

Commit message: Update Mini
Parts:
- D201, D202: symbol tronixio:PMEG3030 -> tronixio:NEXPERIA-PMEG3030; MOUSER 771-PMEG3030EP115 -> (none); Mouser (none) -> 771-PMEG3030EP115; Name (none) -> PMEG3030
- F201: value F050 -> (none); footprint tronixio:FUSE-1206 -> (none); MOUSER 652-MF-NSMF050-2 -> (none); Mouser (none) -> 652-MF-NSMF050-2; Name (none) -> 500mA
- IC201: symbol tronixio:TLV1117-33-SOT -> tronixio:TI-TLV1117-33-SOT; MOUSER 595-TLV1117-33CDC -> (none); Mouser (none) -> 595-TLV1117-33CDC; Name (none) -> TLV1117-33
- IC202: MOUSER 579-PIC16F1778-I/SP -> (none); Mouser (none) -> 579-PIC16F1778-I/SP; Name PIC16F1778-ISP -> PIC16F/PIC18F
- JP201, JP203: MOUSER 855-M20-999024 -> (none); Mouser (none) -> 855-M20-999024
- JP202: value SCL -> (none); MOUSER 855-M20-999024 -> (none); Mouser (none) -> 855-M20-999024
- JP204: value SDA -> (none); MOUSER 855-M20-999024 -> (none); Mouser (none) -> 855-M20-999024
- K201: MOUSER 649-10118193-0001LF -> (none); Mouser (none) -> 649-10118193-0001LF
- K202, K205: MOUSER 855-M20-999144 -> (none); Mouser (none) -> 855-M20-999144
- K203, K206: MOUSER 855-M20-782144 -> (none); Mouser (none) -> 855-M20-782144
- K204: MOUSER 200-SSW10602TSRA -> (none); Mouser (none) -> 200-SSW10602TSRA
- LED201: MOUSER 604-APT3216LVBCD -> (none); Mouser (none) -> 604-APT3216LVBCD
- S201: value Reset -> (none); MOUSER 688-SKRPACE010 -> (none); Mouser (none) -> 688-SKRPACE010
- TP201, TP202: MOUSER 534-5006 -> (none); Mouser (none) -> 534-5006

Commit message: Update
Parts:
- added TP203: (no value), symbol tronixio:KEYSTONE-2000-3
- F201: value (none) -> F050; footprint (none) -> tronixio:FUSE-1206
- JP202: value (none) -> SCL
- JP204: value (none) -> SDA
- S201: value (none) -> Reset
Connections:
- net GND: now also TP203.1
Other:
- moved on the sheet: C203, LED201, R204, TP201, TP202

Commit message: Update Mini
Parts:
- TP203: value (none) -> KEYSTONE-2000-3; footprint (none) -> tronixio:KEYSTONE-2000-3
Changed lines of the file:
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@@
   (symbol (lib_id "tronixio:POWER-GND") (at 157.48 187.96 0) (unit 1)
     (in_bom yes) (on_board yes) (fields_autoplaced)
-    (property "Reference" "#PWR?" (id 0) (at 157.48 193.04 0)
+    (property "Reference" "#PWR0102" (id 0) (at 157.48 193.04 0)
       (effects (font (size 1 1)) hide)
     )
@@
       (effects (font (size 1.15 1.15)))
     )
-    (property "Value" "" (id 1) (at 160.02 161.2899 0)
+    (property "Value" "KEYSTONE-2000-3" (id 1) (at 160.02 161.2899 0)
       (effects (font (size 1.15 1.15)) (justify left) hide)
     )
-    (property "Footprint" "" (id 2) (at 157.48 170.18 0)
+    (property "Footprint" "tronixio:KEYSTONE-2000-3" (id 2) (at 157.48 170.18 0)
       (effects (font (size 1 1)) hide)
     )

Commit message: Update
Parts:
- IC202: Name PIC16F/PIC18F -> PIC16F1778-ISP
- K203, K206: footprint tronixio:zzHARWIN-M20-782144x -> tronixio:HARWIN-M20-782144x
Other:
- moved on the sheet: C204, C205, F201, JP203

Commit message: Up
Parts:
- U202: renamed from IC202; footprint tronixio:DIP-28-W762-SOCKET -> tronixio:DIP-28-W762
- renumbered IC201 to U201
Changed lines of the file:
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@@
   (symbol (lib_id "tronixio:TI-TLV1117-33-SOT") (at 93.98 170.18 0) (unit 1)
     (in_bom yes) (on_board yes)
-    (property "Reference" "IC201" (id 0) (at 93.98 163.83 0)
+    (property "Reference" "U201" (id 0) (at 93.98 163.83 0)
       (effects (font (size 1.15 1.15)))
     )
@@
   (symbol (lib_id "tronixio:MICROCHIP-PIC16F1778-ISP") (at 144.78 72.39 0) (unit 1)
     (in_bom yes) (on_board yes)
-    (property "Reference" "IC202" (id 0) (at 132.08 52.07 0)
+    (property "Reference" "U202" (id 0) (at 132.08 52.07 0)
       (effects (font (size 1.15 1.15)) (justify left))
     )
@@
       (effects (font (size 1 1)) hide)
     )
-    (property "Footprint" "tronixio:DIP-28-W762-SOCKET" (id 2) (at 144.78 95.25 0)
-      (effects (font (size 1 1)) hide)
-    )
+    (property "Footprint" "tronixio:DIP-28-W762" (id 2) (at 144.78 95.25 0)
+      (effects (font (size 1 1)) hide)
+    )

Commit message: Up
Parts:
- U202: Name PIC16F1778-ISP -> PIC16F/PIC18F
Changed lines of the file:
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@@
       (effects (font (size 1 1)) hide)
     )
-    (property "Name" "PIC16F1778-ISP" (id 5) (at 157.48 52.07 0)
+    (property "Name" "PIC16F/PIC18F" (id 5) (at 157.48 52.07 0)
       (effects (font (size 1.15 1.15)) (justify right))
     )

Commit message: Update
Parts:
- C201, C203: value 10µ -> KEMET-C322-10U-508; footprint tronixio:CAPACITOR-1206 -> tronixio:KEMET-C322; symbol tronixio:C-0805 -> tronixio:KEMET-C322-10U-508; Mouser (none) -> 80-C322C106K3R; Name (none) -> KEMET-C32210U-508; Tolerance (none) -> 10%
- C202, C205: symbol tronixio:C-0805 -> tronixio:CAPACITOR-1206-100N; Mouser (none) -> 80-C1206C104M5R; Name (none) -> CAPACITOR-1206-100N; Tolerance (none) -> 20%; Voltage (none) -> 50V
- C204: symbol tronixio:KEMET-C322 -> tronixio:KEMET-C322-10U-508; Mouser (none) -> 80-C322C106K3R; Name (none) -> KEMET-C32210U-508; Tolerance (none) -> 10%
- D201, D202: Name PMEG3030 -> NEXPERIA-PMEG3030
- F201: value F050 -> 500mA; footprint tronixio:FUSE-1206 -> tronixio:FUSE-0805; Name 500mA -> BOURNS-FUSE-MF-NSMF050
- JP201: Name (none) -> HARWIN-254-M-1X02-JUMPER-VERTICAL
- K201: Name (none) -> FCI-USB-TYPE-B-MICRO-THT
- K202: Name (none) -> HARWIN-254-M-1X14-VERTICAL
- K203: value MCU 1 -> MCU 2; Name (none) -> HARWIN-254-F-1X14-VERTICAL
- K204: Name ICSP -> MICROCHIP-ICSP-F-1X06
- K205: value MCU 2 -> MCU 1; Name (none) -> HARWIN-254-M-1X14-VERTICAL
- K206: Name (none) -> HARWIN-254-F-1X14-VERTICAL
- LED201: symbol tronixio:LED-1206-BLUE -> tronixio:KINGBRIGHT-LED-1206-BLUE; Name (none) -> KINGBRIGHT-LED-1206-BLUE
- R201: symbol tronixio:R-0805 -> tronixio:RESISTOR-1206-10K; Mouser (none) -> 660-RK73B2BTTDD103J; Name (none) -> RESISTOR-1206-10K; Tolerance (none) -> 5%
- R202: symbol tronixio:R-0805 -> tronixio:RESISTOR-1206-1K; Mouser (none) -> 660-RK73B2BTTDD102J; Name (none) -> RESISTOR-1206-1K; Tolerance (none) -> 5%
- R203, R204, R205: symbol tronixio:R-0805 -> tronixio:RESISTOR-1206-4K7; Mouser (none) -> 660-RK73B2BTTDD472J; Name (none) -> RESISTOR-1206-4K7; Tolerance (none) -> 5%
- S201: Name (none) -> ALPS-SKRPAC
- TP201, TP202: Name (none) -> KEYSTONE-5006
- TP203: Name (none) -> KEYSTONE-2000-3
- U201: Name TLV1117-33 -> TI-TLV1117-33-SOT
