File: Kicad/mini/pic8bit-mcu.kicad_sch (KiCad schematic)
At the start: 30 parts, among them K201 *Power & UART, K202 MCU 1, K203 MCU 2, K204 ICSP, K205 MCU 1, K206 MCU 2, U201 TLV1117-33, U202 MICROCHIP-PIC16F1778-ISP

Commit message: Update
Parts:
- JP201: value *Power IN -> HARWIN-254-M-1X02-JUMPER-VERTICAL
- JP202, JP203, JP204: Name (none) -> HARWIN-254-M-1X02-JUMPER-VERTICAL
Changed lines of the file:
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@@
       (effects (font (size 1.15 1.15)) (justify left))
     )
-    (property "Footprint" "tronixio:HARWIN-M20-999024x" (id 2) (at 119.38 107.95 0)
-      (effects (font (size 1 1)) hide)
-    )
-    (property "Datasheet" "https://www.harwin.com/products/M20-9990846/" (id 3) (at 119.38 110.49 0)
-      (effects (font (size 1 1)) hide)
-    )
-    (property "Mouser" "855-M20-999024" (id 4) (at 119.38 113.03 0)
+    (property "Footprint" "tronixio:HARWIN-M20-999024x" (id 2) (at 119.38 110.49 0)
+      (effects (font (size 1 1)) hide)
+    )
+    (property "Datasheet" "https://www.harwin.com/products/M20-9990846/" (id 3) (at 119.38 113.03 0)
+      (effects (font (size 1 1)) hide)
+    )
+    (property "Mouser" "855-M20-999024" (id 4) (at 119.38 115.57 0)
+      (effects (font (size 1 1)) hide)
+    )
+    (property "Name" "HARWIN-254-M-1X02-JUMPER-VERTICAL" (id 5) (at 119.38 107.95 0)
       (effects (font (size 1 1)) hide)
     )
@@
     (pin "1")
   )
-  (symbol (lib_name "HARWIN-254-M-1X02-JUMPER-VERTICAL_1") (lib_id "tronixio:HARWIN-254-M-1X02-JUMPER-VERTICAL") (at 58.42 180.34 0) (mirror y) (unit 1)
+  (symbol (lib_id "tronixio:HARWIN-254-M-1X02-JUMPER-VERTICAL") (at 58.42 180.34 0) (mirror y) (unit 1)
     (in_bom yes) (on_board yes)
     (property "Reference" "JP201" (id 0) (at 57.785 177.8 0)
       (effects (font (size 1.15 1.15)) (justify left))
     )
-    (property "Value" "*Power IN" (id 1) (at 57.785 185.42 0)
+    (property "Value" "HARWIN-254-M-1X02-JUMPER-VERTICAL" (id 1) (at 55.88 182.88 0)
       (effects (font (size 1.15 1.15)) (justify left))
     )
@@
     (pin "1")
   )
-  (symbol (lib_id "tronixio:HARWIN-254-M-1X02-JUMPER-VERTICAL") (at 180.34 45.72 0) (mirror y) (unit 1)
+  (symbol (lib_name "HARWIN-254-M-1X02-JUMPER-VERTICAL_3") (lib_id "tronixio:HARWIN-254-M-1X02-JUMPER-VERTICAL") (at 180.34 45.72 0) (mirror y) (unit 1)
     (in_bom yes) (on_board yes)
     (property "Reference" "JP204" (id 0) (at 180.975 43.18 0)
@@
       (effects (font (size 1.15 1.15)) (justify right))
     )
-    (property "Footprint" "tronixio:HARWIN-M20-999024x" (id 2) (at 180.34 58.42 0)
-      (effects (font (size 1 1)) hide)
-    )
-    (property "Datasheet" "https://www.harwin.com/products/M20-9990846/" (id 3) (at 180.34 60.96 0)
-      (effects (font (size 1 1)) hide)
-    )
-    (property "Mouser" "855-M20-999024" (id 4) (at 180.34 63.5 0)
+    (property "Footprint" "tronixio:HARWIN-M20-999024x" (id 2) (at 180.34 60.96 0)
+      (effects (font (size 1 1)) hide)
+    )
+    (property "Datasheet" "https://www.harwin.com/products/M20-9990846/" (id 3) (at 180.34 63.5 0)
+      (effects (font (size 1 1)) hide)
+    )
+    (property "Mouser" "855-M20-999024" (id 4) (at 180.34 66.04 0)
+      (effects (font (size 1 1)) hide)
+    )
+    (property "Name" "HARWIN-254-M-1X02-JUMPER-VERTICAL" (id 5) (at 180.34 58.42 0)
       (effects (font (size 1 1)) hide)
     )
@@
       (effects (font (size 1.15 1.15)) (justify left))
     )
-    (property "Footprint" "tronixio:HARWIN-M20-999024x" (id 2) (at 109.22 58.42 0)
-      (effects (font (size 1 1)) hide)
-    )
-    (property "Datasheet" "https://www.harwin.com/products/M20-9990846/" (id 3) (at 109.22 60.96 0)
-      (effects (font (size 1 1)) hide)
-    )
-    (property "Mouser" "855-M20-999024" (id 4) (at 109.22 63.5 0)
-      (effects (font (size 1 1)) hide)
-    )
+    (property "Footprint" "tronixio:HARWIN-M20-999024x" (id 2) (at 109.22 60.96 0)
+      (effects (font (size 1 1)) hide)
+    )
+    (property "Datasheet" "https://www.harwin.com/products/M20-9990846/" (id 3) (at 109.22 63.5 0)
+      (effects (font (size 1 1)) hide)
+    )
+    (property "Mouser" "855-M20-999024" (id 4) (at 109.22 66.04 0)
+      (effects (font (size 1 1)) hide)
+    )
+    (property "Name" "HARWIN-254-M-1X02-JUMPER-VERTICAL" (id 5) (at 109.22 58.42 0)
+      (effects (font (size 1 1)) hide)
+    )

Commit message: Update
Parts:
- C201, C203: value KEMET-C322-10U-508 -> 10µ; footprint tronixio:KEMET-C322 -> tronixio:CAPACITOR-1206; symbol tronixio:KEMET-C322-10U-508 -> tronixio:CAPACITOR-1206-10U; Mouser 80-C322C106K3R -> 80-C1206C106M3R; Name KEMET-C32210U-508 -> CAPACITOR-1206-10U; Tolerance 10% -> 20%; Voltage (none) -> 25V
- JP201: value HARWIN-254-M-1X02-JUMPER-VERTICAL -> Power IN
- U202: value MICROCHIP-PIC16F1778-ISP -> PIC16F/PIC18F; Name PIC16F/PIC18F -> MICROCHIP-PIC16F1778-ISP
Changed lines of the file:
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@@
     (pin "1")
   )
-  (symbol (lib_id "tronixio:KEMET-C322-10U-508") (at 81.28 180.34 0) (unit 1)
+  (symbol (lib_id "tronixio:CAPACITOR-1206-10U") (at 81.28 180.34 0) (unit 1)
     (in_bom yes) (on_board yes)
     (property "Reference" "C201" (id 0) (at 80.645 177.8 0)
       (effects (font (size 1.15 1.15)) (justify right))
     )
-    (property "Value" "KEMET-C322-10U-508" (id 1) (at 81.915 182.88 0)
-      (effects (font (size 1.15 1.15)) (justify left))
-    )
-    (property "Footprint" "tronixio:KEMET-C322" (id 2) (at 81.28 195.58 0)
-      (effects (font (size 1 1)) hide)
-    )
-    (property "Datasheet" "https://content.kemet.com/datasheets/KEM_C1054_HIVOLT_GOLDMAX_300_C0G.pdf" (id 3) (at 81.28 193.04 0)
-      (effects (font (size 1 1)) hide)
-    )
-    (property "Tolerance" "10%" (id 4) (at 81.915 185.42 0)
-      (effects (font (size 1.15 1.15)) (justify left) hide)
-    )
-    (property "Mouser" "80-C322C106K3R" (id 5) (at 81.28 198.12 0)
-      (effects (font (size 1 1)) hide)
-    )
-    (property "Name" "KEMET-C32210U-508" (id 6) (at 81.28 190.5 0)
-      (effects (font (size 1 1)) hide)
+    (property "Value" "10µ" (id 1) (at 80.645 182.88 0)
+      (effects (font (size 1.15 1.15)) (justify right))
+    )
+    (property "Footprint" "tronixio:CAPACITOR-1206" (id 2) (at 81.28 193.04 0)
+      (effects (font (size 1 1)) hide)
+    )
+    (property "Datasheet" "https://content.kemet.com/datasheets/KEM_C1090_X7R_ESD.pdf" (id 3) (at 81.28 195.58 0)
+      (effects (font (size 1 1)) hide)
+    )
+    (property "Tolerance" "20%" (id 4) (at 81.915 186.69 0)
+      (effects (font (size 1.15 1.15)) (justify left) hide)
+    )
+    (property "Mouser" "80-C1206C106M3R" (id 5) (at 81.28 198.12 0)
+      (effects (font (size 1 1)) hide)
+    )
+    (property "Name" "CAPACITOR-1206-10U" (id 6) (at 81.28 190.5 0)
+      (effects (font (size 1 1)) hide)
+    )
+    (property "Voltage" "25V" (id 7) (at 81.915 184.785 0)
+      (effects (font (size 1.15 1.15)) (justify left) hide)
     )
     (pin "1")
@@
       (effects (font (size 1.15 1.15)) (justify left))
     )
-    (property "Value" "HARWIN-254-M-1X02-JUMPER-VERTICAL" (id 1) (at 55.88 182.88 0)
+    (property "Value" "Power IN" (id 1) (at 57.785 185.42 0)
       (effects (font (size 1.15 1.15)) (justify left))
     )
@@
     (pin "2")
   )
-  (symbol (lib_id "tronixio:KEMET-C322-10U-508") (at 106.68 180.34 0) (unit 1)
+  (symbol (lib_id "tronixio:CAPACITOR-1206-10U") (at 106.68 180.34 0) (unit 1)
     (in_bom yes) (on_board yes)
     (property "Reference" "C203" (id 0) (at 107.315 177.8 0)
       (effects (font (size 1.15 1.15)) (justify left))
     )
-    (property "Value" "KEMET-C322-10U-508" (id 1) (at 107.315 182.88 0)
-      (effects (font (size 1.15 1.15)) (justify left))
-    )
-    (property "Footprint" "tronixio:KEMET-C322" (id 2) (at 106.68 195.58 0)
-      (effects (font (size 1 1)) hide)
-    )
-    (property "Datasheet" "https://content.kemet.com/datasheets/KEM_C1054_HIVOLT_GOLDMAX_300_C0G.pdf" (id 3) (at 106.68 193.04 0)
-      (effects (font (size 1 1)) hide)
-    )
-    (property "Tolerance" "10%" (id 4) (at 107.315 185.42 0)
-      (effects (font (size 1.15 1.15)) (justify left) hide)
-    )
-    (property "Mouser" "80-C322C106K3R" (id 5) (at 106.68 198.12 0)
-      (effects (font (size 1 1)) hide)
-    )
-    (property "Name" "KEMET-C32210U-508" (id 6) (at 106.68 190.5 0)
-      (effects (font (size 1 1)) hide)
+    (property "Value" "10µ" (id 1) (at 107.315 182.88 0)
+      (effects (font (size 1.15 1.15)) (justify left))
+    )
+    (property "Footprint" "tronixio:CAPACITOR-1206" (id 2) (at 106.68 193.04 0)
+      (effects (font (size 1 1)) hide)
+    )
+    (property "Datasheet" "https://content.kemet.com/datasheets/KEM_C1090_X7R_ESD.pdf" (id 3) (at 106.68 195.58 0)
+      (effects (font (size 1 1)) hide)
+    )
+    (property "Tolerance" "20%" (id 4) (at 107.315 186.69 0)
+      (effects (font (size 1.15 1.15)) (justify left) hide)
+    )
+    (property "Mouser" "80-C1206C106M3R" (id 5) (at 106.68 198.12 0)
+      (effects (font (size 1 1)) hide)
+    )
+    (property "Name" "CAPACITOR-1206-10U" (id 6) (at 106.68 190.5 0)
+      (effects (font (size 1 1)) hide)
+    )
+    (property "Voltage" "25V" (id 7) (at 107.315 184.785 0)
+      (effects (font (size 1.15 1.15)) (justify left) hide)
     )
     (pin "1")
@@
   (symbol (lib_id "tronixio:POWER-FLAG") (at 177.8 190.5 180) (unit 1)
     (in_bom yes) (on_board yes) (fields_autoplaced)
-    (property "Reference" "#FLG?" (id 0) (at 177.8 188.595 0)
+    (property "Reference" "#FLG0101" (id 0) (at 177.8 188.595 0)
       (effects (font (size 1.27 1.27)) hide)
     )
@@
     (pin "2")
   )
-  (symbol (lib_id "tronixio:MICROCHIP-PIC16F1778-ISP") (at 144.78 72.39 0) (unit 1)
+  (symbol (lib_id "tronixio:MICROCHIP-PIC16F1778-ISP") (at 129.54 55.88 0) (unit 1)
     (in_bom yes) (on_board yes)
     (property "Reference" "U202" (id 0) (at 132.08 52.07 0)
       (effects (font (size 1.15 1.15)) (justify left))
     )
-    (property "Value" "MICROCHIP-PIC16F1778-ISP" (id 1) (at 144.78 92.71 0)
-      (effects (font (size 1 1)) hide)
-    )
-    (property "Footprint" "tronixio:DIP-28-W762" (id 2) (at 144.78 95.25 0)
-      (effects (font (size 1 1)) hide)
-    )
-    (property "Datasheet" "https://www.microchip.com/en-us/product/PIC16F1778" (id 3) (at 144.78 97.79 0)
-      (effects (font (size 1 1)) hide)
-    )
-    (property "Name" "PIC16F/PIC18F" (id 5) (at 157.48 52.07 0)
+    (property "Value" "PIC16F/PIC18F" (id 1) (at 157.48 52.07 0)
       (effects (font (size 1.15 1.15)) (justify right))
     )
-    (property "Mouser" "579-PIC16F1778-I/SP" (id 6) (at 144.78 100.33 0)
-      (effects (font (size 1 1)) hide)
-    )
+    (property "Footprint" "tronixio:DIP-28-W762" (id 2) (at 144.78 96.52 0)
+      (effects (font (size 1 1)) hide)
+    )
+    (property "Datasheet" "https://www.microchip.com/en-us/product/PIC16F1778" (id 3) (at 144.78 99.06 0)
+      (effects (font (size 1 1)) hide)
+    )
+    (property "Name" "MICROCHIP-PIC16F1778-ISP" (id 5) (at 144.78 52.07 0)
+      (effects (font (size 1 1)) hide)
+    )
+    (property "Mouser" "579-PIC16F1778-I/SP" (id 6) (at 144.78 101.6 0)
+      (effects (font (size 1 1)) hide)
+    )

Commit message: Update
Parts:
- K203: value MCU 2 -> MCU 1
- K205: value MCU 1 -> MCU 2
- U201: symbol tronixio:TI-TLV1117-33-SOT -> tronixio:TI-TLV1117-33-SOT-223; Name TI-TLV1117-33-SOT -> TI-TLV1117-33-SOT-223
- U202: footprint tronixio:DIP-28-W762 -> tronixio:DIP-28-W762-SOCKET

Commit message: Update
Parts:
- F201: footprint tronixio:FUSE-0805 -> tronixio:FUSE-1206
Changed lines of the file:
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@@
       (effects (font (size 1.15 1.15)))
     )
-    (property "Footprint" "tronixio:FUSE-0805" (id 2) (at 55.88 177.8 0)
+    (property "Footprint" "tronixio:FUSE-1206" (id 2) (at 55.88 177.8 0)
       (effects (font (size 1 1)) hide)
     )

Commit message: Update
Other:
- note added: "U202: Check the pinout for the desired MCU family"
- note removed: "IC202: Check the pinout for the desired MCU family"
Changed lines of the file:
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@@
     (effects (font (size 1.15 1.15)) (justify left bottom))
   )
-  (text "IC202: Check the pinout for the desired MCU family"
-    (at 180.34 173.99 0)
+  (text "U202: Check the pinout for the desired MCU family" (at 180.34 173.99 0)
     (effects (font (size 1.27 1.27)) (justify left bottom))
   )

Commit message: Update
Parts:
- C201, C202, C203, C205: footprint tronixio:CAPACITOR-1206 -> tronixio:CAPACITOR-SMD-1206
- F201: footprint tronixio:FUSE-1206 -> tronixio:FUSE-SMD-1206
- LED201: footprint tronixio:LED-1206 -> tronixio:LED-SMD-1206
- R201, R202, R203, R204, R205: footprint tronixio:RESISTOR-1206 -> tronixio:RESISTOR-SMD-1206
- U202: footprint tronixio:DIP-28-W762-SOCKET -> tronixio:DIP-28-W762
Changed lines of the file:
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@@
     (pin "1")
   )
-  (symbol (lib_id "tronixio:CAPACITOR-1206-10U") (at 81.28 180.34 0) (unit 1)
+  (symbol (lib_name "CAPACITOR-1206-10U_1") (lib_id "tronixio:CAPACITOR-1206-10U") (at 81.28 180.34 0) (unit 1)
     (in_bom yes) (on_board yes)
     (property "Reference" "C201" (id 0) (at 80.645 177.8 0)
@@
       (effects (font (size 1.15 1.15)) (justify right))
     )
-    (property "Footprint" "tronixio:CAPACITOR-1206" (id 2) (at 81.28 193.04 0)
+    (property "Footprint" "tronixio:CAPACITOR-SMD-1206" (id 2) (at 81.28 193.04 0)
       (effects (font (size 1 1)) hide)
     )
@@
     (pin "1")
   )
-  (symbol (lib_id "tronixio:CAPACITOR-1206-100N") (at 170.18 100.33 0) (unit 1)
+  (symbol (lib_name "CAPACITOR-1206-100N_1") (lib_id "tronixio:CAPACITOR-1206-100N") (at 170.18 100.33 0) (unit 1)
     (in_bom yes) (on_board yes)
     (property "Reference" "C205" (id 0) (at 170.815 97.79 0)
@@
       (effects (font (size 1.15 1.15)) (justify left))
     )
-    (property "Footprint" "tronixio:CAPACITOR-1206" (id 2) (at 170.18 113.03 0)
+    (property "Footprint" "tronixio:CAPACITOR-SMD-1206" (id 2) (at 170.18 113.03 0)
       (effects (font (size 1 1)) hide)
     )
@@
       (effects (font (size 1.15 1.15)) (justify left))
     )
-    (property "Footprint" "tronixio:CAPACITOR-1206" (id 2) (at 106.68 193.04 0)
+    (property "Footprint" "tronixio:CAPACITOR-SMD-1206" (id 2) (at 106.68 193.04 0)
       (effects (font (size 1 1)) hide)
     )
@@
     )
     (property "Footprint" "" (id 2) (at 177.8 190.5 0)
-      (effects (font (size 1.27 1.27)) hide)
-    )
-    (property "Datasheet" "~" (id 3) (at 177.8 190.5 0)
-      (effects (font (size 1.27 1.27)) hide)
+      (effects (font (size 1 1)) hide)
+    )
+    (property "Datasheet" "" (id 3) (at 177.8 190.5 0)
+      (effects (font (size 1 1)) hide)
     )
     (pin "1")
@@
       (effects (font (size 1.15 1.15)))
     )
-    (property "Footprint" "tronixio:RESISTOR-1206" (id 2) (at 76.2 38.1 0)
-      (effects (font (size 1 1)) hide)
-    )
-    (property "Datasheet" "https://www.koaspeer.com/pdfs/RK73B.pdf" (id 3) (at 73.66 38.1 0)
+    (property "Footprint" "tronixio:RESISTOR-SMD-1206" (id 2) (at 76.2 38.1 0)
+      (effects (font (size 1 1)) hide)
+    )
+    (property "Datasheet" "https://www.koaspeer.com/products/resistors/general-purpose/rk73b/" (id 3) (at 73.66 38.1 0)
       (effects (font (size 1 1)) hide)
     )
@@
     (pin "2")
   )
-  (symbol (lib_id "tronixio:RESISTOR-1206-4K7") (at 109.22 35.56 0) (unit 1)
+  (symbol (lib_name "RESISTOR-1206-4K7_2") (lib_id "tronixio:RESISTOR-1206-4K7") (at 109.22 35.56 0) (unit 1)
     (in_bom yes) (on_board yes)
     (property "Reference" "R203" (id 0) (at 108.585 31.75 0)
@@
       (effects (font (size 1.15 1.15)))
     )
-    (property "Footprint" "tronixio:RESISTOR-1206" (id 2) (at 109.22 50.8 0)
-      (effects (font (size 1 1)) hide)
-    )
-    (property "Datasheet" "https://www.koaspeer.com/pdfs/RK73B.pdf" (id 3) (at 109.22 53.34 0)
+    (property "Footprint" "tronixio:RESISTOR-SMD-1206" (id 2) (at 109.22 50.8 0)
+      (effects (font (size 1 1)) hide)
+    )
+    (property "Datasheet" "https://www.koaspeer.com/products/resistors/general-purpose/rk73b/" (id 3) (at 109.22 53.34 0)
       (effects (font (size 1 1)) hide)
     )
@@
       (effects (font (size 1.15 1.15)) (justify left))
     )
-    (property "Footprint" "tronixio:CAPACITOR-1206" (id 2) (at 83.82 55.88 0)
+    (property "Footprint" "tronixio:CAPACITOR-SMD-1206" (id 2) (at 83.82 55.88 0)
       (effects (font (size 1 1)) hide)
     )
@@
     (pin "2")
   )
-  (symbol (lib_id "tronixio:RESISTOR-1206-4K7") (at 180.34 35.56 0) (unit 1)
+  (symbol (lib_name "RESISTOR-1206-4K7_1") (lib_id "tronixio:RESISTOR-1206-4K7") (at 180.34 35.56 0) (unit 1)
     (in_bom yes) (on_board yes)
     (property "Reference" "R205" (id 0) (at 180.975 31.75 0)
@@
       (effects (font (size 1.15 1.15)))
     )
-    (property "Footprint" "tronixio:RESISTOR-1206" (id 2) (at 180.34 50.8 0)
-      (effects (font (size 1 1)) hide)
-    )
-    (property "Datasheet" "https://www.koaspeer.com/pdfs/RK73B.pdf" (id 3) (at 180.34 53.34 0)
+    (property "Footprint" "tronixio:RESISTOR-SMD-1206" (id 2) (at 180.34 50.8 0)
+      (effects (font (size 1 1)) hide)
+    )
+    (property "Datasheet" "https://www.koaspeer.com/products/resistors/general-purpose/rk73b/" (id 3) (at 180.34 53.34 0)
       (effects (font (size 1 1)) hide)
     )
@@
       (effects (font (size 1.15 1.15)))
     )
-    (property "Footprint" "tronixio:FUSE-1206" (id 2) (at 55.88 177.8 0)
+    (property "Footprint" "tronixio:FUSE-SMD-1206" (id 2) (at 55.88 177.8 0)
       (effects (font (size 1 1)) hide)
     )
@@
       (effects (font (size 1.15 1.15)))
     )
-    (property "Footprint" "tronixio:RESISTOR-1206" (id 2) (at 76.2 48.26 0)
-      (effects (font (size 1 1)) hide)
-    )
-    (property "Datasheet" "https://www.koaspeer.com/pdfs/RK73B.pdf" (id 3) (at 76.2 50.8 0)
+    (property "Footprint" "tronixio:RESISTOR-SMD-1206" (id 2) (at 76.2 48.26 0)
+      (effects (font (size 1 1)) hide)
+    )
+    (property "Datasheet" "https://www.koaspeer.com/products/resistors/general-purpose/rk73b/" (id 3) (at 76.2 50.8 0)
       (effects (font (size 1 1)) hide)
     )
@@
       (effects (font (size 1.15 1.15)) (justify right))
     )
-    (property "Footprint" "tronixio:DIP-28-W762-SOCKET" (id 2) (at 129.54 99.06 0)
-      (effects (font (size 1 1)) hide)
-    )
-    (property "Datasheet" "https://www.microchip.com/en-us/product/PIC16F1778" (id 3) (at 129.54 101.6 0)
-      (effects (font (size 1 1)) hide)
-    )
-    (property "Name" "MICROCHIP-PIC16F1778-ISP" (id 5) (at 129.54 96.52 0)
-      (effects (font (size 1 1)) hide)
-    )
-    (property "Mouser" "579-PIC16F1778-I/SP" (id 6) (at 129.54 104.14 0)
+    (property "Footprint" "tronixio:DIP-28-W762" (id 2) (at 144.78 99.06 0)
+      (effects (font (size 1 1)) hide)
+    )
+    (property "Datasheet" "https://www.microchip.com/en-us/product/PIC16F1778" (id 3) (at 144.78 101.6 0)
+      (effects (font (size 1 1)) hide)
+    )
+    (property "Name" "MICROCHIP-PIC16F1778-ISP" (id 5) (at 144.78 96.52 0)
+      (effects (font (size 1 1)) hide)
+    )
+    (property "Mouser" "579-PIC16F1778-I/SP" (id 6) (at 144.78 104.14 0)
       (effects (font (size 1 1)) hide)
     )
@@
       (effects (font (size 1.15 1.15)))
     )
-    (property "Footprint" "tronixio:RESISTOR-1206" (id 2) (at 121.92 185.42 0)
-      (effects (font (size 1 1)) hide)
-    )
-    (property "Datasheet" "https://www.koaspeer.com/pdfs/RK73B.pdf" (id 3) (at 121.92 187.96 0)
+    (property "Footprint" "tronixio:RESISTOR-SMD-1206" (id 2) (at 121.92 185.42 0)
+      (effects (font (size 1 1)) hide)
+    )
+    (property "Datasheet" "https://www.koaspeer.com/products/resistors/general-purpose/rk73b/" (id 3) (at 121.92 187.96 0)
       (effects (font (size 1 1)) hide)
     )
@@
       (effects (font (size 1.15 1.15)) (justify left))
     )
-    (property "Footprint" "tronixio:LED-1206" (id 2) (at 111.76 180.34 0)
-      (effects (font (size 1 1)) hide)
-    )
+    (property "Footprint" "tronixio:LED-SMD-1206" (id 2) (at 111.76 180.34 0)
+      (effects (font (size 1 1)) hide)
+    )

Commit message: Update
Other:
- note added: "*"
- note added: "*Power & UART OR Power IN"
- note added: "*U202: Check the pinout for the desired MCU family"
- note removed: "Power & UART OR Power IN"
- note removed: "U202: Check the pinout for the desired MCU family"
Changed lines of the file:
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@@
     (effects (font (size 1.15 1.15)) (justify left bottom))
   )
-  (text "U202: Check the pinout for the desired MCU family" (at 180.34 173.99 0)
+  (text "*U202: Check the pinout for the desired MCU family"
+    (at 180.34 173.99 0)
     (effects (font (size 1.27 1.27)) (justify left bottom))
   )
@@
     (effects (font (size 1.15 1.15)) (justify right bottom))
   )
-  (text "Power & UART OR Power IN" (at 180.34 171.45 0)
+  (text "*Power & UART OR Power IN" (at 180.34 171.45 0)
     (effects (font (size 1.27 1.27)) (justify left bottom))
   )
@@
   )
   (text "RB4" (at 223.52 109.22 0)
+    (effects (font (size 1.15 1.15)) (justify left bottom))
+  )
+  (text "*" (at 132.08 53.34 0)
     (effects (font (size 1.15 1.15)) (justify left bottom))
   )
@@
   (symbol (lib_id "tronixio:MICROCHIP-PIC16F1778-ISP") (at 129.54 55.88 0) (unit 1)
     (in_bom yes) (on_board yes)
-    (property "Reference" "U202" (id 0) (at 132.08 52.07 0)
-      (effects (font (size 1.15 1.15)) (justify left))
-    )
+    (property "Reference" "U202" (id 0) (at 133.35 52.07 0)
+      (effects (font (size 1.15 1.15)) (justify left))
+    )

Commit message: Update Mini
Parts:
- C201, C203: symbol tronixio:CAPACITOR-1206-10U -> tronixio:KEMET-X5R-1206-10U-25V-20P; Mouser 80-C1206C106M3R -> 80-C1206C106M3P; Name CAPACITOR-1206-10U -> (none)
- C202, C205: symbol tronixio:CAPACITOR-1206-100N -> tronixio:KEMET-X7R-1206-100N-50V-20P; Name CAPACITOR-1206-100N -> (none)
- C204: symbol tronixio:KEMET-C322-10U-508 -> tronixio:KEMET-C322-0508-10U-25V-10P; Name KEMET-C32210U-508 -> (none); Voltage (none) -> 25V
- D201, D202: Name NEXPERIA-PMEG3030 -> (none)
- F201: Name BOURNS-FUSE-MF-NSMF050 -> (none)
- JP201, JP202, JP203, JP204: Name HARWIN-254-M-1X02-JUMPER-VERTICAL -> (none)
- K201: Name FCI-USB-TYPE-B-MICRO-THT -> (none)
- K202, K205: Name HARWIN-254-M-1X14-VERTICAL -> (none)
- K203, K206: Name HARWIN-254-F-1X14-VERTICAL -> (none)
- K204: Name MICROCHIP-ICSP-F-1X06 -> (none)
- LED201: Name KINGBRIGHT-LED-1206-BLUE -> (none)
- R201: symbol tronixio:RESISTOR-1206-10K -> tronixio:KOASPEER-RK73B-1206-10K-5P; Name RESISTOR-1206-10K -> (none)
- R202: symbol tronixio:RESISTOR-1206-1K -> tronixio:KOASPEER-RK73B-1206-1K-5P; Name RESISTOR-1206-1K -> (none)
- R203, R204, R205: symbol tronixio:RESISTOR-1206-4K7 -> tronixio:KOASPEER-RK73B-1206-4K7-5P; Name RESISTOR-1206-4K7 -> (none)
- S201: Name ALPS-SKRPAC -> (none)
- TP201, TP202: Name KEYSTONE-5006 -> (none)
- TP203: Name KEYSTONE-2000-3 -> (none)
- U201: Name TI-TLV1117-33-SOT-223 -> (none)
- U202: Name MICROCHIP-PIC16F1778-ISP -> (none)
Other:
- moved on the sheet: JP201, JP202, JP203, JP204
