File: Kicad/mini/pic8bit-mcu.kicad_sch (KiCad schematic)
At the start: 30 parts, among them K201 *Power & UART, K202 MCU 1, K203 MCU 1, K204 ICSP, K205 MCU 2, K206 MCU 2, U201 TLV1117-33, U202 PIC16F/PIC18F

Commit message: Update Mini
Parts:
- C201, C203: symbol tronixio:KEMET-X5R-1206-10U-25V-20P -> tronixio:KEMET-X5R-1206-10U-6V3-20P; Mouser 80-C1206C106M3P -> 80-C1206C106M9P; Voltage 25V -> 6V3
Changed lines of the file:
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@@
       (effects (font (size 1 1)) hide)
     )
-    (property "Name" "+3V3" (id 4) (at 121.92 157.48 0)
+    (property "Name" "3V3" (id 4) (at 121.92 157.48 0)
       (effects (font (size 1.15 1.15)))
     )
@@
     (pin "1")
   )
-  (symbol (lib_id "tronixio:POWER-+3V3") (at 170.18 27.94 0) (unit 1)
+  (symbol (lib_name "POWER-+3V3_1") (lib_id "tronixio:POWER-+3V3") (at 170.18 27.94 0) (unit 1)
     (in_bom yes) (on_board yes) (fields_autoplaced)
     (property "Reference" "#PWR0221" (id 0) (at 170.18 40.64 0)
@@
       (effects (font (size 1 1)) hide)
     )
-    (property "Name" "+3V3" (id 4) (at 170.18 22.86 0)
-      (effects (font (size 1.15 1.15)))
-    )
-    (pin "1")
-  )
-  (symbol (lib_id "tronixio:POWER-+3V3") (at 144.78 107.95 0) (unit 1)
+    (property "Name" "3V3" (id 4) (at 170.18 22.86 0)
+      (effects (font (size 1.15 1.15)))
+    )
+    (pin "1")
+  )
+  (symbol (lib_name "POWER-+3V3_3") (lib_id "tronixio:POWER-+3V3") (at 144.78 107.95 0) (unit 1)
     (in_bom yes) (on_board yes) (fields_autoplaced)
     (property "Reference" "#PWR0216" (id 0) (at 144.78 120.65 0)
@@
       (effects (font (size 1 1)) hide)
     )
-    (property "Name" "+3V3" (id 4) (at 144.78 102.87 0)
+    (property "Name" "3V3" (id 4) (at 144.78 102.87 0)
       (effects (font (size 1.15 1.15)))
     )
@@
     (pin "1")
   )
-  (symbol (lib_id "tronixio:KEMET-X5R-1206-10U-25V-20P") (at 81.28 180.34 0) (unit 1)
+  (symbol (lib_id "tronixio:KEMET-X5R-1206-10U-6V3-20P") (at 81.28 180.34 0) (unit 1)
     (in_bom yes) (on_board yes)
     (property "Reference" "C201" (id 0) (at 80.645 177.8 0)
@@
       (effects (font (size 1.15 1.15)) (justify left) hide)
     )
-    (property "Mouser" "80-C1206C106M3P" (id 5) (at 81.28 195.58 0)
-      (effects (font (size 1 1)) hide)
-    )
-    (property "Voltage" "25V" (id 7) (at 82.55 185.42 0)
+    (property "Mouser" "80-C1206C106M9P" (id 5) (at 81.28 195.58 0)
+      (effects (font (size 1 1)) hide)
+    )
+    (property "Voltage" "6V3" (id 7) (at 82.55 185.42 0)
       (effects (font (size 1.15 1.15)) (justify left) hide)
     )
@@
     (pin "2")
   )
-  (symbol (lib_id "tronixio:KEMET-X5R-1206-10U-25V-20P") (at 106.68 180.34 0) (unit 1)
+  (symbol (lib_id "tronixio:KEMET-X5R-1206-10U-6V3-20P") (at 106.68 180.34 0) (unit 1)
     (in_bom yes) (on_board yes)
     (property "Reference" "C203" (id 0) (at 107.315 177.8 0)
@@
       (effects (font (size 1.15 1.15)) (justify left) hide)
     )
-    (property "Mouser" "80-C1206C106M3P" (id 5) (at 106.68 195.58 0)
-      (effects (font (size 1 1)) hide)
-    )
-    (property "Voltage" "25V" (id 7) (at 107.95 185.42 0)
+    (property "Mouser" "80-C1206C106M9P" (id 5) (at 106.68 195.58 0)
+      (effects (font (size 1 1)) hide)
+    )
+    (property "Voltage" "6V3" (id 7) (at 107.95 185.42 0)
       (effects (font (size 1.15 1.15)) (justify left) hide)
     )
@@
     (pin "1")
   )
-  (symbol (lib_id "tronixio:POWER-+3V3") (at 109.22 27.94 0) (unit 1)
+  (symbol (lib_name "POWER-+3V3_5") (lib_id "tronixio:POWER-+3V3") (at 109.22 27.94 0) (unit 1)
     (in_bom yes) (on_board yes) (fields_autoplaced)
     (property "Reference" "#PWR0209" (id 0) (at 109.22 40.64 0)
@@
       (effects (font (size 1 1)) hide)
     )
-    (property "Name" "+3V3" (id 4) (at 109.22 22.86 0)
-      (effects (font (size 1.15 1.15)))
-    )
-    (pin "1")
-  )
-  (symbol (lib_id "tronixio:POWER-+3V3") (at 76.2 27.94 0) (mirror y) (unit 1)
+    (property "Name" "3V3" (id 4) (at 109.22 22.86 0)
+      (effects (font (size 1.15 1.15)))
+    )
+    (pin "1")
+  )
+  (symbol (lib_name "POWER-+3V3_4") (lib_id "tronixio:POWER-+3V3") (at 76.2 27.94 0) (mirror y) (unit 1)
     (in_bom yes) (on_board yes) (fields_autoplaced)
     (property "Reference" "#PWR0203" (id 0) (at 76.2 40.64 0)
@@
       (effects (font (size 1 1)) hide)
     )
-    (property "Name" "+3V3" (id 4) (at 76.2 22.86 0)
+    (property "Name" "3V3" (id 4) (at 76.2 22.86 0)
       (effects (font (size 1.15 1.15)))
     )
@@
       (effects (font (size 1.15 1.15)) (justify right))
     )
-    (property "Footprint" "tronixio:DIP-28-W762" (id 2) (at 144.78 99.06 0)
-      (effects (font (size 1 1)) hide)
-    )
-    (property "Datasheet" "https://www.microchip.com/en-us/product/PIC16F1778" (id 3) (at 144.78 101.6 0)
-      (effects (font (size 1 1)) hide)
-    )
-    (property "Mouser" "579-PIC16F1778-I/SP" (id 6) (at 144.78 104.14 0)
+    (property "Footprint" "tronixio:DIP-28-W762" (id 2) (at 144.78 96.52 0)
+      (effects (font (size 1 1)) hide)
+    )
+    (property "Datasheet" "https://www.microchip.com/en-us/product/PIC16F1778" (id 3) (at 144.78 99.06 0)
+      (effects (font (size 1 1)) hide)
+    )
+    (property "Mouser" "579-PIC16F1778-I/SP" (id 6) (at 144.78 101.6 0)
       (effects (font (size 1 1)) hide)
     )
@@
     (pin "2")
   )
-  (symbol (lib_id "tronixio:POWER-+3V3") (at 180.34 27.94 0) (unit 1)
+  (symbol (lib_name "POWER-+3V3_2") (lib_id "tronixio:POWER-+3V3") (at 180.34 27.94 0) (unit 1)
     (in_bom yes) (on_board yes) (fields_autoplaced)
     (property "Reference" "#PWR0223" (id 0) (at 180.34 40.64 0)
@@
       (effects (font (size 1 1)) hide)
     )
-    (property "Name" "+3V3" (id 4) (at 180.34 22.86 0)
+    (property "Name" "3V3" (id 4) (at 180.34 22.86 0)
       (effects (font (size 1.15 1.15)))
     )
@@
     (pin "1")
   )
-  (symbol (lib_id "tronixio:POWER-+3V3") (at 106.68 162.56 0) (unit 1)
+  (symbol (lib_name "POWER-+3V3_6") (lib_id "tronixio:POWER-+3V3") (at 106.68 162.56 0) (unit 1)
     (in_bom yes) (on_board yes) (fields_autoplaced)
     (property "Reference" "#PWR0210" (id 0) (at 106.68 175.26 0)
@@
       (effects (font (size 1 1)) hide)
     )
-    (property "Name" "+3V3" (id 4) (at 106.68 157.48 0)
+    (property "Name" "3V3" (id 4) (at 106.68 157.48 0)
       (effects (font (size 1.15 1.15)))
     )
@@
       (effects (font (size 1 1)) hide)
     )
-    (property "Name" "+5V" (id 4) (at 177.8 177.8 0)
+    (property "Name" "5V" (id 4) (at 177.8 177.8 0)
       (effects (font (size 1.15 1.15)))
     )
@@
       (effects (font (size 1.15 1.15)))
     )
-    (property "Footprint" "tronixio:SAMTEC-SSW-106-02-T-S-RA" (id 2) (at 149.86 133.35 0)
-      (effects (font (size 1 1)) hide)
-    )
-    (property "Datasheet" "https://ww1.microchip.com/downloads/en/DeviceDoc/30277d.pdf" (id 3) (at 149.86 135.89 0)
-      (effects (font (size 1 1)) hide)
-    )
-    (property "Mouser" "200-SSW10602TSRA" (id 6) (at 149.86 138.43 0)
+    (property "Footprint" "tronixio:SAMTEC-SSW-106-02-T-S-RA" (id 2) (at 149.86 130.81 0)
+      (effects (font (size 1 1)) hide)
+    )
+    (property "Datasheet" "https://ww1.microchip.com/downloads/en/DeviceDoc/30277d.pdf" (id 3) (at 149.86 133.35 0)
+      (effects (font (size 1 1)) hide)
+    )
+    (property "Mouser" "200-SSW10602TSRA" (id 6) (at 149.86 135.89 0)
       (effects (font (size 1 1)) hide)
     )
@@
     (pin "9")
   )
-  (symbol (lib_id "tronixio:POWER-+5V") (at 81.28 162.56 0) (unit 1)
+  (symbol (lib_name "POWER-+5V_1") (lib_id "tronixio:POWER-+5V") (at 81.28 162.56 0) (unit 1)
     (in_bom yes) (on_board yes) (fields_autoplaced)
     (property "Reference" "#PWR0205" (id 0) (at 81.28 172.72 0)
@@
       (effects (font (size 1 1)) hide)
     )
-    (property "Name" "+5V" (id 4) (at 81.28 157.48 0)
-      (effects (font (size 1.15 1.15)))
-    )
+    (property "Name" "5V" (id 4) (at 81.28 157.48 0)
+      (effects (font (size 1.15 1.15)))
+    )

Commit message: Up
Parts:
- C201, C203: symbol tronixio:KEMET-X5R-1206-10U-6V3-20P -> tronixio:CAPACITOR-1206-10U-20P-X7R
- C202, C205: symbol tronixio:KEMET-X7R-1206-100N-50V-20P -> tronixio:CAPACITOR-1206-100N-10P-X7R; Mouser 80-C1206C104M5R -> 80-C1206C104K5R; Tolerance 20% -> 10%
- R201: symbol tronixio:KOASPEER-RK73B-1206-10K-5P -> tronixio:RESISTOR-1206-10K-5P
- R202: symbol tronixio:KOASPEER-RK73B-1206-1K-5P -> tronixio:RESISTOR-1206-1K-5P
- R203, R204, R205: symbol tronixio:KOASPEER-RK73B-1206-4K7-5P -> tronixio:RESISTOR-1206-4K7-5P
Other:
- moved on the sheet: C204, C205, JP203, K203, K204, K206

Commit message: Update
Parts:
- C201, C203: symbol tronixio:CAPACITOR-1206-10U-20P-X7R -> tronixio:CAPACITOR-1206-10U-10P-X7R; Mouser 80-C1206C106M9P -> 80-C1206C106K3R; Tolerance 20% -> 10%; Voltage 6V3 -> 25V
- C202, C205: Mouser 80-C1206C104K5R -> 187-CL31B106KAHNFNE
Changed lines of the file:
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@@
     )
   )
-  (symbol (lib_id "tronixio:CAPACITOR-1206-10U-20P-X7R") (at 81.28 180.34 0) (unit 1)
+  (symbol (lib_id "tronixio:CAPACITOR-1206-10U-10P-X7R") (at 81.28 180.34 0) (unit 1)
     (in_bom yes) (on_board yes) (dnp no)
     (property "Reference" "C201" (at 80.645 177.8 0)
@@
       (effects (font (size 1 1)) hide)
     )
-    (property "Tolerance" "20%" (at 82.28 185.42 0) (do_not_autoplace)
-      (effects (font (size 1.15 1.15)) (justify left) hide)
-    )
-    (property "Mouser" "80-C1206C106M9P" (at 81.28 193.04 0)
-      (effects (font (size 1 1)) hide)
-    )
-    (property "Voltage" "6V3" (at 86.28 185.42 0) (do_not_autoplace)
+    (property "Tolerance" "10%" (at 82.28 185.42 0) (do_not_autoplace)
+      (effects (font (size 1.15 1.15)) (justify left) hide)
+    )
+    (property "Mouser" "80-C1206C106K3R" (at 81.28 193.04 0)
+      (effects (font (size 1 1)) hide)
+    )
+    (property "Voltage" "25V" (at 86.28 185.42 0) (do_not_autoplace)
       (effects (font (size 1.15 1.15)) (justify left) hide)
     )
@@
       (effects (font (size 1.15 1.15)) (justify left) hide)
     )
-    (property "Mouser" "80-C1206C104K5R" (at 170.18 114.3 0)
+    (property "Mouser" "187-CL31B106KAHNFNE" (at 170.18 114.3 0)
       (effects (font (size 1 1)) hide)
     )
@@
     )
   )
-  (symbol (lib_id "tronixio:CAPACITOR-1206-10U-20P-X7R") (at 106.68 180.34 0) (unit 1)
+  (symbol (lib_id "tronixio:CAPACITOR-1206-10U-10P-X7R") (at 106.68 180.34 0) (unit 1)
     (in_bom yes) (on_board yes) (dnp no)
     (property "Reference" "C203" (at 107.315 177.8 0)
@@
       (effects (font (size 1 1)) hide)
     )
-    (property "Tolerance" "20%" (at 107.68 185.42 0) (do_not_autoplace)
-      (effects (font (size 1.15 1.15)) (justify left) hide)
-    )
-    (property "Mouser" "80-C1206C106M9P" (at 106.68 193.04 0)
-      (effects (font (size 1 1)) hide)
-    )
-    (property "Voltage" "6V3" (at 111.68 185.42 0) (do_not_autoplace)
+    (property "Tolerance" "10%" (at 107.68 185.42 0) (do_not_autoplace)
+      (effects (font (size 1.15 1.15)) (justify left) hide)
+    )
+    (property "Mouser" "80-C1206C106K3R" (at 106.68 193.04 0)
+      (effects (font (size 1 1)) hide)
+    )
+    (property "Voltage" "25V" (at 111.68 185.42 0) (do_not_autoplace)
       (effects (font (size 1.15 1.15)) (justify left) hide)
     )
@@
       (effects (font (size 1.15 1.15)) (justify left) hide)
     )
-    (property "Mouser" "80-C1206C104K5R" (at 83.82 55.88 0)
-      (effects (font (size 1 1)) hide)
-    )
+    (property "Mouser" "187-CL31B106KAHNFNE" (at 83.82 55.88 0)
+      (effects (font (size 1 1)) hide)
+    )

Commit message: Up
Parts:
- C201, C203: symbol tronixio:CAPACITOR-1206-10U-10P-X7R -> tronixio:CAPACITOR-1206-10U-25V-5P-X7R; Mouser 80-C1206C106K3R -> 791-1206X106J250CT; Tolerance 10% -> 5%
- C202, C205: symbol tronixio:CAPACITOR-1206-100N-10P-X7R -> tronixio:CAPACITOR-1206-100N-50V-5P-X7R; Mouser 187-CL31B106KAHNFNE -> 80-C1206C104J5R; Tolerance 10% -> 5%
- R201: value 10K -> 10k
- R202: value 1K -> 1k
- R203, R204, R205: value 4K7 -> 4k7
Other:
- moved on the sheet: JP204

Commit message: Up
Parts:
- removed C204: 10µ, tronixio:KEMET-C322, symbol tronixio:KEMET-C322-0508-10U-25V-10P
- added C204: 10µ, tronixio:CAPACITOR-SMD-1206, symbol tronixio:CAPACITOR-1206-10U-25V-5P-X7R
- K201: footprint tronixio:FCI-USB-TYPE-B-MICRO-THT -> tronixio:USB-TYPE-B-MICRO-TH
- U202: footprint tronixio:DIP-28-W762 -> tronixio:DIP-28-W762-SOCKET
Connections:
- net GND: now also K201.SH (SHIELD), C204.2; no longer K201.6 (SHIELD)
- net at JP203.2: now also C204.1
Changed lines of the file:
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@@
+    )
+  )
+  (symbol (lib_id "tronixio:CAPACITOR-1206-10U-25V-5P-X7R") (at 119.38 104.14 0) (unit 1)
+    (in_bom yes) (on_board yes) (dnp no)
+    (property "Reference" "C204" (at 118.745 106.68 0)
+      (effects (font (size 1.15 1.15)) (justify right))
+    )
+    (property "Value" "10µ" (at 118.745 109.22 0)
+      (effects (font (size 1.15 1.15)) (justify right))
+    )
+    (property "Footprint" "tronixio:CAPACITOR-SMD-1206" (at 119.38 114.3 0) (do_not_autoplace)
+      (effects (font (size 1 1)) hide)
+    )
+    (property "Datasheet" "" (at 119.38 119.38 0)
+      (effects (font (size 1 1)) hide)
+    )
+    (property "Tolerance" "5%" (at 120.38 109.22 0) (do_not_autoplace)
+      (effects (font (size 1.15 1.15)) (justify left) hide)
+    )
+    (property "Mouser" "791-1206X106J250CT" (at 119.38 116.84 0) (do_not_autoplace)
+      (effects (font (size 1 1)) hide)
+    )
+    (property "Voltage" "25V" (at 124.38 109.22 0) (do_not_autoplace)
+      (effects (font (size 1.15 1.15)) (justify left) hide)
+    )
+    (pin "1")
+    (pin "2")
+    (instances
+      (project "pic8bit"
+        (path "/d431d485-8cd8-4e00-afcd-f39218d614ca/64edc06d-d6ae-4dac-9759-3f1fbed6457d"
+          (reference "C204") (unit 1)
+        )
+      )
     )
   )
@@
       (effects (font (size 1.15 1.15)))
     )
-    (property "Footprint" "tronixio:FCI-USB-TYPE-B-MICRO-THT" (at 38.1 193.04 0) (do_not_autoplace)
+    (property "Footprint" "tronixio:USB-TYPE-B-MICRO-TH" (at 38.1 193.04 0) (do_not_autoplace)
       (effects (font (size 1 1)) hide)
     )
@@
     (pin "4")
     (pin "5")
-    (pin "6")
+    (pin "SH")
     (instances
       (project "pic8bit"
@@
       (effects (font (size 1.15 1.15)) (justify right))
     )
-    (property "Footprint" "tronixio:DIP-28-W762" (at 144.78 96.52 0) (do_not_autoplace)
+    (property "Footprint" "tronixio:DIP-28-W762-SOCKET" (at 144.78 96.52 0) (do_not_autoplace)
       (effects (font (size 1 1)) hide)
     )
@@
         )
       )
-    )
-  )
-  (symbol (lib_id "tronixio:KEMET-C322-0508-10U-25V-10P") (at 119.38 104.14 0) (unit 1)
-    (in_bom yes) (on_board yes) (dnp no)
-    (property "Reference" "C204" (at 118.745 106.68 0)
-      (effects (font (size 1.15 1.15)) (justify right))
-    )
-    (property "Value" "10µ" (at 118.745 109.22 0)
-      (effects (font (size 1.15 1.15)) (justify right))
-    )
-    (property "Footprint" "tronixio:KEMET-C322" (at 119.38 116.84 0) (do_not_autoplace)
-      (effects (font (size 1 1)) hide)
-    )
-    (property "Datasheet" "https://content.kemet.com/datasheets/KEM_C1054_HIVOLT_GOLDMAX_300_C0G.pdf" (at 119.38 114.3 0) (do_not_autoplace)
-      (effects (font (size 1 1)) hide)
-    )
-    (property "Tolerance" "10%" (at 124.46 109.22 0) (do_not_autoplace)
-      (effects (font (size 1.15 1.15)) (justify left) hide)
-    )
-    (property "Mouser" "80-C322C106K3R" (at 119.38 119.38 0) (do_not_autoplace)
-      (effects (font (size 1 1)) hide)
-    )
-    (property "Voltage" "25V" (at 120.65 109.22 0) (do_not_autoplace)
-      (effects (font (size 1.15 1.15)) (justify left) hide)
-    )
-    (pin "1")
-    (pin "2")
-    (instances
-      (project "pic8bit"
-        (path "/d431d485-8cd8-4e00-afcd-f39218d614ca/64edc06d-d6ae-4dac-9759-3f1fbed6457d"
-          (reference "C204") (unit 1)
-        )
-      )

Commit message: Up
Parts:
- K201: symbol tronixio:FCI-USB-TYPE-B-MICRO-THT -> tronixio:FCI-USB-TYPE-B-MICRO-TH
Changed lines of the file:
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@@
     )
   )
-  (symbol (lib_id "tronixio:FCI-USB-TYPE-B-MICRO-THT") (at 38.1 175.26 0) (unit 1)
+  (symbol (lib_id "tronixio:FCI-USB-TYPE-B-MICRO-TH") (at 38.1 175.26 0) (unit 1)
     (in_bom yes) (on_board yes) (dnp no)
     (property "Reference" "K201" (at 38.1 162.56 0)

Commit message: Up
Parts:
- K204: symbol tronixio:MICROCHIP-ICSP-F-1X06 -> tronixio:MICROCHIP-ICSP-F-RIGHT-ANGLE-TH
- U202: footprint tronixio:DIP-28-W762-SOCKET -> tronixio:DIP-28-W762
Changed lines of the file:
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@@
       (effects (font (size 1.15 1.15)) (justify right))
     )
-    (property "Footprint" "tronixio:DIP-28-W762-SOCKET" (at 144.78 96.52 0) (do_not_autoplace)
+    (property "Footprint" "tronixio:DIP-28-W762" (at 144.78 96.52 0) (do_not_autoplace)
       (effects (font (size 1 1)) hide)
     )
@@
     )
   )
-  (symbol (lib_id "tronixio:MICROCHIP-ICSP-F-1X06") (at 149.86 111.76 0) (unit 1)
+  (symbol (lib_id "tronixio:MICROCHIP-ICSP-F-RIGHT-ANGLE-TH") (at 149.86 111.76 0) (unit 1)
     (in_bom yes) (on_board yes) (dnp no)
     (property "Reference" "K204" (at 149.86 109.22 0)

Commit message: Update
Parts:
- C201, C203, C204: Mouser 791-1206X106J250CT -> 80-C1206C106J3R
- D201, D202: symbol tronixio:NEXPERIA-PMEG3030 -> tronixio:NEXPERIA-PMEG3030-SOD
Changed lines of the file:
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@@
       (effects (font (size 1.15 1.15)) (justify left) hide)
     )
-    (property "Mouser" "791-1206X106J250CT" (at 119.38 116.84 0) (do_not_autoplace)
+    (property "Mouser" "80-C1206C106J3R" (at 119.38 116.84 0) (do_not_autoplace)
       (effects (font (size 1 1)) hide)
     )
@@
     )
   )
-  (symbol (lib_id "tronixio:NEXPERIA-PMEG3030") (at 68.58 175.26 180) (unit 1)
+  (symbol (lib_id "tronixio:NEXPERIA-PMEG3030-SOD") (at 68.58 175.26 180) (unit 1)
     (in_bom yes) (on_board yes) (dnp no)
     (property "Reference" "D202" (at 68.58 180.34 0)
@@
       (effects (font (size 1.15 1.15)) (justify left) hide)
     )
-    (property "Mouser" "791-1206X106J250CT" (at 81.28 193.04 0) (do_not_autoplace)
+    (property "Mouser" "80-C1206C106J3R" (at 81.28 193.04 0) (do_not_autoplace)
       (effects (font (size 1 1)) hide)
     )
@@
       (effects (font (size 1.15 1.15)) (justify left) hide)
     )
-    (property "Mouser" "791-1206X106J250CT" (at 106.68 193.04 0) (do_not_autoplace)
+    (property "Mouser" "80-C1206C106J3R" (at 106.68 193.04 0) (do_not_autoplace)
       (effects (font (size 1 1)) hide)
     )
@@
     )
   )
-  (symbol (lib_id "tronixio:NEXPERIA-PMEG3030") (at 68.58 170.18 180) (unit 1)
+  (symbol (lib_id "tronixio:NEXPERIA-PMEG3030-SOD") (at 68.58 170.18 180) (unit 1)
     (in_bom yes) (on_board yes) (dnp no)
     (property "Reference" "D201" (at 68.58 165.1 0)
