File: Kicad/trainer/pic8bit-hid.kicad_sch (KiCad schematic)
At the start: 24 parts, among them K301 I2C/GPIO, K302 I2C/SPI, K303 SPI/GPIO, K304 EUSART/TTL

Commit message: Update
Parts:
- removed K302: I2C/SPI, tronixio:HARWIN-M20-974034x, symbol tronixio:HARWIN-254-M-2X03-HORIZONTAL
- added K302: HARWIN-254-M-2X03-RIGHT-ANGLE, tronixio:HARWIN-M20-974034x, symbol tronixio:HARWIN-254-M-2X03-RIGHT-ANGLE
- D301, D302, D303, D304: MOUSER 511-ESDA14V2SC5Y -> (none); Mouser (none) -> 511-ESDA14V2SC5Y
- K301, K304: MOUSER 200-SSW10602TSRA -> (none); Mouser (none) -> 200-SSW10602TSRA
- K303: value SPI/GPIO -> (none); footprint tronixio:SAMTEC-SSW-106-02-T-D-RA -> (none); MOUSER 200-SSW10602TDRA -> (none); Mouser (none) -> 200-SSW10602TDRA
Connections:
- net GND: now also K303.10, K303.9; no longer K303.11, K303.5
- net RC3/SCK: now also K302.5
- net RC3/SCL: now also K302.1
- net RC3/SCL/SCK: now also K302.3
- net RC4/MISO: now also K302.6
- net RC4/SDA: now also K302.2
- net RC4/SDA/MISO: now also K302.4
- net SPI_CS2: now also K303.6; no longer K303.9
- net SPI_CS3: now also K303.8; no longer K303.10
- net SPI_INT: now also K303.2; no longer K303.7
- net SPI_MISO: now also K303.5; no longer K303.3
- net SPI_MOSI: now also K303.3; no longer K303.2
- net SPI_RESET: now also K303.4; no longer K303.8
- net SPI_SCK: now also K303.7; no longer K303.4
- net VCC: now also K303.11; no longer K303.6

Commit message: Up
Parts:
- removed D301, D302, D303, D304: ST-ESDA14V2SC5Y, tronixio:SOT-23-5, symbol tronixio:ST-ESDA14V2SC5Y
- removed K301: I2C/GPIO, tronixio:SAMTEC-SSW-106-02-T-S-RA, symbol tronixio:SAMTEC-SSW-106-02-T-S-RA
- removed K302: HARWIN-254-M-2X03-RIGHT-ANGLE, tronixio:HARWIN-M20-974034x, symbol tronixio:HARWIN-254-M-2X03-RIGHT-ANGLE
- removed K303: (no value), symbol tronixio:SAMTEC-SSW-106-02-T-D-RA
- removed K304: EUSART/TTL, tronixio:SAMTEC-SSW-106-02-T-S-RA, symbol tronixio:SAMTEC-SSW-106-02-T-S-RA
- removed R301, R302, R303, R304, R305, R306, R307, R308, R309, R310, R311, R312, R313, R314, R315, R316: 200R, tronixio:RESISTOR-1206, symbol tronixio:R-1206
- added BB401: BREADBOARD-170, tronixio:BREADBOARD-170, symbol tronixio:BREADBOARD-170
- added EB401: TRONIXIO-EXPANSION-BOARD, tronixio:zzzTRONIXIO-EXPANSION-BOARD, symbol tronixio:TRONIXIO-EXPANSION-BOARD
- added JP401: VEE, tronixio:HARWIN-M20-999024x, symbol tronixio:HARWIN-254-M-1X02-JUMPER-VERTICAL
- added JP402: BCKL, tronixio:HARWIN-M20-999024x, symbol tronixio:HARWIN-254-M-1X02-JUMPER-VERTICAL
- added K401: VIN, tronixio:zzHARWIN-M20-782044x, symbol tronixio:HARWIN-254-F-1X04-VERTICAL
- added K402, K408: SYMBOL-HEADER-F-1X10, tronixio:zzHARWIN-M20-782104x, symbol tronixio:SYMBOL-HEADER-F-1X10
- added K403: VIN, tronixio:HARWIN-M20-999044x, symbol tronixio:HARWIN-254-M-1X04-VERTICAL
- added K404: VDD, tronixio:zzHARWIN-M20-782044x, symbol tronixio:HARWIN-254-F-1X04-VERTICAL
- added K405: GND, tronixio:zzHARWIN-M20-782044x, symbol tronixio:HARWIN-254-F-1X04-VERTICAL
- added K406: VDD, tronixio:HARWIN-M20-999044x, symbol tronixio:HARWIN-254-M-1X04-VERTICAL
- added K407: GND, tronixio:HARWIN-M20-999044x, symbol tronixio:HARWIN-254-M-1X04-VERTICAL
- added K409: HARWIN-254-F-1X16-VERTICAL, tronixio:zzHARWIN-M20-782164x, symbol tronixio:HARWIN-254-F-1X16-VERTICAL
- added K410: LED, tronixio:zzHARWIN-M20-782104x, symbol tronixio:SYMBOL-HEADER-F-1X10
- added LED401: KINGBRIGHT-DC10EWA, tronixio:KINGBRIGHT-DC, symbol tronixio:KINGBRIGHT-DC10EWA
- added P401: AN1, tronixio:PIHER-PT10MV, symbol tronixio:PIHER-PT10MV-10K
- added P402: AN2, tronixio:PIHER-PT10MV, symbol tronixio:PIHER-PT10MV-10K
- added R401: PIHER-PT10LV-5K, tronixio:PIHER-PT10LV, symbol tronixio:PIHER-PT10LV-5K
- added R402: 10Ω, tronixio:RESISTOR-1016-TH, symbol tronixio:R-0805
- added RA401: BOURNS-4611X, tronixio:4611X, symbol tronixio:BOURNS-4611X-330R
- added S401: S1, tronixio:CK-KSA-TH, symbol tronixio:CK-KSA
- added S402: S3, tronixio:CK-KSA-TH, symbol tronixio:CK-KSA
- added S403: BOURNS-PEC12R-24DENTS, tronixio:BOURNS-PEC12R, symbol tronixio:BOURNS-PEC12R-24DENTS
- added S404: S2, tronixio:CK-KSA-TH, symbol tronixio:CK-KSA
- added S405: S4, tronixio:CK-KSA-TH, symbol tronixio:CK-KSA
Connections:
- net GND: now also K402.5 (Pin_5), K405.1, K405.2, K405.3, K405.4, K407.1, K407.2, K407.3, K407.4, K408.10 (Pin_10), K408.6 (Pin_6), K408.7 (Pin_7), K408.8 (Pin_8), K408.9 (Pin_9), P401.1, P402.1, R401.3, RA401.1, S401.3, S401.4, S402.3, S402.4, S403.2 (C), S403.4 (2), S404.3, S404.4, S405.3, S405.4
- net VCC: now also K404.1, K404.2, K404.3, K404.4, K406.1, K406.2, K406.3, K406.4, K408.1 (Pin_1), K408.2 (Pin_2), K408.3 (Pin_3), K408.4 (Pin_4), K408.5 (Pin_5), P401.3, P402.3, R401.1, R402.1
- new net: K410.1 (Pin_1), LED401.1 (A1)
- new net: K410.10 (Pin_10), LED401.10 (A10)
- new net: LED401.11 (C10), RA401.11
- new net: LED401.12 (C9), RA401.10
- new net: LED401.13 (C8), RA401.9
- new net: LED401.14 (C7), RA401.8
- new net: LED401.15 (C6), RA401.7
- new net: LED401.16 (C5), RA401.6
- new net: LED401.17 (C4), RA401.5
- new net: LED401.18 (C3), RA401.4
- new net: LED401.19 (C2), RA401.3
- new net: K410.2 (Pin_2), LED401.2 (A2)
- new net: LED401.20 (C1), RA401.2
- new net: K410.3 (Pin_3), LED401.3 (A3)
- new net: K410.4 (Pin_4), LED401.4 (A4)
- new net: K410.5 (Pin_5), LED401.5 (A5)
- new net: K410.6 (Pin_6), LED401.6 (A6)
- new net: K410.7 (Pin_7), LED401.7 (A7)
- new net: K410.8 (Pin_8), LED401.8 (A8)
- new net: K410.9 (Pin_9), LED401.9 (A9)
- new net: JP401.1, R401.2
- new net: JP402.1, R402.2
- new net: EB401.15, JP402.2, K409.15 (Pin_15)
- new net: EB401.3, JP401.2, K409.3 (Pin_3)
- new net: EB401.1, K409.1 (Pin_1)
- new net: EB401.10, K409.10 (Pin_10)
- new net: EB401.11, K409.11 (Pin_11)
- new net: EB401.12, K409.12 (Pin_12)
- new net: EB401.13, K409.13 (Pin_13)
- new net: EB401.14, K409.14 (Pin_14)
- new net: EB401.16, K409.16 (Pin_16)
- new net: EB401.2, K409.2 (Pin_2)
- new net: EB401.4, K409.4 (Pin_4)
- new net: EB401.5, K409.5 (Pin_5)
- new net: EB401.6, K409.6 (Pin_6)
- new net: EB401.7, K409.7 (Pin_7)
- new net: EB401.8, K409.8 (Pin_8)
- new net: EB401.9, K409.9 (Pin_9)
- new net A: K402.7 (Pin_7), S403.1 (A)
- new net AN1: K402.9 (Pin_9), P401.2
- new net AN2: K402.10 (Pin_10), P402.2
- new net B: K402.8 (Pin_8), S403.3 (B)
- new net S1: K402.1 (Pin_1), S401.1, S401.2
- new net S2: K402.2 (Pin_2), S404.1, S404.2
- new net S3: K402.3 (Pin_3), S402.1, S402.2
- new net S4: K402.4 (Pin_4), S405.1, S405.2
- new net S5: K402.6 (Pin_6), S403.5 (1)
- new net VIN: K401.1, K401.2, K401.3, K401.4, K403.1, K403.2, K403.3, K403.4
Other:
- note added: "01"
- note added: "02"
- note added: "03"
- note added: "04"
- note added: "05"
- note added: "06"
- note added: "07"
- note added: "08"
- note added: "09"
- note added: "10"
- note added: "11"
- note added: "12"
- note added: "13"
- note added: "14"
- note added: "15"
- note added: "16"
- note added: "A"
- note added: "AN1"
- note added: "AN2"
- note added: "B"
- note added: "S1"
- note added: "S2"
- note added: "S3"
- note added: "S4"
- note added: "S5"
- note removed: "CTS"
- note removed: "INT"
- note removed: "RESET"
- note removed: "RTS"
- note removed: "RX"
- note removed: "SCL"
- note removed: "SDA"
- note removed: "TX"
- note removed: "VDD"
- title: HID -> Modules

Commit message: Up
Parts:
- added C401, C402: 10n, tronixio:zzzKEMET-C315, symbol tronixio:C-0805
- added R403, R404, R405, R406, R407, R408: 10K, tronixio:RESISTOR-1016-TH, symbol tronixio:R-0805
Connections:
- net GND: now also C401.2, C402.2
- net S1: now also R403.2
- net S2: now also R408.2
- net S3: now also R404.2
- net S4: now also R407.2
- net VCC: now also R403.1, R404.1, R405.1, R406.1, R407.1, R408.1
- net A renamed ROTARY_A
- net ROTARY_A: now also C401.1, R405.2
- net B renamed ROTARY_B
- net ROTARY_B: now also C402.1, R406.2

Commit message: Update
Parts:
- removed K401: VIN, tronixio:zzHARWIN-M20-782044x, symbol tronixio:HARWIN-254-F-1X04-VERTICAL
- removed K403: VIN, tronixio:HARWIN-M20-999044x, symbol tronixio:HARWIN-254-M-1X04-VERTICAL
- removed K404: VDD, tronixio:zzHARWIN-M20-782044x, symbol tronixio:HARWIN-254-F-1X04-VERTICAL
- removed K405: GND, tronixio:zzHARWIN-M20-782044x, symbol tronixio:HARWIN-254-F-1X04-VERTICAL
- removed K406: VDD, tronixio:HARWIN-M20-999044x, symbol tronixio:HARWIN-254-M-1X04-VERTICAL
- removed K407: GND, tronixio:HARWIN-M20-999044x, symbol tronixio:HARWIN-254-M-1X04-VERTICAL
- removed K408: SYMBOL-HEADER-F-1X10, tronixio:zzHARWIN-M20-782104x, symbol tronixio:SYMBOL-HEADER-F-1X10
- added R409: 10K, tronixio:RESISTOR-1016-TH, symbol tronixio:R-0805
- EB401: Mouser (none) -> 200-CES11601TS
Connections:
- net S2: now also R404.2; no longer R408.2
- net S3: now also R405.2; no longer R404.2
- net S4: now also R406.2; no longer R407.2
- net S5: now also R407.2
- net VCC: now also R409.1
- net ROTARY_A renamed A
- net A: now also R408.2; no longer R405.2
- net ROTARY_B renamed B
- net B: now also R409.2; no longer R406.2
Other:
- title: Modules -> HID
- moved on the sheet: BB401, EB401, JP401, JP402, K402, K409, K410, LED401, P401, P402, R401, R402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

Commit message: Update
Parts:
- S403: footprint tronixio:BOURNS-PEC12R -> tronixio:BOURNS-PEC12R-SWITCH; symbol tronixio:BOURNS-PEC12R-24DENTS -> tronixio:BOURNS-PEC12R-24DENTS-SWITCH-15MM
Changed lines of the file:
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@@
     (pin "1")
   )
-  (symbol (lib_id "tronixio:BOURNS-PEC12R-24DENTS") (at 104.14 96.52 0) (unit 1)
+  (symbol (lib_id "tronixio:BOURNS-PEC12R-24DENTS-SWITCH-15MM") (at 104.14 96.52 0) (unit 1)
     (in_bom yes) (on_board yes)
     (property "Reference" "S403" (id 0) (at 104.14 87.63 0)
@@
       (effects (font (size 1.15 1.15)) hide)
     )
-    (property "Footprint" "tronixio:BOURNS-PEC12R" (id 2) (at 104.14 111.76 0)
+    (property "Footprint" "tronixio:BOURNS-PEC12R-SWITCH" (id 2) (at 104.14 111.76 0)
       (effects (font (size 1 1)) hide)
     )

Commit message: Up
Parts:
- removed C401, C402: 10n, tronixio:zzzKEMET-C315, symbol tronixio:C-0805
- removed R403, R404, R405, R406, R407, R408, R409: 10K, tronixio:RESISTOR-1016-TH, symbol tronixio:R-0805
Other:
- moved on the sheet: BB401, EB401, JP401, JP402, K402, K409, K410, LED401, P401, P402, R401, R402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

Commit message: Update
Parts:
- removed K410: LED, tronixio:zzHARWIN-M20-782104x, symbol tronixio:SYMBOL-HEADER-F-1X10
- added K?: SYMBOL-HEADER-F-1X10, tronixio:HARWIN-M20-782104x, symbol tronixio:HARWIN-254-F-1X10-VERTICAL
- EB401: footprint tronixio:zzzTRONIXIO-EXPANSION-BOARD -> tronixioZZZ:TRONIXIO-EXPANSION-BOARD
- JP401, JP402: Name (none) -> HARWIN-254-M-1X02-JUMPER-VERTICAL
- K402: footprint tronixio:zzHARWIN-M20-782104x -> tronixio:HARWIN-M20-782104x; symbol tronixio:SYMBOL-HEADER-F-1X10 -> tronixio:HARWIN-254-F-1X10-VERTICAL; Mouser (none) -> 855-M20-782104; Name (none) -> HARWIN-254-F-1X10-VERTICAL
- K409: footprint tronixio:zzHARWIN-M20-782164x -> tronixio:HARWIN-M20-782164x
- LED401: Name DC10EWA -> KINGBRIGHT-DC10EWA
- P401, P402: Name 10K -> PIHER-PT10MV-10K; Tolerance (none) -> 20%
- R401: Tolrance (none) -> 20%
- R402: symbol tronixio:R-0805 -> tronixio:RESISTOR; Tolerance (none) -> 5%
- RA401: Tolerance (none) -> 2%
- S401, S402, S404, S405: Name (none) -> CK-KSA
- S403: symbol tronixio:BOURNS-PEC12R-24DENTS-SWITCH-15MM -> tronixio:BOURNS-PEC12R-24DENTS-SWITCH; Name (none) -> BOURNS-PEC12R-24DENTS-SWITCH
Connections:
- net at LED401.1 (A1): now also K?.1 (Pin_1)
- net at LED401.10 (A10): now also K?.10 (Pin_10)
- net at LED401.2 (A2): now also K?.2 (Pin_2)
- net at LED401.3 (A3): now also K?.3 (Pin_3)
- net at LED401.4 (A4): now also K?.4 (Pin_4)
- net at LED401.5 (A5): now also K?.5 (Pin_5)
- net at LED401.6 (A6): now also K?.6 (Pin_6)
- net at LED401.7 (A7): now also K?.7 (Pin_7)
- net at LED401.8 (A8): now also K?.8 (Pin_8)
- net at LED401.9 (A9): now also K?.9 (Pin_9)
- net VCC renamed VDD
Other:
- moved on the sheet: BB401, EB401, JP401, JP402, K409, LED401, R401, R402, RA401

Commit message: Update
Parts:
- EB401: value TRONIXIO-EXPANSION-BOARD -> EXPANSION-BOARD; footprint tronixioZZZ:TRONIXIO-EXPANSION-BOARD -> tronixio:TRONIXIO-EXPANSION-BOARD; Name EXPANSION-BOARD -> TRONIXIO-EXPANSION-BOARD
- K401: renamed from K?; value SYMBOL-HEADER-F-1X10 -> HARWIN-254-F-1X10-VERTICAL
- K402: value SYMBOL-HEADER-F-1X10 -> HARWIN-254-F-1X10-VERTICAL
- R401: value PIHER-PT10LV-5K -> 5K; Name 5K -> PIHER-PT10LV-5K
- R402: symbol tronixio:RESISTOR -> tronixio:RESISTOR-1016TH-10R; Mouser (none) -> 594-5043EM10R00J; Name (none) -> RESISTOR-1016TH-10R
- RA401: value BOURNS-4611X -> 330Ω; Name 330Ω -> BOURNS-4611X-330R
Changed lines of the file:
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@@
       (effects (font (size 1.15 1.15)))
     )
-    (property "Value" "KINGBRIGHT-DC10EWA" (id 1) (at 142.24 86.36 0)
-      (effects (font (size 1 1)) hide)
+    (property "Value" "KINGBRIGHT-DC10EWA" (id 1) (at 144.78 83.82 0)
+      (effects (font (size 1.15 1.15)) hide)
     )
     (property "Footprint" "tronixio:KINGBRIGHT-DC" (id 2) (at 144.78 91.44 0)
@@
       (effects (font (size 1.15 1.15)) (justify right))
     )
-    (property "Value" "PIHER-PT10LV-5K" (id 1) (at 208.28 57.15 0)
-      (effects (font (size 1 1)) hide)
+    (property "Value" "5K" (id 1) (at 207.645 74.295 0)
+      (effects (font (size 1.15 1.15)) (justify right))
     )
     (property "Footprint" "tronixio:PIHER-PT10LV" (id 2) (at 208.28 54.61 0)
@@
       (effects (font (size 1 1)) hide)
     )
-    (property "Name" "5K" (id 4) (at 205.74 68.58 0)
-      (effects (font (size 1.15 1.15)) (justify right))
+    (property "Name" "PIHER-PT10LV-5K" (id 4) (at 208.28 57.15 0)
+      (effects (font (size 1 1)) hide)
     )
     (property "Mouser" "531-PT10LV-5K" (id 5) (at 208.28 49.53 0)
       (effects (font (size 1 1)) hide)
     )
-    (property "Tolrance" "20%" (id 6) (at 209.55 62.23 0)
+    (property "Tolrance" "20%" (id 6) (at 208.915 62.23 0)
       (effects (font (size 1.15 1.15)) (justify left) hide)
     )
@@
       (effects (font (size 1.15 1.15)))
     )
-    (property "Value" "SYMBOL-HEADER-F-1X10" (id 1) (at 48.795 72.39 0)
+    (property "Value" "HARWIN-254-F-1X10-VERTICAL" (id 1) (at 48.26 101.6 0)
       (effects (font (size 1.15 1.15)) hide)
     )
@@
       (effects (font (size 1.15 1.15)))
     )
-    (property "Value" "BOURNS-4611X" (id 1) (at 160.02 83.82 0)
-      (effects (font (size 1 1)) hide)
+    (property "Value" "330Ω" (id 1) (at 160.02 55.88 0)
+      (effects (font (size 1.15 1.15)))
     )
     (property "Footprint" "tronixio:4611X" (id 2) (at 160.02 83.82 0)
@@
       (effects (font (size 1 1)) hide)
     )
-    (property "Name" "330Ω" (id 4) (at 160.02 55.88 0)
-      (effects (font (size 1.15 1.15)))
+    (property "Name" "BOURNS-4611X-330R" (id 4) (at 160.02 55.88 0)
+      (effects (font (size 1 1)) hide)
     )
     (property "Mouser" "652-4611X-1LF-330" (id 5) (at 160.02 88.9 0)
@@
     )
     (property "Tolerance" "2%" (id 6) (at 160.02 58.42 0)
-      (effects (font (size 1 1)) hide)
+      (effects (font (size 1.15 1.15)) hide)
     )
     (pin "1")
@@
     (pin "1")
   )
-  (symbol (lib_id "tronixio:RESISTOR") (at 220.98 69.85 0) (unit 1)
+  (symbol (lib_id "tronixio:RESISTOR-1016TH-10R") (at 220.98 69.85 0) (unit 1)
     (in_bom yes) (on_board yes)
     (property "Reference" "R402" (id 0) (at 221.615 66.04 0)
@@
       (effects (font (size 1.15 1.15)))
     )
-    (property "Footprint" "tronixio:RESISTOR-1016-TH" (id 2) (at 220.98 82.55 0)
-      (effects (font (size 1 1)) hide)
-    )
-    (property "Datasheet" "~" (id 3) (at 220.98 87.63 0)
+    (property "Footprint" "tronixio:RESISTOR-1016-TH" (id 2) (at 220.98 85.09 0)
+      (effects (font (size 1 1)) hide)
+    )
+    (property "Datasheet" "https://www.vishay.com/docs/28722/sfr16s25.pdf" (id 3) (at 220.98 87.63 0)
       (effects (font (size 1 1)) hide)
     )
@@
       (effects (font (size 1.15 1.15)) (justify left) hide)
     )
-    (property "Mouser" "~" (id 5) (at 220.98 90.17 0)
+    (property "Mouser" "594-5043EM10R00J" (id 5) (at 220.98 90.17 0)
+      (effects (font (size 1 1)) hide)
+    )
+    (property "Name" "RESISTOR-1016TH-10R" (id 6) (at 220.98 82.55 0)
       (effects (font (size 1 1)) hide)
     )
@@
       (effects (font (size 1.15 1.15)))
     )
-    (property "Value" "TRONIXIO-EXPANSION-BOARD" (id 1) (at 245.11 106.6799 0)
-      (effects (font (size 1.15 1.15)) hide)
-    )
-    (property "Footprint" "tronixioZZZ:TRONIXIO-EXPANSION-BOARD" (id 2) (at 236.22 132.08 0)
+    (property "Value" "EXPANSION-BOARD" (id 1) (at 236.22 128.27 0)
+      (effects (font (size 1.15 1.15)))
+    )
+    (property "Footprint" "tronixio:TRONIXIO-EXPANSION-BOARD" (id 2) (at 226.06 134.62 0)
       (effects (font (size 1 1)) hide)
     )
@@
       (effects (font (size 1 1)) hide)
     )
-    (property "Name" "EXPANSION-BOARD" (id 4) (at 236.22 128.27 0)
-      (effects (font (size 1.15 1.15)))
-    )
-    (property "Mouser" "200-CES11601TS" (id 5) (at 236.22 137.16 0)
+    (property "Name" "TRONIXIO-EXPANSION-BOARD" (id 4) (at 226.06 132.08 0)
+      (effects (font (size 1 1)) hide)
+    )
+    (property "Mouser" "200-CES11601TS" (id 5) (at 226.06 137.16 0)
       (effects (font (size 1 1)) hide)
     )
@@
   (symbol (lib_id "tronixio:HARWIN-254-F-1X10-VERTICAL") (at 132.08 55.88 0) (mirror y) (unit 1)
     (in_bom yes) (on_board yes)
-    (property "Reference" "K?" (id 0) (at 132.08 53.34 0)
-      (effects (font (size 1.15 1.15)))
-    )
-    (property "Value" "SYMBOL-HEADER-F-1X10" (id 1) (at 132.615 52.07 0)
+    (property "Reference" "K401" (id 0) (at 132.08 53.34 0)
+      (effects (font (size 1.15 1.15)))
+    )
+    (property "Value" "HARWIN-254-F-1X10-VERTICAL" (id 1) (at 132.08 81.28 0)
       (effects (font (size 1.15 1.15)) hide)
     )
@@
     (pin "1")
   )
-  (symbol (lib_name "PIHER-PT10MV-10K_1") (lib_id "tronixio:PIHER-PT10MV-10K") (at 73.66 119.38 0) (mirror y) (unit 1)
+  (symbol (lib_id "tronixio:PIHER-PT10MV-10K") (at 73.66 119.38 0) (mirror y) (unit 1)
     (in_bom yes) (on_board yes)
     (property "Reference" "P401" (id 0) (at 68.58 115.57 0)
