File: Kicad/trainer/pic8bit-hid.kicad_sch (KiCad schematic)
At the start: 18 parts, among them K401 HARWIN-254-F-1X10-VERTICAL, K402 HARWIN-254-F-1X10-VERTICAL, K409 HARWIN-254-F-1X16-VERTICAL, P401 AN1, P402 AN2

Commit message: Update
Parts:
- K409: Name (none) -> HARWIN-254-F-1X16-VERTICAL
- R401: Tolerance (none) -> 20%; Tolrance 20% -> (none)

Commit message: Update
Parts:
- R402: footprint tronixio:RESISTOR-1016-TH -> tronixio:RESISTOR-TH-1016
Changed lines of the file:
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@@
       (effects (font (size 1.15 1.15)))
     )
-    (property "Footprint" "tronixio:4611X" (id 2) (at 154.94 86.36 0)
+    (property "Footprint" "tronixio:4611X" (id 2) (at 160.02 83.82 0)
       (effects (font (size 1 1)) hide)
     )
-    (property "Datasheet" "https://www.bourns.com/docs/Product-Datasheets/4600x.pdf?sfvrsn=92b2512c_0" (id 3) (at 154.94 88.9 0)
+    (property "Datasheet" "https://www.bourns.com/docs/Product-Datasheets/4600x.pdf?sfvrsn=92b2512c_0" (id 3) (at 160.02 86.36 0)
       (effects (font (size 1 1)) hide)
     )
-    (property "Name" "BOURNS-4611X-330R" (id 4) (at 154.94 83.82 0)
+    (property "Name" "BOURNS-4611X-330R" (id 4) (at 160.02 81.28 0)
       (effects (font (size 1 1)) hide)
     )
-    (property "Mouser" "652-4611X-1LF-330" (id 5) (at 154.94 91.44 0)
+    (property "Mouser" "652-4611X-1LF-330" (id 5) (at 160.02 88.9 0)
       (effects (font (size 1 1)) hide)
     )
@@
       (effects (font (size 1.15 1.15)))
     )
-    (property "Footprint" "tronixio:RESISTOR-1016-TH" (id 2) (at 220.98 85.09 0)
+    (property "Footprint" "tronixio:RESISTOR-TH-1016" (id 2) (at 220.98 85.09 0)
       (effects (font (size 1 1)) hide)
     )
@@
       (effects (font (size 1 1)) hide)
     )
-    (property "Tolerance" "5%" (id 4) (at 223.52 71.12 0)
+    (property "Tolerance" "5%" (id 4) (at 223.52 73.66 0)
       (effects (font (size 1.15 1.15)) (justify left) hide)
     )
@@
       (effects (font (size 1.15 1.15)))
     )
-    (property "Footprint" "tronixio:TRONIXIO-EXPANSION-BOARD" (id 2) (at 226.06 134.62 0)
+    (property "Footprint" "tronixio:TRONIXIO-EXPANSION-BOARD" (id 2) (at 236.22 134.62 0)
       (effects (font (size 1 1)) hide)
     )
@@
       (effects (font (size 1 1)) hide)
     )
-    (property "Name" "TRONIXIO-EXPANSION-BOARD" (id 4) (at 226.06 132.08 0)
+    (property "Name" "TRONIXIO-EXPANSION-BOARD" (id 4) (at 236.22 132.08 0)
       (effects (font (size 1 1)) hide)
     )
-    (property "Mouser" "200-CES11601TS" (id 5) (at 226.06 137.16 0)
+    (property "Mouser" "200-CES11601TS" (id 5) (at 236.22 137.16 0)
       (effects (font (size 1 1)) hide)
     )

Commit message: Update
Changed lines of the file:
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@@
   (symbol (lib_id "tronixio:BOURNS-PEC12R-24DENTS-SWITCH") (at 78.74 99.06 0) (unit 1)
     (in_bom yes) (on_board yes)
-    (property "Reference" "S403" (id 0) (at 81.28 92.71 0)
-      (effects (font (size 1.15 1.15)) (justify left))
+    (property "Reference" "S403" (id 0) (at 78.74 88.265 0)
+      (effects (font (size 1.15 1.15)))
     )
     (property "Value" "BOURNS-PEC12R-24DENTS" (id 1) (at 78.74 88.9 0)
@@
   (symbol (lib_id "tronixio:BOURNS-4611X-330R") (at 154.94 55.88 0) (unit 1)
     (in_bom yes) (on_board yes)
-    (property "Reference" "RA401" (id 0) (at 154.94 53.34 0)
+    (property "Reference" "RA401" (id 0) (at 160.02 53.34 0)
       (effects (font (size 1.15 1.15)))
     )
-    (property "Value" "330Ω" (id 1) (at 154.94 55.88 0)
+    (property "Value" "330Ω" (id 1) (at 160.02 55.88 0)
       (effects (font (size 1.15 1.15)))
     )

Commit message: Update pic8bit trainer
Parts:
- EB401: Name TRONIXIO-EXPANSION-BOARD -> (none)
- JP401, JP402: Name HARWIN-254-M-1X02-JUMPER-VERTICAL -> (none)
- K401, K402: Name HARWIN-254-F-1X10-VERTICAL -> (none)
- K409: Name HARWIN-254-F-1X16-VERTICAL -> (none)
- LED401: Name KINGBRIGHT-DC10EWA -> (none)
- P401, P402: Name PIHER-PT10MV-10K -> (none)
- R401: Name PIHER-PT10LV-5K -> (none)
- R402: Name RESISTOR-1016TH-10R -> (none)
- RA401: footprint tronixio:4611X -> tronixio:BOURNS-4611X; Name BOURNS-4611X-330R -> (none)
- S401, S402, S404, S405: Name CK-KSA -> (none)
- S403: Name BOURNS-PEC12R-24DENTS-SWITCH -> (none)
Other:
- moved on the sheet: R401, R402

Commit message: Update
Parts:
- S403: symbol tronixio:BOURNS-PEC12R-24DENTS-SWITCH -> tronixio:BOURNS-PEC12R-24-DENTS-SWITCH
Changed lines of the file:
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@@
     )
   )
-  (symbol (lib_id "tronixio:BOURNS-PEC12R-24DENTS-SWITCH") (at 78.74 99.06 0) (unit 1)
+  (symbol (lib_id "tronixio:BOURNS-PEC12R-24-DENTS-SWITCH") (at 78.74 99.06 0) (unit 1)
     (in_bom yes) (on_board yes) (dnp no)
     (property "Reference" "S403" (at 78.74 88.265 0)

Commit message: Up
Parts:
- R401: footprint tronixio:PIHER-PT10LV -> tronixio:PIHER-PT10MV
- R402: symbol tronixio:RESISTOR-1016TH-10R -> tronixio:RESISTOR-1016TH-10R-5P
Connections:
- net GND: now also S403.5; no longer S403.4
- net S5: now also S403.4; no longer S403.5
- net VDD renamed +VDD
