File: Kicad/trainer/pic8bit-hid.kicad_sch (KiCad schematic)
At the start: 18 parts, among them K401 HARWIN-254-F-1X10-VERTICAL, K402 HARWIN-254-F-1X10-VERTICAL, K409 HARWIN-254-F-1X16-VERTICAL, P401 AN1, P402 AN2

Commit message: Update Trainer Kicad 8
Connections:
- net +VDD renamed POWER-VDD
- net GND renamed POWER-GND

Commit message: Update Trainer
Changed lines of the file:
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@@
 		(on_board yes)
 		(dnp no)
-		(fields_autoplaced yes)
 		(property "Reference" "#PWR0158"
 			(at 208.28 68.58 0)
@@
 			)
 		)
-		(property "Description" ""
-			(at 208.28 58.42 0)
-			(effects
-				(font
-					(size 1.27 1.27)
-				)
-				(hide yes)
-			)
-		)
-		(property "Name" "VDD"
+		(property "Description" "VDD"
 			(at 208.28 53.34 0)
-			(do_not_autoplace yes)
-			(effects
-				(font
-					(size 1.15 1.15)
+			(effects
+				(font
+					(size 1.27 1.27)
 				)
 			)
@@
 		(on_board yes)
 		(dnp no)
-		(fields_autoplaced yes)
 		(property "Reference" "#PWR0151"
 			(at 73.66 124.46 0)
@@
 			)
 		)
-		(property "Description" ""
-			(at 73.66 114.3 0)
-			(effects
-				(font
-					(size 1.27 1.27)
-				)
-				(hide yes)
-			)
-		)
-		(property "Name" "VDD"
+		(property "Description" "VDD"
 			(at 73.66 109.22 0)
-			(do_not_autoplace yes)
-			(effects
-				(font
-					(size 1.15 1.15)
+			(effects
+				(font
+					(size 1.27 1.27)
 				)
 			)
@@
 		(on_board yes)
 		(dnp no)
-		(fields_autoplaced yes)
 		(property "Reference" "#PWR0150"
 			(at 83.82 124.46 0)
@@
 			)
 		)
-		(property "Description" ""
-			(at 83.82 114.3 0)
-			(effects
-				(font
-					(size 1.27 1.27)
-				)
-				(hide yes)
-			)
-		)
-		(property "Name" "VDD"
+		(property "Description" "VDD"
 			(at 83.82 109.22 0)
-			(do_not_autoplace yes)
-			(effects
-				(font
-					(size 1.15 1.15)
-				)
-			)
+			(effects
+				(font
+					(size 1.27 1.27)
+				)
+			)

Commit message: Up
Parts:
- K401: value HARWIN-254-F-1X10-VERTICAL -> LED ARRAY
- K402: value HARWIN-254-F-1X10-VERTICAL -> SWITCH, ENCODER & ANALOG
- K409: value HARWIN-254-F-1X16-VERTICAL -> EXPANSION BOARD
Changed lines of the file:
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@@
 			)
 		)
-		(property "Value" "HARWIN-254-F-1X10-VERTICAL"
+		(property "Value" "SWITCH, ENCODER & ANALOG"
 			(at 48.26 101.6 0)
 			(effects
@@
 			)
 		)
-		(property "Datasheet" "https://www.bourns.com/docs/Product-Datasheets/4600x.pdf?sfvrsn=92b2512c_0"
+		(property "Datasheet" "https://www.bourns.com/docs/Product-Datasheets/4600x.pdf"
 			(at 160.02 86.36 0)
 			(effects
@@
 			)
 		)
-		(property "Value" "HARWIN-254-F-1X10-VERTICAL"
+		(property "Value" "LED ARRAY"
 			(at 132.08 81.28 0)
 			(effects
@@
 			)
 		)
-		(property "Value" "HARWIN-254-F-1X16-VERTICAL"
+		(property "Value" "EXPANSION BOARD"
 			(at 208.815 82.55 0)
 			(effects
