File: Kicad/trainer/pic8bit-mod.kicad_sch (KiCad schematic)
At the start: 25 parts, among them K401 VIN, K402 SYMBOL-HEADER-F-1X10, K403 VIN, K404 VDD, K405 GND, K406 VDD, K407 GND, K408 SYMBOL-HEADER-F-1X10, K409 HARWIN-254-F-1X16-VERTICAL, K410 LED, P401 AN1, P402 AN2

Commit message: Update
Parts:
- BB401: MOUSER 854-BB170 -> (none); Mouser (none) -> 854-BB170
- EB401: Name (none) -> EXPANSION-BOARD
- JP401, JP402: MOUSER 855-M20-999024 -> (none); Mouser (none) -> 855-M20-999024
- K401, K404, K405: MOUSER 855-M20-782044 -> (none); Mouser (none) -> 855-M20-782044
- K403, K406, K407: MOUSER 855-M20-999084 -> (none); Mouser (none) -> 855-M20-999044
- K409: MOUSER 855-M20-782164 -> (none); Mouser (none) -> 855-M20-782164
- LED401: MOUSER 604-DC-10EWA -> (none); Mouser (none) -> 604-DC-10EWA
- P401, P402: MOUSER 531-PT10MV-10K -> (none); Mouser (none) -> 531-PT10MV-10K; NAME 10K -> (none); Name (none) -> 10K
- R401: MOUSER 531-PT10LV-5K -> (none); Mouser (none) -> 531-PT10LV-5K; NAME 5K -> (none); Name (none) -> 5K
- RA401: MOUSER 652-4611X-1LF-330 -> (none); Mouser (none) -> 652-4611X-1LF-330; NAME 330R -> (none); Name (none) -> 330Ω
- S401, S402, S404, S405: MOUSER 611-KSA0M911LFT -> (none); Mouser (none) -> 611-KSA0M911LFT
- S403: MOUSER 652-PEC12R-4215F-S24 -> (none); Mouser (none) -> 652-PEC12R-4215F-S24
Changed lines of the file:
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@@
-      (effects (font (size 1 1)) hide)
-    )
-    (property "MOUSER" "604-DC-10EWA" (id 4) (at 139.7 85.09 0)
       (effects (font (size 1 1)) hide)
     )
     (property "Name" "DC10EWA" (id 5) (at 139.7 73.66 0)
       (effects (font (size 1.15 1.15)))
+    )
+    (property "Mouser" "604-DC-10EWA" (id 6) (at 139.7 85.09 0)
+      (effects (font (size 1 1)) hide)
     )
     (pin "1")
@@
       (effects (font (size 1 1)) hide)
     )
-    (property "MOUSER" "611-KSA0M911LFT" (id 4) (at 76.2 58.42 0)
+    (property "Mouser" "611-KSA0M911LFT" (id 4) (at 76.2 58.42 0)
       (effects (font (size 1 1)) hide)
     )
@@
       (effects (font (size 1 1)) hide)
     )
-    (property "MOUSER" "611-KSA0M911LFT" (id 4) (at 58.42 40.64 0)
+    (property "Mouser" "611-KSA0M911LFT" (id 4) (at 58.42 40.64 0)
       (effects (font (size 1 1)) hide)
     )
@@
       (effects (font (size 1 1)) hide)
     )
-    (property "MOUSER" "611-KSA0M911LFT" (id 4) (at 58.42 58.42 0)
+    (property "Mouser" "611-KSA0M911LFT" (id 4) (at 58.42 58.42 0)
       (effects (font (size 1 1)) hide)
     )
@@
       (effects (font (size 1 1)) hide)
     )
-    (property "MOUSER" "855-M20-782044" (id 4) (at 83.82 177.8 0)
+    (property "Mouser" "855-M20-782044" (id 4) (at 83.82 177.8 0)
       (effects (font (size 1 1)) hide)
     )
@@
   (symbol (lib_id "tronixio:PIHER-PT10LV-5K") (at 205.74 53.34 0) (mirror x) (unit 1)
     (in_bom yes) (on_board yes)
-    (property "Reference" "R401" (id 0) (at 205.74 46.99 0)
+    (property "Reference" "R401" (id 0) (at 205.105 49.53 0)
       (effects (font (size 1.15 1.15)) (justify right))
     )
@@
       (effects (font (size 1 1)) hide)
     )
-    (property "MOUSER" "531-PT10LV-5K" (id 4) (at 205.74 33.02 0)
-      (effects (font (size 1 1)) hide)
-    )
-    (property "NAME" "5K" (id 5) (at 205.74 49.53 0)
+    (property "Name" "5K" (id 4) (at 205.105 57.785 0)
       (effects (font (size 1.15 1.15)) (justify right))
+    )
+    (property "Mouser" "531-PT10LV-5K" (id 5) (at 205.74 33.02 0)
+      (effects (font (size 1 1)) hide)
     )
     (pin "1")
@@
       (effects (font (size 1 1)) hide)
     )
-    (property "MOUSER" "855-M20-782044" (id 4) (at 53.34 162.56 0)
+    (property "Mouser" "855-M20-782044" (id 4) (at 53.34 162.56 0)
       (effects (font (size 1 1)) hide)
     )
@@
       (effects (font (size 1 1)) hide)
     )
-    (property "Datasheet" "https://www.harwin.com/products/M20-9990846/" (id 3) (at 99.06 160.02 0)
-      (effects (font (size 1 1)) hide)
-    )
-    (property "MOUSER" "855-M20-999084" (id 4) (at 99.06 162.56 0)
+    (property "Datasheet" "https://www.harwin.com/products/M20-9990446/" (id 3) (at 99.06 160.02 0)
+      (effects (font (size 1 1)) hide)
+    )
+    (property "Mouser" "855-M20-999044" (id 4) (at 99.06 162.56 0)
       (effects (font (size 1 1)) hide)
     )
@@
       (effects (font (size 1 1)) hide)
     )
-    (property "MOUSER" "855-M20-999024" (id 4) (at 218.44 78.74 0)
+    (property "Mouser" "855-M20-999024" (id 4) (at 218.44 78.74 0)
       (effects (font (size 1 1)) hide)
     )
@@
       (effects (font (size 1 1)) hide)
     )
-    (property "Datasheet" "https://www.harwin.com/products/M20-9990846/" (id 3) (at 68.58 160.02 0)
-      (effects (font (size 1 1)) hide)
-    )
-    (property "MOUSER" "855-M20-999084" (id 4) (at 68.58 162.56 0)
+    (property "Datasheet" "https://www.harwin.com/products/M20-9990446/" (id 3) (at 68.58 160.02 0)
+      (effects (font (size 1 1)) hide)
+    )
+    (property "Mouser" "855-M20-999044" (id 4) (at 68.58 162.56 0)
       (effects (font (size 1 1)) hide)
     )
@@
       (effects (font (size 1 1)) hide)
     )
-    (property "MOUSER" "531-PT10MV-10K" (id 4) (at 83.82 124.46 0)
-      (effects (font (size 1 1)) hide)
-    )
-    (property "NAME" "10K" (id 5) (at 80.01 107.95 0)
-      (effects (font (size 1.15 1.15)) (justify right))
+    (property "Name" "10K" (id 4) (at 81.915 104.14 0)
+      (effects (font (size 1.15 1.15)) (justify left))
+    )
+    (property "Mouser" "531-PT10MV-10K" (id 5) (at 83.82 124.46 0)
+      (effects (font (size 1 1)) hide)
     )
     (pin "1")
@@
       (effects (font (size 1 1)) hide)
     )
-    (property "MOUSER" "652-PEC12R-4215F-S24" (id 4) (at 78.74 101.6 0)
+    (property "Mouser" "652-PEC12R-4215F-S24" (id 4) (at 78.74 101.6 0)
       (effects (font (size 1 1)) hide)
     )
@@
       (effects (font (size 1 1)) hide)
     )
-    (property "MOUSER" "652-4611X-1LF-330" (id 4) (at 154.94 82.55 0)
-      (effects (font (size 1 1)) hide)
-    )
-    (property "NAME" "330R" (id 5) (at 154.94 46.99 0)
-      (effects (font (size 1.15 1.15)))
+    (property "Name" "330Ω" (id 4) (at 154.94 46.99 0)
+      (effects (font (size 1.15 1.15)))
+    )
+    (property "Mouser" "652-4611X-1LF-330" (id 5) (at 154.94 80.01 0)
+      (effects (font (size 1 1)) hide)
     )
     (pin "1")
@@
       (effects (font (size 1 1)) hide)
     )
-    (property "MOUSER" "855-M20-999024" (id 4) (at 215.9 78.74 0)
+    (property "Mouser" "855-M20-999024" (id 4) (at 215.9 78.74 0)
       (effects (font (size 1 1)) hide)
     )
@@
       (effects (font (size 1 1)) hide)
     )
-    (property "MOUSER" "855-M20-782044" (id 4) (at 83.82 162.56 0)
+    (property "Mouser" "855-M20-782044" (id 4) (at 83.82 162.56 0)
       (effects (font (size 1 1)) hide)
     )
@@
       (effects (font (size 1 1)) hide)
     )
-    (property "MOUSER" "611-KSA0M911LFT" (id 4) (at 76.2 40.64 0)
+    (property "Mouser" "611-KSA0M911LFT" (id 4) (at 76.2 40.64 0)
       (effects (font (size 1 1)) hide)
     )
@@
       (effects (font (size 1 1)) hide)
     )
-    (property "Datasheet" "https://www.harwin.com/products/M20-9990846/" (id 3) (at 99.06 175.26 0)
-      (effects (font (size 1 1)) hide)
-    )
-    (property "MOUSER" "855-M20-999084" (id 4) (at 99.06 177.8 0)
+    (property "Datasheet" "https://www.harwin.com/products/M20-9990446/" (id 3) (at 99.06 175.26 0)
+      (effects (font (size 1 1)) hide)
+    )
+    (property "Mouser" "855-M20-999044" (id 4) (at 99.06 177.8 0)
       (effects (font (size 1 1)) hide)
     )
@@
     (property "Datasheet" "" (id 3) (at 223.52 95.25 0)
       (effects (font (size 1 1)) hide)
+    )
+    (property "Name" "EXPANSION-BOARD" (id 4) (at 233.68 111.76 0)
+      (effects (font (size 1.15 1.15)))
     )
     (pin "1")
@@
       (effects (font (size 1 1)) hide)
     )
-    (property "MOUSER" "854-BB170" (id 4) (at 139.7 114.3 0)
+    (property "Mouser" "854-BB170" (id 4) (at 139.7 114.3 0)
       (effects (font (size 1 1)) hide)
     )
@@
       (effects (font (size 1 1)) hide)
     )
-    (property "MOUSER" "531-PT10MV-10K" (id 4) (at 73.66 124.46 0)
-      (effects (font (size 1 1)) hide)
-    )
-    (property "NAME" "10K" (id 5) (at 69.85 107.95 0)
-      (effects (font (size 1.15 1.15)) (justify right))
+    (property "Name" "10K" (id 4) (at 71.755 104.14 0)
+      (effects (font (size 1.15 1.15)) (justify left))
+    )
+    (property "Mouser" "531-PT10MV-10K" (id 5) (at 73.66 124.46 0)
+      (effects (font (size 1 1)) hide)
     )
     (pin "1")
@@
       (effects (font (size 1 1)) hide)
     )
-    (property "MOUSER" "855-M20-782164" (id 4) (at 205.74 118.11 0)
-      (effects (font (size 1 1)) hide)
-    )
+    (property "Mouser" "855-M20-782164" (id 4) (at 205.74 118.11 0)
+      (effects (font (size 1 1)) hide)
+    )

Commit message: Up
Parts:
- removed BB401: BREADBOARD-170, tronixio:BREADBOARD-170, symbol tronixio:BREADBOARD-170
- removed EB401: TRONIXIO-EXPANSION-BOARD, tronixio:zzzTRONIXIO-EXPANSION-BOARD, symbol tronixio:TRONIXIO-EXPANSION-BOARD
- removed JP401: VEE, tronixio:HARWIN-M20-999024x, symbol tronixio:HARWIN-254-M-1X02-JUMPER-VERTICAL
- removed JP402: BCKL, tronixio:HARWIN-M20-999024x, symbol tronixio:HARWIN-254-M-1X02-JUMPER-VERTICAL
- removed K401: VIN, tronixio:zzHARWIN-M20-782044x, symbol tronixio:HARWIN-254-F-1X04-VERTICAL
- removed K402, K408: SYMBOL-HEADER-F-1X10, tronixio:zzHARWIN-M20-782104x, symbol tronixio:SYMBOL-HEADER-F-1X10
- removed K403: VIN, tronixio:HARWIN-M20-999044x, symbol tronixio:HARWIN-254-M-1X04-VERTICAL
- removed K404: VDD, tronixio:zzHARWIN-M20-782044x, symbol tronixio:HARWIN-254-F-1X04-VERTICAL
- removed K405: GND, tronixio:zzHARWIN-M20-782044x, symbol tronixio:HARWIN-254-F-1X04-VERTICAL
- removed K406: VDD, tronixio:HARWIN-M20-999044x, symbol tronixio:HARWIN-254-M-1X04-VERTICAL
- removed K407: GND, tronixio:HARWIN-M20-999044x, symbol tronixio:HARWIN-254-M-1X04-VERTICAL
- removed K409: HARWIN-254-F-1X16-VERTICAL, tronixio:zzHARWIN-M20-782164x, symbol tronixio:HARWIN-254-F-1X16-VERTICAL
- removed K410: LED, tronixio:zzHARWIN-M20-782104x, symbol tronixio:SYMBOL-HEADER-F-1X10
- removed LED401: KINGBRIGHT-DC10EWA, tronixio:KINGBRIGHT-DC, symbol tronixio:KINGBRIGHT-DC10EWA
- removed P401: AN1, tronixio:PIHER-PT10MV, symbol tronixio:PIHER-PT10MV-10K
- removed P402: AN2, tronixio:PIHER-PT10MV, symbol tronixio:PIHER-PT10MV-10K
- removed R401: PIHER-PT10LV-5K, tronixio:PIHER-PT10LV, symbol tronixio:PIHER-PT10LV-5K
- removed R402: 10R, tronixio:RESISTOR-1016-TH, symbol tronixio:R-0805
- removed RA401: BOURNS-4611X, tronixio:4611X, symbol tronixio:BOURNS-4611X-330R
- removed S401: S1, tronixio:CK-KSA-TH, symbol tronixio:CK-KSA
- removed S402: S3, tronixio:CK-KSA-TH, symbol tronixio:CK-KSA
- removed S403: BOURNS-PEC12R-24DENTS, tronixio:BOURNS-PEC12R, symbol tronixio:BOURNS-PEC12R-24DENTS
- removed S404: S2, tronixio:CK-KSA-TH, symbol tronixio:CK-KSA
- removed S405: S4, tronixio:CK-KSA-TH, symbol tronixio:CK-KSA
- added D301, D302, D303, D304: ST-ESDA14V2SC5Y, tronixio:SOT-23-5, symbol tronixio:ST-ESDA14V2SC5Y
- added K301: I2C/GPIO, tronixio:SAMTEC-SSW-106-02-T-S-RA, symbol tronixio:SAMTEC-SSW-106-02-T-S-RA
- added K302: I2C/SPI, tronixio:HARWIN-M20-974034x, symbol tronixio:HARWIN-254-M-2X03-RIGHT-ANGLE
- added K303: SPI/GPIO, tronixio:SAMTEC-SSW-106-02-T-D-RA, symbol tronixio:SAMTEC-SSW-106-02-T-D-RA
- added K304: EUSART/TTL, tronixio:SAMTEC-SSW-106-02-T-S-RA, symbol tronixio:SAMTEC-SSW-106-02-T-S-RA
- added R301, R302, R303, R304, R305, R306, R307, R308, R309, R310, R311, R312, R313, R314, R315, R316: 200Ω, tronixio:RESISTOR-1206, symbol tronixio:R-1206
Connections:
- net GND: now also D301.2 (A), D301.2 (A), D301.2 (A), D301.2 (A), D302.2 (A), D302.2 (A), D302.2 (A), D302.2 (A), D303.2 (A), D303.2 (A), D303.2 (A), D303.2 (A), D304.2 (A), D304.2 (A), D304.2 (A), D304.2 (A), K301.5, K303.10, K303.9, K304.5
- net VCC: now also K301.6, K303.11, K303.12, K304.6
- new net I2C_INT: D301.1 (C), K301.1, R301.2
- new net I2C_RESET: D301.5 (C), K301.2, R302.2
- new net I2C_SDA: D301.3 (C), K301.4, R304.2
- new net IC2_SCL: D301.4 (C), K301.3, R303.2
- new net RA0/SPI_CS3: R312.2
- new net RA1/SPI_CS2: R311.2
- new net RA2/SPI_RESET: R310.2
- new net RA3/SPI_INT: R309.2
- new net RA5/SPI_CS: R305.1
- new net RB4/URTS: R316.1
- new net RB5/UCTS: R313.1
- new net RC1/I2C_INT: R301.1
- new net RC2/I2C_RESET: R302.1
- new net RC3/SCK: K302.5, R308.1
- new net RC3/SCL: K302.1, R303.1
- new net RC3/SCL/SCK: K302.3
- new net RC4/MISO: K302.6, R307.1
- new net RC4/SDA: K302.2, R304.1
- new net RC4/SDA/MISO: K302.4
- new net RC5/MOSI: R306.1
- new net RC6/UTX: R314.1
- new net RC7/URX: R315.1
- new net SPI_CS: D302.1 (C), K303.1, R305.2
- new net SPI_CS2: D303.5 (C), K303.6, R311.1
- new net SPI_CS3: D303.4 (C), K303.8, R312.1
- new net SPI_INT: D302.5 (C), K303.2, R309.1
- new net SPI_MISO: D303.1 (C), K303.5, R307.2
- new net SPI_MOSI: D302.3 (C), K303.3, R306.2
- new net SPI_RESET: D302.4 (C), K303.4, R310.1
- new net SPI_SCK: D303.3 (C), K303.7, R308.2
- new net UART_CTS: D304.1 (C), K304.1, R313.2
- new net UART_RTS: D304.3 (C), K304.4, R316.2
- new net UART_RX: D304.4 (C), K304.3, R315.2
- new net UART_TX: D304.5 (C), K304.2, R314.2
Other:
- note added: "CTS"
- note added: "INT"
- note added: "RESET"
- note added: "RTS"
- note added: "RX"
- note added: "SCL"
- note added: "SDA"
- note added: "TX"
- note added: "VDD"
- note removed: "01"
- note removed: "02"
- note removed: "03"
- note removed: "04"
- note removed: "05"
- note removed: "06"
- note removed: "07"
- note removed: "08"
- note removed: "09"
- note removed: "10"
- note removed: "11"
- note removed: "12"
- note removed: "13"
- note removed: "14"
- note removed: "15"
- note removed: "16"
- note removed: "A"
- note removed: "AN1"
- note removed: "AN2"
- note removed: "B"
- note removed: "S1"
- note removed: "S2"
- note removed: "S3"
- note removed: "S4"
- note removed: "S5"
- title: Modules -> Module

Commit message: Update
Changed lines of the file:
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@@
     (effects (font (size 1.15 1.15)) (justify right bottom))
   )
-  (global_label "RC3{slash}SCK" (shape input) (at 83.82 132.08 180) (fields_autoplaced)
+  (global_label "RC3{slash}SCK" (shape bidirectional) (at 83.82 132.08 180) (fields_autoplaced)
     (effects (font (size 1.15 1.15)) (justify right))
     (property "Intersheet References" "${INTERSHEET_REFS}" (id 0) (at 73.4672 132.0081 0)
@@
     )
   )
-  (global_label "RC4{slash}MISO" (shape output) (at 129.54 96.52 180) (fields_autoplaced)
+  (global_label "RC4{slash}MISO" (shape bidirectional) (at 129.54 96.52 180) (fields_autoplaced)
     (effects (font (size 1.15 1.15)) (justify right))
     (property "Intersheet References" "${INTERSHEET_REFS}" (id 0) (at 118.4205 96.4481 0)
@@
     )
   )
-  (global_label "RC3{slash}SCK" (shape output) (at 152.4 96.52 0) (fields_autoplaced)
+  (global_label "RC3{slash}SCK" (shape bidirectional) (at 152.4 96.52 0) (fields_autoplaced)
     (effects (font (size 1.15 1.15)) (justify left))
     (property "Intersheet References" "${INTERSHEET_REFS}" (id 0) (at 162.7528 96.4481 0)
@@
     )
   )
-  (global_label "RC4{slash}MISO" (shape input) (at 83.82 129.54 180) (fields_autoplaced)
+  (global_label "RC4{slash}MISO" (shape bidirectional) (at 83.82 129.54 180) (fields_autoplaced)
     (effects (font (size 1.15 1.15)) (justify right))
     (property "Intersheet References" "${INTERSHEET_REFS}" (id 0) (at 72.7005 129.4681 0)
@@
   (symbol (lib_id "tronixio:HARWIN-254-M-2X03-RIGHT-ANGLE") (at 142.24 91.44 0) (mirror y) (unit 1)
     (in_bom yes) (on_board yes)
-    (property "Reference" "K302" (id 0) (at 140.97 86.36 0)
-      (effects (font (size 1.15 1.15)))
-    )
-    (property "Value" "I2C/SPI" (id 1) (at 140.97 88.9 0)
-      (effects (font (size 1.15 1.15)))
-    )
+    (property "Reference" "K302" (id 0) (at 140.97 88.9 0)
+      (effects (font (size 1.15 1.15)))
+    )
+    (property "Value" "I2C/SPI" (id 1) (at 140.97 99.06 0)
+      (effects (font (size 1.15 1.15)))
+    )

Commit message: Update
Parts:
- K301, K304: Name (none) -> SAMTEC-SSW-106-02-T-S-RA
- K302: Name (none) -> HARWIN-254-M-2X03-RIGHT-ANGLE
- K303: Name (none) -> SAMTEC-SSW-106-02-T-D-RA
- R301, R302, R303, R304, R305, R306, R307, R308, R309, R310, R311, R312, R313, R314, R315, R316: symbol tronixio:R-1206 -> tronixio:RESISTOR; Tolerance (none) -> 5%
Connections:
- net VCC renamed VDD

Commit message: Update
Parts:
- D301, D302, D303, D304: value ST-ESDA14V2SC5Y -> ESDA14V2SC5Y; Name ESDA14V2SC5Y -> ST-ESDA14V2SC5Y
- R301, R302, R303, R304, R305, R306, R307, R308, R309, R310, R311, R312, R313, R314, R315, R316: symbol tronixio:RESISTOR -> tronixio:RESISTOR-1206-200R; Mouser (none) -> 660-RK73B2BTTDD201J; Name (none) -> RESISTOR-1206-200R
