File: Kicad/trainer/pic8bit-mod.kicad_sch (KiCad schematic)
At the start: 24 parts, among them K301 I2C/GPIO, K302 I2C/SPI, K303 SPI/GPIO, K304 EUSART/TTL

Commit message: Update
Parts:
- D301, D302, D303, D304: symbol tronixio:ST-ESDA14V2SC5Y -> tronixio:ST-ESDA14V2SC5Y-SOT-23; Name ST-ESDA14V2SC5Y -> ST-ESDA14V2SC5Y-SOT-23
Changed lines of the file:
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@@
     (pin "1")
   )
-  (symbol (lib_id "tronixio:ST-ESDA14V2SC5Y") (at 121.92 152.4 0) (unit 1)
+  (symbol (lib_id "tronixio:ST-ESDA14V2SC5Y-SOT-23") (at 121.92 152.4 0) (unit 1)
     (in_bom yes) (on_board yes)
     (property "Reference" "D303" (id 0) (at 120.65 154.94 90)
@@
       (effects (font (size 1 1)) hide)
     )
-    (property "Name" "ST-ESDA14V2SC5Y" (id 5) (at 121.92 162.56 0)
+    (property "Name" "ST-ESDA14V2SC5Y-SOT-23" (id 5) (at 121.92 162.56 0)
       (effects (font (size 1 1)) hide)
     )
@@
     (pin "5")
   )
-  (symbol (lib_id "tronixio:ST-ESDA14V2SC5Y") (at 81.28 68.58 0) (unit 4)
+  (symbol (lib_id "tronixio:ST-ESDA14V2SC5Y-SOT-23") (at 81.28 68.58 0) (unit 4)
     (in_bom yes) (on_board yes)
     (property "Reference" "D301" (id 0) (at 80.01 71.12 90)
@@
       (effects (font (size 1 1)) hide)
     )
-    (property "Name" "ST-ESDA14V2SC5Y" (id 5) (at 81.28 78.74 0)
+    (property "Name" "ST-ESDA14V2SC5Y-SOT-23" (id 5) (at 81.28 78.74 0)
       (effects (font (size 1 1)) hide)
     )
@@
     (pin "2")
   )
-  (symbol (lib_id "tronixio:ST-ESDA14V2SC5Y") (at 228.6 68.58 0) (unit 1)
+  (symbol (lib_id "tronixio:ST-ESDA14V2SC5Y-SOT-23") (at 228.6 68.58 0) (unit 1)
     (in_bom yes) (on_board yes)
     (property "Reference" "D304" (id 0) (at 229.87 71.12 90)
@@
       (effects (font (size 1 1)) hide)
     )
-    (property "Name" "ST-ESDA14V2SC5Y" (id 5) (at 228.6 78.74 0)
+    (property "Name" "ST-ESDA14V2SC5Y-SOT-23" (id 5) (at 228.6 78.74 0)
       (effects (font (size 1 1)) hide)
     )
@@
     (pin "2")
   )
-  (symbol (lib_id "tronixio:ST-ESDA14V2SC5Y") (at 154.94 152.4 0) (unit 3)
+  (symbol (lib_id "tronixio:ST-ESDA14V2SC5Y-SOT-23") (at 154.94 152.4 0) (unit 3)
     (in_bom yes) (on_board yes)
     (property "Reference" "D303" (id 0) (at 156.21 154.94 90)
@@
       (effects (font (size 1 1)) hide)
     )
-    (property "Name" "ST-ESDA14V2SC5Y" (id 5) (at 154.94 162.56 0)
+    (property "Name" "ST-ESDA14V2SC5Y-SOT-23" (id 5) (at 154.94 162.56 0)
       (effects (font (size 1 1)) hide)
     )
@@
     (pin "5")
   )
-  (symbol (lib_id "tronixio:ST-ESDA14V2SC5Y") (at 170.18 152.4 0) (unit 4)
+  (symbol (lib_id "tronixio:ST-ESDA14V2SC5Y-SOT-23") (at 170.18 152.4 0) (unit 4)
     (in_bom yes) (on_board yes)
     (property "Reference" "D302" (id 0) (at 171.45 154.94 90)
@@
       (effects (font (size 1 1)) hide)
     )
-    (property "Name" "ST-ESDA14V2SC5Y" (id 5) (at 170.18 162.56 0)
+    (property "Name" "ST-ESDA14V2SC5Y-SOT-23" (id 5) (at 170.18 162.56 0)
       (effects (font (size 1 1)) hide)
     )
@@
     (pin "1")
   )
-  (symbol (lib_id "tronixio:ST-ESDA14V2SC5Y") (at 165.1 152.4 0) (unit 3)
+  (symbol (lib_id "tronixio:ST-ESDA14V2SC5Y-SOT-23") (at 165.1 152.4 0) (unit 3)
     (in_bom yes) (on_board yes)
     (property "Reference" "D302" (id 0) (at 166.37 154.94 90)
@@
       (effects (font (size 1 1)) hide)
     )
-    (property "Name" "ST-ESDA14V2SC5Y" (id 5) (at 165.1 162.56 0)
+    (property "Name" "ST-ESDA14V2SC5Y-SOT-23" (id 5) (at 165.1 162.56 0)
       (effects (font (size 1 1)) hide)
     )
@@
     (pin "1")
   )
-  (symbol (lib_id "tronixio:ST-ESDA14V2SC5Y") (at 91.44 68.58 0) (unit 2)
+  (symbol (lib_id "tronixio:ST-ESDA14V2SC5Y-SOT-23") (at 91.44 68.58 0) (unit 2)
     (in_bom yes) (on_board yes)
     (property "Reference" "D301" (id 0) (at 90.17 71.12 90)
@@
       (effects (font (size 1 1)) hide)
     )
-    (property "Name" "ST-ESDA14V2SC5Y" (id 5) (at 91.44 78.74 0)
+    (property "Name" "ST-ESDA14V2SC5Y-SOT-23" (id 5) (at 91.44 78.74 0)
       (effects (font (size 1 1)) hide)
     )
@@
     (pin "1")
   )
-  (symbol (lib_id "tronixio:ST-ESDA14V2SC5Y") (at 213.36 68.58 0) (unit 2)
+  (symbol (lib_id "tronixio:ST-ESDA14V2SC5Y-SOT-23") (at 213.36 68.58 0) (unit 2)
     (in_bom yes) (on_board yes)
     (property "Reference" "D304" (id 0) (at 214.63 71.12 90)
@@
       (effects (font (size 1 1)) hide)
     )
-    (property "Name" "ST-ESDA14V2SC5Y" (id 5) (at 213.36 78.74 0)
+    (property "Name" "ST-ESDA14V2SC5Y-SOT-23" (id 5) (at 213.36 78.74 0)
       (effects (font (size 1 1)) hide)
     )
@@
     (pin "1")
   )
-  (symbol (lib_id "tronixio:ST-ESDA14V2SC5Y") (at 111.76 152.4 0) (unit 1)
+  (symbol (lib_id "tronixio:ST-ESDA14V2SC5Y-SOT-23") (at 111.76 152.4 0) (unit 1)
     (in_bom yes) (on_board yes)
     (property "Reference" "D302" (id 0) (at 110.49 154.94 90)
@@
       (effects (font (size 1 1)) hide)
     )
-    (property "Name" "ST-ESDA14V2SC5Y" (id 5) (at 111.76 162.56 0)
+    (property "Name" "ST-ESDA14V2SC5Y-SOT-23" (id 5) (at 111.76 162.56 0)
       (effects (font (size 1 1)) hide)
     )
@@
     (pin "1")
   )
-  (symbol (lib_id "tronixio:ST-ESDA14V2SC5Y") (at 223.52 68.58 0) (unit 4)
+  (symbol (lib_id "tronixio:ST-ESDA14V2SC5Y-SOT-23") (at 223.52 68.58 0) (unit 4)
     (in_bom yes) (on_board yes)
     (property "Reference" "D304" (id 0) (at 224.79 71.12 90)
@@
       (effects (font (size 1 1)) hide)
     )
-    (property "Name" "ST-ESDA14V2SC5Y" (id 5) (at 223.52 78.74 0)
+    (property "Name" "ST-ESDA14V2SC5Y-SOT-23" (id 5) (at 223.52 78.74 0)
       (effects (font (size 1 1)) hide)
     )
@@
     (pin "5")
   )
-  (symbol (lib_id "tronixio:ST-ESDA14V2SC5Y") (at 76.2 68.58 0) (unit 1)
+  (symbol (lib_id "tronixio:ST-ESDA14V2SC5Y-SOT-23") (at 76.2 68.58 0) (unit 1)
     (in_bom yes) (on_board yes)
     (property "Reference" "D301" (id 0) (at 74.93 71.12 90)
@@
       (effects (font (size 1 1)) hide)
     )
-    (property "Name" "ST-ESDA14V2SC5Y" (id 5) (at 76.2 78.74 0)
+    (property "Name" "ST-ESDA14V2SC5Y-SOT-23" (id 5) (at 76.2 78.74 0)
       (effects (font (size 1 1)) hide)
     )
@@
     (pin "5")
   )
-  (symbol (lib_id "tronixio:ST-ESDA14V2SC5Y") (at 160.02 152.4 0) (unit 4)
+  (symbol (lib_id "tronixio:ST-ESDA14V2SC5Y-SOT-23") (at 160.02 152.4 0) (unit 4)
     (in_bom yes) (on_board yes)
     (property "Reference" "D303" (id 0) (at 161.29 154.94 90)
@@
       (effects (font (size 1 1)) hide)
     )
-    (property "Name" "ST-ESDA14V2SC5Y" (id 5) (at 160.02 162.56 0)
+    (property "Name" "ST-ESDA14V2SC5Y-SOT-23" (id 5) (at 160.02 162.56 0)
       (effects (font (size 1 1)) hide)
     )
@@
     (pin "5")
   )
-  (symbol (lib_id "tronixio:ST-ESDA14V2SC5Y") (at 127 152.4 0) (unit 2)
+  (symbol (lib_id "tronixio:ST-ESDA14V2SC5Y-SOT-23") (at 127 152.4 0) (unit 2)
     (in_bom yes) (on_board yes)
     (property "Reference" "D303" (id 0) (at 125.73 154.94 90)
@@
       (effects (font (size 1 1)) hide)
     )
-    (property "Name" "ST-ESDA14V2SC5Y" (id 5) (at 127 162.56 0)
+    (property "Name" "ST-ESDA14V2SC5Y-SOT-23" (id 5) (at 127 162.56 0)
       (effects (font (size 1 1)) hide)
     )
@@
     (pin "5")
   )
-  (symbol (lib_id "tronixio:ST-ESDA14V2SC5Y") (at 86.36 68.58 0) (unit 3)
+  (symbol (lib_id "tronixio:ST-ESDA14V2SC5Y-SOT-23") (at 86.36 68.58 0) (unit 3)
     (in_bom yes) (on_board yes)
     (property "Reference" "D301" (id 0) (at 85.09 71.12 90)
@@
       (effects (font (size 1 1)) hide)
     )
-    (property "Name" "ST-ESDA14V2SC5Y" (id 5) (at 86.36 78.74 0)
+    (property "Name" "ST-ESDA14V2SC5Y-SOT-23" (id 5) (at 86.36 78.74 0)
       (effects (font (size 1 1)) hide)
     )
@@
     (pin "2")
   )
-  (symbol (lib_id "tronixio:ST-ESDA14V2SC5Y") (at 116.84 152.4 0) (unit 2)
+  (symbol (lib_id "tronixio:ST-ESDA14V2SC5Y-SOT-23") (at 116.84 152.4 0) (unit 2)
     (in_bom yes) (on_board yes)
     (property "Reference" "D302" (id 0) (at 115.57 154.94 90)
@@
       (effects (font (size 1 1)) hide)
     )
-    (property "Name" "ST-ESDA14V2SC5Y" (id 5) (at 116.84 162.56 0)
+    (property "Name" "ST-ESDA14V2SC5Y-SOT-23" (id 5) (at 116.84 162.56 0)
       (effects (font (size 1 1)) hide)
     )
@@
     (pin "5")
   )
-  (symbol (lib_id "tronixio:ST-ESDA14V2SC5Y") (at 218.44 68.58 0) (unit 3)
+  (symbol (lib_id "tronixio:ST-ESDA14V2SC5Y-SOT-23") (at 218.44 68.58 0) (unit 3)
     (in_bom yes) (on_board yes)
     (property "Reference" "D304" (id 0) (at 219.71 71.12 90)
@@
       (effects (font (size 1 1)) hide)
     )
-    (property "Name" "ST-ESDA14V2SC5Y" (id 5) (at 218.44 78.74 0)
-      (effects (font (size 1 1)) hide)
-    )
+    (property "Name" "ST-ESDA14V2SC5Y-SOT-23" (id 5) (at 218.44 78.74 0)
+      (effects (font (size 1 1)) hide)
+    )

Commit message: Update
Parts:
- R301, R302, R303, R304, R305, R306, R307, R308, R309, R310, R311, R312, R313, R314, R315, R316: footprint tronixio:RESISTOR-1206 -> tronixio:RESISTOR-SMD-1206

Commit message: Update pic8bit trainer
Parts:
- D301, D302, D303, D304: Name ST-ESDA14V2SC5Y-SOT-23 -> (none)
- K301, K304: Name SAMTEC-SSW-106-02-T-S-RA -> (none)
- K302: Name HARWIN-254-M-2X03-RIGHT-ANGLE -> (none)
- K303: Name SAMTEC-SSW-106-02-T-D-RA -> (none)
- R301, R302, R303, R304, R305, R306, R307, R308, R309, R310, R311, R312, R313, R314, R315, R316: symbol tronixio:RESISTOR-1206-200R -> tronixio:KOASPEER-RK73B-1206-200R-5P; Name RESISTOR-1206-200R -> (none)
Other:
- title: Module -> Modules

Commit message: Up
Parts:
- R301, R302, R303, R304, R305, R306, R307, R308, R309, R310, R311, R312, R313, R314, R315, R316: symbol tronixio:KOASPEER-RK73B-1206-200R-5P -> tronixio:RESISTOR-1206-200R-5P
