File: Kicad/trainer/pic8bit-mod.kicad_sch (KiCad schematic)
At the start: 24 parts, among them K301 I2C/GPIO, K302 I2C/SPI, K303 SPI/GPIO, K304 EUSART/TTL

Commit message: Up
Connections:
- net VDD renamed +VDD

Commit message: Update Trainer Kicad 8
Connections:
- net +VDD renamed POWER-VDD
- net GND renamed POWER-GND

Commit message: Update Trainer
Changed lines of the file:
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@@
 		(on_board yes)
 		(dnp no)
-		(fields_autoplaced yes)
 		(property "Reference" "#PWR0126"
 			(at 236.22 45.72 0)
@@
 			)
 		)
-		(property "Description" ""
-			(at 236.22 35.56 0)
-			(effects
-				(font
-					(size 1.27 1.27)
-				)
-				(hide yes)
-			)
-		)
-		(property "Name" "VDD"
+		(property "Description" "VDD"
 			(at 236.22 30.48 0)
-			(do_not_autoplace yes)
 			(effects
 				(font
-					(size 1.15 1.15)
+					(size 1.27 1.27)
 				)
 			)
@@
 			)
 		)
-		(property "Description" ""
-			(at 134.62 116.84 0)
-			(effects
-				(font
-					(size 1.27 1.27)
-				)
-				(hide yes)
-			)
-		)
-		(property "Name" "VDD"
+		(property "Description" "VDD"
 			(at 134.62 111.76 0)
-			(do_not_autoplace yes)
 			(effects
 				(font
-					(size 1.15 1.15)
+					(size 1.27 1.27)
 				)
 			)
@@
 		(on_board yes)
 		(dnp no)
-		(fields_autoplaced yes)
 		(property "Reference" "#PWR0125"
 			(at 99.06 45.72 0)
@@
 			)
 		)
-		(property "Description" ""
-			(at 99.06 35.56 0)
-			(effects
-				(font
-					(size 1.27 1.27)
-				)
-				(hide yes)
-			)
-		)
-		(property "Name" "VDD"
+		(property "Description" "VDD"
 			(at 99.06 30.48 0)
-			(do_not_autoplace yes)
 			(effects
 				(font
-					(size 1.15 1.15)
+					(size 1.27 1.27)
 				)
 			)
@@
 		(on_board yes)
 		(dnp no)
-		(fields_autoplaced yes)
 		(property "Reference" "#PWR0138"
 			(at 147.32 127 0)
@@
 			)
 		)
-		(property "Description" ""
-			(at 147.32 116.84 0)
-			(effects
-				(font
-					(size 1.27 1.27)
-				)
-				(hide yes)
-			)
-		)
-		(property "Name" "VDD"
+		(property "Description" "VDD"
 			(at 147.32 111.76 0)
-			(do_not_autoplace yes)
 			(effects
 				(font
-					(size 1.15 1.15)
+					(size 1.27 1.27)
 				)
 			)

Commit message: Up
Parts:
- K301, K304: symbol tronixio:SAMTEC-SSW-106-02-T-S-RA -> tronixio:SAMTEC-254-F-1X06-RIGHT-ANGLE; Mouser 200-SSW10602TSRA -> 200-SSW10603TSRA
- K303: symbol tronixio:SAMTEC-SSW-106-02-T-D-RA -> tronixio:SAMTEC-254-F-2X06-RIGHT-ANGLE
Changed lines of the file:
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@@
 	)
 	(symbol
-		(lib_id "tronixio:SAMTEC-SSW-106-02-T-S-RA")
+		(lib_id "tronixio:SAMTEC-254-F-1X06-RIGHT-ANGLE")
 		(at 241.3 43.18 0)
 		(unit 1)
@@
 			)
 		)
-		(property "Mouser" "200-SSW10602TSRA"
+		(property "Mouser" "200-SSW10603TSRA"
 			(at 241.3 66.04 0)
 			(do_not_autoplace yes)
@@
 	)
 	(symbol
-		(lib_id "tronixio:SAMTEC-SSW-106-02-T-S-RA")
+		(lib_id "tronixio:SAMTEC-254-F-1X06-RIGHT-ANGLE")
 		(at 104.14 43.18 0)
 		(unit 1)
@@
 			)
 		)
-		(property "Mouser" "200-SSW10602TSRA"
+		(property "Mouser" "200-SSW10603TSRA"
 			(at 104.14 66.04 0)
 			(do_not_autoplace yes)
@@
 	)
 	(symbol
-		(lib_id "tronixio:SAMTEC-SSW-106-02-T-D-RA")
+		(lib_id "tronixio:SAMTEC-254-F-2X06-RIGHT-ANGLE")
 		(at 139.7 124.46 0)
 		(unit 1)
