File: Kicad/trainer/pic8bit.kicad_pcb (KiCad board)
At the start: 2 copper layers, 160 x 100 mm, 97 parts, among them IC101 NCP5662-ADJ, IC201 MICROCHIP-PIC16F1778-ISP, K101 AC/DC 9-12V, K102 AC/DC 9-12V, K103 PE-450-4X6X-BLACK, K201 MCU 1, K202 MCU 2, K203 ICSP, K301 I2C/GPIO, K302 I2C/SPI, K303 SPI/GPIO, K304 EUSART/TTL, K401 VIN, K402 SYMBOL-HEADER-F-1X10, K403 VIN, K404 VDD, K405 GND, K406 VDD, K407 GND, K408 SYMBOL-HEADER-F-1X10, K409 HARWIN-254-F-1X16-VERTICAL, K410 LED, P401 AN1, P402 AN2, U101 KEYSTONE-24283, U102 KEYSTONE-24283, U103 KEYSTONE-24283, U104 KEYSTONE-24283, X101 3M-SJ5376, X102 3M-SJ5376, X103 3M-SJ5376, X104 3M-SJ5376, X105 3M-SJ5376

Commit message: Update
Parts:
- B101: value DF01M -> ONSEMI-DF01M
- C203: value 100n -> C-0805
- IC101: value NCP5662-ADJ -> NCP5662-ADJ-TO263
- K302: value I2C/SPI -> HARWIN-254-M-2X03-RIGHT-ANGLE
- S403: value PEC12R-24DENTS -> BOURNS-PEC12R-24DENTS
- TP103: value GND -> KEYSTONE-2000-3; footprint tronixio:KEYSTONE-5006 -> tronixio:KEYSTONE-2000-3
- moved TP103 94.6 mm to (183.0, 50.5), turned to 0 degrees
- moved TP102 93.8 mm to (200.5, 143.5)
- moved TP101 30.0 mm to (213.0, 50.5)
- moved K302 2.54 mm to (79.5, 108.9)
Connections:
- K302 pad 1: RC4/SDA -> RC3/SCL
- K302 pad 2: /MCU/RC4/SDA/MISO -> RC4/SDA
- K302 pad 3: RC4/MISO -> /MCU/RC3/SCL/SCK
- K302 pad 4: RC3/SCL -> /MCU/RC4/SDA/MISO
- K302 pad 5: /MCU/RC3/SCL/SCK -> RC3/SCK
- K302 pad 6: RC3/SCK -> RC4/MISO
- K303 pad 10: /MOD/SPI_CS3 -> GND
- K303 pad 11: GND -> VCC
- K303 pad 2: /MOD/SPI_MOSI -> /MOD/SPI_INT
- K303 pad 3: /MOD/SPI_MISO -> /MOD/SPI_MOSI
- K303 pad 4: /MOD/SPI_SCK -> /MOD/SPI_RESET
- K303 pad 5: GND -> /MOD/SPI_MISO
- K303 pad 6: VCC -> /MOD/SPI_CS2
- K303 pad 7: /MOD/SPI_INT -> /MOD/SPI_SCK
- K303 pad 8: /MOD/SPI_RESET -> /MOD/SPI_CS3
- K303 pad 9: /MOD/SPI_CS2 -> GND
Routing:
- net Net-(IC101-Pad5): track 15.5 -> 16.1 mm

Commit message: Up
Parts:
- removed *X1: XTAL-DIL08, tronixio:DIP-08-W762-SOCKET
- removed IC101: NCP5662-ADJ-TO263, tronixio:TO-263-5
- removed IC201: MICROCHIP-PIC16F1778-ISP, tronixio:DIP-28-W762-SOCKET
- added U105: NCP5662-ADJ-TO263, tronixio:TO-263-5, F.Cu at (107.0, 61.0)
- added U201: MICROCHIP-PIC16F1778-ISP, tronixio:DIP-28-W762-SOCKET, F.Cu at (168.6, 88.6)
- added X1: XTAL-DIL08, tronixio:DIP-08-W762-SOCKET, F.Cu at (168.5, 77.0)
- added kibuzzard-62A777FA: G***, kibuzzard-62A777FA, F.Cu at (212.5, 77.8)
- added kibuzzard-62A777FA: G***, kibuzzard-62A777FA, F.Cu at (183.0, 53.0)
- added kibuzzard-62A777FA: G***, kibuzzard-62A777FA, F.Cu at (200.5, 140.5)
- added kibuzzard-62A777FA: G***, kibuzzard-62A777FA, F.Cu at (147.8, 51.8)
- added kibuzzard-62A777FA: G***, kibuzzard-62A777FA, F.Cu at (213.0, 53.5)
- added kibuzzard-62A77857: G***, kibuzzard-62A77857, F.Cu at (190.5, 77.8)
- added kibuzzard-62A778D1: G***, kibuzzard-62A778D1, F.Cu at (200.2, 133.0)
- added kibuzzard-62A778D1: G***, kibuzzard-62A778D1, F.Cu at (200.3, 60.5)
- added kibuzzard-62A778F0: G***, kibuzzard-62A778F0, F.Cu at (202.9, 60.5)
- added kibuzzard-62A77FCE: G***, kibuzzard-62A77FCE, F.Cu at (135.8, 51.8)
- added kibuzzard-62A77FF4: G***, kibuzzard-62A77FF4, F.Cu at (159.8, 51.8)
- added kibuzzard-62A78037: G***, kibuzzard-62A78037, F.Cu at (213.5, 67.0)
- added kibuzzard-62A78078: G***, kibuzzard-62A78078, F.Cu at (213.5, 69.5)
- added kibuzzard-62A780A0: G***, kibuzzard-62A780A0, F.Cu at (80.5, 115.2)
- added kibuzzard-62A780A0: G***, kibuzzard-62A780A0, F.Cu at (83.0, 87.3)
- added kibuzzard-62A780A0: G***, kibuzzard-62A780A0, F.Cu at (80.5, 117.8)
- added kibuzzard-62A780B6: G***, kibuzzard-62A780B6, F.Cu at (83.0, 84.8)
- C203: value C-0805 -> 100n
- K201, K202: footprint tronixio:zzHARWIN-M20-782144x -> tronixio:HARWIN-M20-782144x
- K302: value HARWIN-254-M-2X03-RIGHT-ANGLE -> I2C/SPI
- R301, R302, R303, R304, R305, R306, R307, R308, R309, R310, R311, R312, R313, R314, R315, R316: value 200R -> 200Ω
- R402: value 10R -> 10Ω
Connections:
- net /MOD/I2C_INT renamed /Module/I2C_INT
- net /MOD/I2C_RESET renamed /Module/I2C_RESET
- net /MOD/I2C_SDA renamed /Module/I2C_SDA
- net /MOD/IC2_SCL renamed /Module/IC2_SCL
- net /MOD/SPI_CS renamed /Module/SPI_CS
- net /MOD/SPI_CS2 renamed /Module/SPI_CS2
- net /MOD/SPI_CS3 renamed /Module/SPI_CS3
- net /MOD/SPI_INT renamed /Module/SPI_INT
- net /MOD/SPI_MISO renamed /Module/SPI_MISO
- net /MOD/SPI_MOSI renamed /Module/SPI_MOSI
- net /MOD/SPI_RESET renamed /Module/SPI_RESET
- net /MOD/SPI_SCK renamed /Module/SPI_SCK
- net /MOD/UART_CTS renamed /Module/UART_CTS
- net /MOD/UART_RTS renamed /Module/UART_RTS
- net /MOD/UART_RX renamed /Module/UART_RX
- net /MOD/UART_TX renamed /Module/UART_TX
Routing:
- net GND: track 75.7 -> 65.5 mm
Other:
- board text removed: "GND"
- board text removed: "VIN"

Commit message: Up
Parts:
- added C401: 10n, tronixio:zzzKEMET-C315, F.Cu at (143.0, 126.0)
- added C402: 10n, tronixio:zzzKEMET-C315, F.Cu at (154.0, 126.0)
- added R403: 10K, tronixio:RESISTOR-1016-TH, F.Cu at (126.0, 122.0)
- added R404: 10K, tronixio:RESISTOR-1016-TH, F.Cu at (134.0, 122.0)
- added R405: 10K, tronixio:RESISTOR-1016-TH, F.Cu at (147.0, 122.0)
- added R406: 10K, tronixio:RESISTOR-1016-TH, F.Cu at (151.0, 122.0)
- added R407: 10K, tronixio:RESISTOR-1016-TH, F.Cu at (138.0, 122.0)
- added R408: 10K, tronixio:RESISTOR-1016-TH, F.Cu at (130.0, 122.0)
Connections:
- net /HID/A renamed /HID/ROTARY_A
- net /HID/B renamed /HID/ROTARY_B
Routing:
- net /HID/S1: track 125.1 -> 170.4 mm
- net VCC: track 410.4 -> 451.2 mm
- net /HID/ROTARY_A: track 38.6 -> 76.7 mm
- net /HID/ROTARY_B: track 36.1 -> 73.7 mm
- net /HID/S2: track 105.2 -> 131.5 mm
- net /HID/S4: track 64.1 -> 80.3 mm
- net /HID/S3: track 85.2 -> 98.5 mm
- net GND: track 65.5 -> 75.7 mm
- net RC4/MISO: track 22.1 -> 22.9 mm
- net RC3/SCK: track 24.3 -> 25.0 mm
- net /MCU/RC4/SDA/MISO: track 210.7 -> 211.2 mm

Commit message: Update
Parts:
- removed K401: VIN, tronixio:zzHARWIN-M20-782044x
- removed K403: VIN, tronixio:HARWIN-M20-999044x
- removed K404: VDD, tronixio:zzHARWIN-M20-782044x
- removed K405: GND, tronixio:zzHARWIN-M20-782044x
- removed K406: VDD, tronixio:HARWIN-M20-999044x
- removed K407: GND, tronixio:HARWIN-M20-999044x
- removed K408: SYMBOL-HEADER-F-1X10, tronixio:zzHARWIN-M20-782104x
- removed the kibuzzard-62A780A0 at (80.5, 115.2)
- added K204: VIN, tronixio:zzHARWIN-M20-782044x, F.Cu at (132.0, 54.0)
- added K205: VIN, tronixio:HARWIN-M20-999044x, F.Cu at (132.0, 49.5)
- added K206: VDD, tronixio:zzHARWIN-M20-782044x, F.Cu at (156.0, 54.0)
- added K207: GND, tronixio:zzHARWIN-M20-782044x, F.Cu at (144.0, 54.0)
- added K208: VDD, tronixio:HARWIN-M20-999044x, F.Cu at (156.0, 49.5)
- added K209: GND, tronixio:HARWIN-M20-999044x, F.Cu at (144.0, 49.5)
- added K210: SYMBOL-HEADER-F-1X10, tronixio:zzHARWIN-M20-782104x, F.Cu at (190.1, 80.7)
- added R409: 10K, tronixio:RESISTOR-1016-TH, F.Cu at (144.5, 129.2)
- added TP104: KEYSTONE-2000-3, tronixio:KEYSTONE-2000-3, F.Cu at (187.0, 50.5)
- added kibuzzard-62A777FA: G***, kibuzzard-62A777FA, F.Cu at (187.0, 53.0)
- added kibuzzard-62A777FA: G***, kibuzzard-62A777FA, F.Cu at (224.5, 111.4)
- added kibuzzard-62AA3F24: G***, kibuzzard-62AA3F24, F.Cu at (80.5, 115.2)
- added kibuzzard-62ACBAD0: G***, kibuzzard-62ACBAD0, F.Cu at (224.5, 108.9)
- added kibuzzard-62ACDA78: G***, kibuzzard-62ACDA78, F.Cu at (113.5, 51.0)
- TP103: value KEYSTONE-2000-3 -> GND; footprint tronixio:KEYSTONE-2000-3 -> tronixio:KEYSTONE-5006
- moved R406 31.5 mm to (120.3, 129.2)
- moved R405 30.1 mm to (117.8, 129.2)
- moved R404 20.1 mm to (115.3, 129.2)
- moved R403 15.1 mm to (112.7, 129.2)
- moved R408 13.9 mm to (141.9, 129.2)
- moved R407 11.5 mm to (147.0, 129.2)
- moved C402 8.89 mm to (150.8, 134.3), turned to 0 degrees
- moved C401 8.04 mm to (150.8, 124.1), turned to 0 degrees
- moved TP103 2.00 mm to (181.0, 50.5), turned to 90 degrees
- moved kibuzzard-62A777FA 2.00 mm to (181.0, 53.0)
- moved G*** 1.00 mm to (119.0, 89.0)
- moved S201 0.94 mm to (190.2, 141.9)
- moved B101 0.50 mm to (85.2, 56.5)
- moved S401 0.25 mm to (82.2, 141.9)
- moved S405 0.20 mm to (150.8, 141.9)
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Connections:
- C401 pad 1: /HID/ROTARY_A -> /HID/A
- C402 pad 1: /HID/ROTARY_B -> /HID/B
- K402 pad 7: /HID/ROTARY_A -> /HID/A
- K402 pad 8: /HID/ROTARY_B -> /HID/B
- R404 pad 2: /HID/S3 -> /HID/S2
- R405 pad 2: /HID/ROTARY_A -> /HID/S3
- R406 pad 2: /HID/ROTARY_B -> /HID/S4
- R407 pad 2: /HID/S4 -> /HID/S5
- R408 pad 2: /HID/S2 -> /HID/A
- S403 pad 1: /HID/ROTARY_A -> /HID/A
- S403 pad 3: /HID/ROTARY_B -> /HID/B
Routing:
- net /HID/A: track 0.00 -> 91.6 mm
- net /HID/B: track 0.00 -> 86.8 mm
- net /HID/ROTARY_A: track 76.7 -> 0.00 mm
- net /HID/ROTARY_B: track 73.7 -> 0.00 mm
- net /HID/S1: track 170.4 -> 116.9 mm
- net /HID/S4: track 80.3 -> 124.2 mm, vias 0 -> 1
- net VCC: track 451.2 -> 484.0 mm
- net /HID/S2: track 131.5 -> 100.3 mm, vias 0 -> 1
- net /HID/S5: track 32.0 -> 59.9 mm
- net /MCU/RC5/MOSI: track 150.7 -> 155.4 mm
- net /HID/S3: track 98.5 -> 102.1 mm, vias 0 -> 1
- net /MCU/~{MCLR}: track 90.3 -> 91.5 mm
- net Net-(EB401-Pad15): track 23.3 -> 24.4 mm
- net Net-(C201-Pad1): track 85.5 -> 86.5 mm
- net VIN: track 81.6 -> 82.1 mm
Other:
- board text added: "RA2/RST - RC5/MOSI"
- board text added: "RC2/RST"
- board text removed: "RA2/RESET - RC5/MOSI"
- board text removed: "RC2/RESET"
- board text removed: "VDD"

Commit message: Update
Parts:
- S403: footprint tronixio:BOURNS-PEC12R -> tronixio:BOURNS-PEC12R-SWITCH
Changed lines of the file:
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@@
     )
   )
-  (footprint "tronixio:BOURNS-PEC12R" (layer "F.Cu")
+  (footprint "tronixio:BOURNS-PEC12R-SWITCH" (layer "F.Cu")
     (at 175.585 136.84)
+    (descr "https://www.bourns.com/resources/design-tools/engineering-files-list?Folder=PEC12R")
     (property "Mouser" "652-PEC12R-4215F-S24")
     (property "Sheetfile" "pic8bit-hid.kicad_sch")
     (property "Sheetname" "HID")
     (attr through_hole)
-    (fp_text reference "S403" (at 0 -5) (layer "F.Fab")
+    (fp_text reference "S403" (at 0 -10.16) (layer "F.Fab")
       (effects (font (size 1 1) (thickness 0.15)))
     )
-    (fp_text value "BOURNS-PEC12R-24DENTS" (at 0 -9) (layer "F.Fab")
+    (fp_text value "BOURNS-PEC12R-24DENTS" (at 0 10.16) (layer "F.Fab")
       (effects (font (size 1 1) (thickness 0.15)))
     )
+    (fp_line (start -6.2 6.7) (end -3.6 6.7) (layer "F.SilkS") (width 0.12))
+    (fp_line (start 3.8 -6.7) (end 6.2 -6.7) (layer "F.SilkS") (width 0.12))
+    (fp_line (start 6.2 -6.7) (end 6.2 -1.9) (layer "F.SilkS") (width 0.12))
+    (fp_line (start -6.2 -6.7) (end -3.8 -6.7) (layer "F.SilkS") (width 0.12))
+    (fp_line (start -6.2 1.9) (end -6.2 6.7) (layer "F.SilkS") (width 0.12))
+    (fp_line (start -6.2 -6.7) (end -6.2 -1.9) (layer "F.SilkS") (width 0.12))
+    (fp_line (start 3.6 6.7) (end 6.2 6.7) (layer "F.SilkS") (width 0.12))
+    (fp_line (start 6.2 1.9) (end 6.2 6.7) (layer "F.SilkS") (width 0.12))
+    (fp_line (start -1.2 -6.7) (end 1.2 -6.7) (layer "F.SilkS") (width 0.12))
     (fp_rect (start -7.7 8.6) (end 7.7 -8.1) (layer "F.CrtYd") (width 0.05) (fill none))
     (fp_line (start -2 1.5) (end -1.8 1) (layer "F.Fab") (width 0.1))
+    (fp_line (start -1.8 1) (end 1.8 1) (layer "F.Fab") (width 0.1))
     (fp_line (start 2 1.5) (end 1.8 1) (layer "F.Fab") (width 0.1))
     (fp_line (start -2 1.5) (end 2 1.5) (layer "F.Fab") (width 0.1))
-    (fp_line (start -1.8 1) (end 1.8 1) (layer "F.Fab") (width 0.1))
+    (fp_rect (start -3 7.1) (end -2 6.7) (layer "F.Fab") (width 0.1) (fill solid))
+    (fp_rect (start 6.2 1.25) (end 7 -1.25) (layer "F.Fab") (width 0.1) (fill solid))
+    (fp_rect (start -6.2 6.7) (end 6.2 -6.7) (layer "F.Fab") (width 0.1) (fill none))
+    (fp_rect (start -3 -6.7) (end -2 -7.1) (layer "F.Fab") (width 0.1) (fill solid))
+    (fp_rect (start 2 7.1) (end 3 6.7) (layer "F.Fab") (width 0.1) (fill solid))
     (fp_rect (start -0.5 7.1) (end 0.5 6.7) (layer "F.Fab") (width 0.1) (fill solid))
-    (fp_rect (start -3 7.1) (end -2 6.7) (layer "F.Fab") (width 0.1) (fill solid))
-    (fp_rect (start -6.2 6.7) (end 6.2 -6.7) (layer "F.Fab") (width 0.1) (fill none))
     (fp_rect (start -7 1.25) (end -6.2 -1.25) (layer "F.Fab") (width 0.1) (fill solid))
-    (fp_rect (start 6.2 1.25) (end 7 -1.25) (layer "F.Fab") (width 0.1) (fill solid))
-    (fp_rect (start 2 7.1) (end 3 6.7) (layer "F.Fab") (width 0.1) (fill solid))
     (fp_rect (start 2 -6.7) (end 3 -7.1) (layer "F.Fab") (width 0.1) (fill solid))
-    (fp_rect (start -3 -6.7) (end -2 -7.1) (layer "F.Fab") (width 0.1) (fill solid))
     (fp_arc (start -1.8 1) (mid 0 -2.046667) (end 1.8 1) (layer "F.Fab") (width 0.1))
     (fp_circle (center 5.3 6) (end 5.6 6) (layer "F.Fab") (width 0.1) (fill none))
     (fp_circle (center 5.3 -5.5) (end 5.6 -5.5) (layer "F.Fab") (width 0.1) (fill none))
+    (fp_circle (center -5.3 -5.5) (end -5 -5.5) (layer "F.Fab") (width 0.1) (fill none))
+    (fp_circle (center -5.3 6) (end -5 6) (layer "F.Fab") (width 0.1) (fill none))
+    (fp_circle (center 0 0) (end 2.5 0) (layer "F.Fab") (width 0.1) (fill none))
     (fp_circle (center 0 0) (end 3.5 0) (layer "F.Fab") (width 0.1) (fill none))
-    (fp_circle (center 0 0) (end 2.5 0) (layer "F.Fab") (width 0.1) (fill none))
-    (fp_circle (center -5.3 6) (end -5 6) (layer "F.Fab") (width 0.1) (fill none))
-    (fp_circle (center -5.3 -5.5) (end -5 -5.5) (layer "F.Fab") (width 0.1) (fill none))
-    (pad "1" thru_hole circle locked (at -2.5 7.5) (size 1.8 1.8) (drill 1) (layers *.Cu *.Mask)
+    (pad "1" thru_hole circle (at -2.5 7.5) (size 2 2) (drill 1) (layers *.Cu *.Mask)
       (net 105 "/HID/A") (pinfunction "A") (pintype "passive"))
-    (pad "2" thru_hole rect locked (at -6.5 0) (size 2 3.2) (drill oval 1 2.4) (layers *.Cu *.Mask)
-      (net 1 "GND") (pinfunction "C") (pintype "passive"))
-    (pad "2" thru_hole circle locked (at 0 7.5) (size 1.8 1.8) (drill 1) (layers *.Cu *.Mask)
-      (net 1 "GND") (pinfunction "C") (pintype "passive"))
-    (pad "2" thru_hole rect locked (at 6.5 0) (size 2 3.2) (drill oval 1 2.4) (layers *.Cu *.Mask)
-      (net 1 "GND") (pinfunction "C") (pintype "passive"))
-    (pad "3" thru_hole circle locked (at 2.5 7.5) (size 1.8 1.8) (drill 1) (layers *.Cu *.Mask)
+    (pad "2" thru_hole circle (at 0 7.5) (size 2 2) (drill 1) (layers *.Cu *.Mask)
+      (net 1 "GND") (pintype "passive"))
+    (pad "2" thru_hole rect (at 6.5 0) (size 2 3.2) (drill oval 1 2.4) (layers *.Cu *.Mask)
+      (net 1 "GND") (pintype "passive"))
+    (pad "2" thru_hole rect (at -6.5 0) (size 2 3.2) (drill oval 1 2.4) (layers *.Cu *.Mask)
+      (net 1 "GND") (pintype "passive"))
+    (pad "3" thru_hole circle (at 2.5 7.5) (size 2 2) (drill 1) (layers *.Cu *.Mask)
       (net 106 "/HID/B") (pinfunction "B") (pintype "passive"))
-    (pad "4" thru_hole circle locked (at 2.5 -7) (size 1.8 1.8) (drill 1) (layers *.Cu *.Mask)
-      (net 1 "GND") (pinfunction "2") (pintype "passive"))
-    (pad "5" thru_hole circle locked (at -2.5 -7) (size 1.8 1.8) (drill 1) (layers *.Cu *.Mask)
-      (net 99 "/HID/S5") (pinfunction "1") (pintype "passive"))
-    (model "${KICAD6_USER_3DMODEL_DIR}/Discret/BOURNS-PEC12R.step"
+    (pad "4" thru_hole circle (at 2.5 -7) (size 2 2) (drill 1) (layers *.Cu *.Mask)
+      (net 1 "GND") (pintype "passive"))
+    (pad "5" thru_hole circle (at -2.5 -7) (size 2 2) (drill 1) (layers *.Cu *.Mask)
+      (net 99 "/HID/S5") (pintype "passive"))
+    (model "${KICAD6_USER_3DMODEL_DIR}/Switch/BOURNS-PEC12R-SWITCH.step"
       (offset (xyz 0 0 0))
       (scale (xyz 1 1 1))

Commit message: Up
Parts:
- removed C401, C402: 10n, tronixio:zzzKEMET-C315
- removed R403, R404, R405, R406, R407, R408, R409: 10K, tronixio:RESISTOR-1016-TH
Routing:
- net VCC: track 484.0 -> 410.4 mm
- net /HID/S4: track 124.2 -> 64.3 mm, vias 1 -> 0
- net /HID/A: track 91.6 -> 40.0 mm
- net /HID/B: track 86.8 -> 37.5 mm
- net /HID/S5: track 59.9 -> 32.0 mm
- net /HID/S3: track 102.1 -> 85.3 mm, vias 1 -> 0
- net /HID/S1: track 116.9 -> 125.4 mm
- net /HID/S2: track 100.3 -> 105.4 mm, vias 1 -> 0

Commit message: Update
Parts:
- C201, C203: footprint tronixio:zzzKEMET-C315 -> tronixio:KEMET-C315
- EB401: footprint tronixio:zzzTRONIXIO-EXPANSION-BOARD -> tronixioZZZ:TRONIXIO-EXPANSION-BOARD
- K204, K206, K207: footprint tronixio:zzHARWIN-M20-782044x -> tronixio:HARWIN-M20-782044x
- K210, K402, K410: footprint tronixio:zzHARWIN-M20-782104x -> tronixio:HARWIN-M20-782104x
- K409: footprint tronixio:zzHARWIN-M20-782164x -> tronixio:HARWIN-M20-782164x
- moved R101 5.08 mm to (103.5, 51.0), turned to 0 degrees
- moved kibuzzard-62A777FA 0.25 mm to (187.0, 53.2)
- moved kibuzzard-62A777FA 0.25 mm to (181.0, 53.2)
- moved kibuzzard-62A777FA 0.25 mm to (213.0, 53.2)
Connections:
- net VCC renamed VDD
Routing:
- net VDD: track 410.4 -> 405.3 mm
Other:
- board text added: "GND"
- board text removed: "VSS"

Commit message: Update
Parts:
- removed K410: LED, tronixio:HARWIN-M20-782104x
- added K401: HARWIN-254-F-1X10-VERTICAL, tronixio:HARWIN-M20-782104x, F.Cu at (142.0, 73.0)
- B101: value ONSEMI-DF01M -> DF01M
- C101, C102: value UVZ-220U-25V -> 220µ/25V
- D301, D302, D303, D304: value ST-ESDA14V2SC5Y -> ESDA14V2SC5Y
- EB401: value TRONIXIO-EXPANSION-BOARD -> EXPANSION-BOARD; footprint tronixioZZZ:TRONIXIO-EXPANSION-BOARD -> tronixio:TRONIXIO-EXPANSION-BOARD
- K210, K402: value SYMBOL-HEADER-F-1X10 -> HARWIN-254-F-1X10-VERTICAL
- R401: value PIHER-PT10LV-5K -> 5K
- RA401: value BOURNS-4611X -> 330Ω
- TP104: value KEYSTONE-2000-3 -> GND
- U101, U102, U103, U104: footprint tronixio:zzzKEYSTONE-24283 -> tronixio:KEYSTONE-24283
- U105: value NCP5662-ADJ-TO263 -> NCP5662-ADJ
- X101, X102, X103, X104, X105: footprint tronixio:zzz3M-SJ5376 -> tronixio:3M-SJ5376
- moved K303 2.54 mm to (79.5, 97.5)
