File: Kicad/trainer/pic8bit.kicad_pcb (KiCad board)
At the start: 2 copper layers, 160 x 100 mm, 119 parts, among them K101 AC/DC 9-12V, K102 AC/DC 9-12V, K103 PE-450-4X6X-BLACK, K201 MCU 1, K202 MCU 2, K203 ICSP, K204 VIN, K205 VIN, K206 VDD, K207 GND, K208 VDD, K209 GND, K210 HARWIN-254-F-1X10-VERTICAL, K301 I2C/GPIO, K302 I2C/SPI, K303 SPI/GPIO, K304 EUSART/TTL, K401 HARWIN-254-F-1X10-VERTICAL, K402 HARWIN-254-F-1X10-VERTICAL, K409 HARWIN-254-F-1X16-VERTICAL, P401 AN1, P402 AN2, U101 KEYSTONE-24283, U102 KEYSTONE-24283, U103 KEYSTONE-24283, U104 KEYSTONE-24283, U105 NCP5662-ADJ, U201 MICROCHIP-PIC16F1778-ISP, X1 XTAL-DIL08, X101 3M-SJ5376, X102 3M-SJ5376, X103 3M-SJ5376, X104 3M-SJ5376, X105 3M-SJ5376

Commit message: Update
Parts:
- U201: value MICROCHIP-PIC16F1778-ISP -> PIC16F/18F

Commit message: Update
Parts:
- LED101: footprint tronixio:LED-05MM-TH -> tronixio:LED-TH-05MM
- R102, R201, R202, R203, R204, R402: footprint tronixio:RESISTOR-1016-TH -> tronixio:RESISTOR-TH-1016
- R301, R302, R303, R304, R305, R306, R307, R308, R309, R310, R311, R312, R313, R314, R315, R316: footprint tronixio:RESISTOR-1206 -> tronixio:RESISTOR-SMD-1206
- U201: footprint tronixio:DIP-28-W762-SOCKET -> tronixio:DIP-28-W762

Commit message: Update
Parts:
- C101, C102: footprint tronixio:CAPACITOR-ELECTROLYTIC-RADIAL-080-115-035 -> tronixio:CAPACITOR-ELECTROLYTIC-RADIAL-080-110-035
Connections:
- net /MCU/PGC renamed PGC
- net /MCU/PGD renamed PGD
- net /MCU/~{MCLR} renamed ~{MCLR}

Commit message: Update
Parts:
- removed X1: XTAL-DIL08, tronixio:DIP-08-W762-SOCKET
- added X201: XTAL-DIL08, tronixio:DIP-08-W762-SOCKET, F.Cu at (168.5, 77.0)
Connections:
- net PGC renamed Net-(K202-Pad2)
- net PGD renamed Net-(K202-Pad1)
- net ~{MCLR} renamed Net-(K201-Pad1)
Other:
- board text added: "X"
- board text removed: "X1"

Commit message: Update pic8bit trainer
Parts:
- RA401: footprint tronixio:4611X -> tronixio:BOURNS-4611X
