File: Kicad/trainer/pic8bit.kicad_sch (KiCad schematic)
At the start: 30 parts, among them IC101 NCP5662-ADJ, K101 AC/DC 9-12V, K102 AC/DC 9-12V, K103 PE-450-4X6X-BLACK, U101 KEYSTONE-24283, U102 KEYSTONE-24283, U103 KEYSTONE-24283, U104 KEYSTONE-24283, X101 3M-SJ5376, X102 3M-SJ5376, X103 3M-SJ5376, X104 3M-SJ5376, X105 3M-SJ5376

Commit message: Update
Parts:
- removed R101: 5K, tronixio:TRIMMER-64W, symbol tronixio:VISHAY-64W
- removed TP103: GND, tronixio:KEYSTONE-5006, symbol tronixio:KEYSTONE-5006
- added R101: 5K, tronixio:TRIMMER-64W, symbol tronixio:VISHAY-5K-64W
- added TP103: KEYSTONE-2000-3, tronixio:KEYSTONE-2000-3, symbol tronixio:KEYSTONE-2000-3
- B101: MOUSER 512-DF01M -> (none); Mouser (none) -> 512-DF01M; NAME DF01M -> (none); Name (none) -> DF01M
- C101, C102: MOUSER 647-UVZ1E221MPD -> (none); Mouser (none) -> 647-UVZ1E221MPD
- H101, H102, H103, H104: MOUSER 855-M7682 -> (none); Mouser (none) -> 855-M7682
- IC101: value NCP5662-ADJ -> NCP5662-ADJ-TO263; MOUSER 863-NCP5662DSADJR4G -> (none); Mouser (none) -> 863-NCP5662DSADJR4G; Name (none) -> NCP5662-ADJ
- JP101: MOUSER 855-M7582 -> (none); Mouser (none) -> 855-M7582
- JP102, JP103: MOUSER 855-M7581 -> (none); Mouser (none) -> 855-M7581
- K101: MOUSER 490-PJ-102AH -> (none); Mouser (none) -> 490-PJ-102AH
- K102: MOUSER 490-TB006-508-02BE -> (none); Mouser (none) -> 490-TB006-508-02BE
- K103: MOUSER 450-476 -> (none); Mouser (none) -> 450-476
- LED101: MOUSER 604-APT3216LVBCD -> (none); Mouser (none) -> 604-APT3216LVBCD
- S101: MOUSER 611-1101M2S3CQE2 -> (none); Mouser (none) -> 611-1101M2S3CQE2
- TP101, TP102: MOUSER 534-5006 -> (none); Mouser (none) -> 534-5006
- U101, U102, U103, U104: MOUSER 534-24283 -> (none); Mouser (none) -> 534-24283
- X101, X102, X103, X104, X105: MOUSER 517-SJ5376 -> (none); Mouser (none) -> 517-SJ5376
Connections:
- net GND: now also R101.1, TP103.1
- net VCC: now also R101.3
- net at IC101.5 (ADJ): now also R101.2

Commit message: Up
Parts:
- removed IC101: NCP5662-ADJ-TO263, tronixio:TO-263-5, symbol tronixio:NCP5662-ADJ-TO263
- added U105: NCP5662-ADJ-TO263, tronixio:TO-263-5, symbol tronixio:NCP5662-ADJ-TO263
Connections:
- net GND: now also U105.3 (GND), U105.6 (GND)
- net VCC: now also U105.4 (VOUT)
- net VIN: now also U105.1 (EN), U105.2 (VIN)
- net at R101.2: now also U105.5 (ADJ)
Other:
- sheet MOD renamed Module
- sheet HID: file pic8bit-mod.kicad_sch -> pic8bit-hid.kicad_sch
- sheet Module: file pic8bit-hid.kicad_sch -> pic8bit-mod.kicad_sch
- title: Diagram -> Power
- moved on the sheet: B101, C101, C102, K101, K102, LED101, R101, R102, S101, TP101, TP102, TP103

Commit message: Update
Parts:
- added TP103: GND, tronixio:KEYSTONE-5006, symbol tronixio:KEYSTONE-5006
- renumbered TP103 to TP104
Connections:
- net GND: now also TP103.1
Other:
- moved on the sheet: TP104

Commit message: Update
Changed lines of the file:
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@@
     )
   )
-  (sheet (at 78.74 139.7) (size 43.18 43.18)
+  (sheet (at 76.2 139.7) (size 43.18 43.18)
     (stroke (width 0.1524) (type solid) (color 0 0 0 0))
     (fill (color 0 0 0 0.0000))
-    (property "Sheet name" "HID" (id 0) (at 78.74 138.43 0)
+    (property "Sheet name" "HID" (id 0) (at 76.2 138.43 0)
       (effects (font (size 2 2)) (justify left bottom))
     )
-    (property "Sheet file" "pic8bit-hid.kicad_sch" (id 1) (at 78.74 183.4166 0)
+    (property "Sheet file" "pic8bit-hid.kicad_sch" (id 1) (at 76.2 183.4166 0)
       (effects (font (size 1.27 1.27)) (justify left top))
     )
@@
     )
     (path "/81f75d1b-1f07-400d-98d6-f22aedb6142f/6eb969ba-5113-4e3c-b3e2-b0815d5c9b95"
-      (reference "S403") (unit 1) (value "BOURNS-PEC12R-24DENTS") (footprint "tronixio:BOURNS-PEC12R")
+      (reference "S403") (unit 1) (value "BOURNS-PEC12R-24DENTS") (footprint "tronixio:BOURNS-PEC12R-SWITCH")
     )
     (path "/81f75d1b-1f07-400d-98d6-f22aedb6142f/90c2329d-8ce7-42b6-8b4e-1a68cd1bb7e9"

Commit message: Update
Parts:
- B101: Name DF01M -> ONSEMI-DF01M
- C101, C102: symbol tronixio:UVZ-220U-25V -> tronixio:NICHICON-UVZ-220U-25V; Tolerance (none) -> 20%; Voltage (none) -> 25V
- K101: Name (none) -> CUI-PJ-102AH-TH
- K102: Name (none) -> CUI-TB006-508-02BE
- LED101: footprint tronixio:LED-05MM-TH -> tronixio:LED-1206; symbol tronixio:LED-1206-BLUE -> tronixio:KINGBRIGHT-LED-BLUE-1206; Name (none) -> KINGBRIGHT-LED-BLUE-1206
- R101: Name (none) -> 5K; Tolerance (none) -> 10%
- R102: footprint tronixio:RESISTOR-1016-TH -> tronixio:RESISTOR-1206; symbol tronixio:R-0805 -> tronixio:RESISTOR; Tolerance (none) -> 5%
- S101: Name (none) -> CK-1101M2
- TP104: Name (none) -> TP
- U105: symbol tronixio:NCP5662-ADJ-TO263 -> tronixio:ONSEMI-NCP5662-ADJ-TO263
Connections:
- net VCC renamed VDD
Other:
- note added: "- Revoir taille / graisse de serigraphie - Ajouter les reference composants datashets..."

Commit message: Update
Parts:
- B101: value ONSEMI-DF01M -> DF01M
- C101, C102: value UVZ-220U-25V -> 220µ/25V; Name 220µ/25V -> NICHICON-UVZ-220U-25V
- LED101: footprint tronixio:LED-1206 -> tronixio:LED-05MM-TH; symbol tronixio:KINGBRIGHT-LED-BLUE-1206 -> tronixio:KINGBRIGHT-LED-05MM-TH; Mouser 604-APT3216LVBCD -> 604-WP7113ID; Name KINGBRIGHT-LED-BLUE-1206 -> KINGBRIGHT-LED-05MM-TH
- R101: Name 5K -> VISHAY-5K-64W
- R102: footprint tronixio:RESISTOR-1206 -> tronixio:RESISTOR-1016-TH; symbol tronixio:RESISTOR -> tronixio:RESISTOR-1016TH-4K7; Mouser (none) -> 594-SFR2500004701JR5; Name (none) -> RESISTOR-1016TH-4K7
- TP101, TP102, TP103: Name (none) -> KEYSTONE-5006
- TP104: value KEYSTONE-2000-3 -> GND; Name TP -> KEYSTONE-2000-3
- U101, U102, U103, U104: footprint tronixio:zzzKEYSTONE-24283 -> tronixio:KEYSTONE-24283
- U105: value NCP5662-ADJ-TO263 -> NCP5662-ADJ; Name NCP5662-ADJ -> ONSEMI-NCP5662-ADJ-TO263
- X101, X102, X103, X104, X105: footprint tronixio:zzz3M-SJ5376 -> tronixio:3M-SJ5376
Connections:
- net GND: no longer U105.6 (GND)
