File: Kicad/trainer/pic8bit.kicad_sch (KiCad schematic)
At the start: 31 parts, among them K101 AC/DC 9-12V, K102 AC/DC 9-12V, K103 PE-450-4X6X-BLACK, U101 KEYSTONE-24283, U102 KEYSTONE-24283, U103 KEYSTONE-24283, U104 KEYSTONE-24283, U105 NCP5662-ADJ, X101 3M-SJ5376, X102 3M-SJ5376, X103 3M-SJ5376, X104 3M-SJ5376, X105 3M-SJ5376

Commit message: Update
Other:
- note removed: "- Revoir taille / graisse de serigraphie - Ajouter les reference composants datashets..."
Changed lines of the file:
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@@
     (stroke (width 0) (type default) (color 0 0 0 0))
-  )
-  (text "- Revoir taille / graisse de serigraphie\n- Ajouter les reference composants datashets...\n"
-    (at 152.4 144.78 0)
-    (effects (font (size 2 2)) (justify left bottom))
   )
   (symbol (lib_id "tronixio:CUI-TB006-508-02BE") (at 78.74 55.88 0) (mirror y) (unit 1)

Commit message: Update
Parts:
- LED101: footprint tronixio:LED-05MM-TH -> tronixio:LED-TH-05MM
- R102: footprint tronixio:RESISTOR-1016-TH -> tronixio:RESISTOR-TH-1016
Changed lines of the file:
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@@
     (pin "1")
   )
-  (symbol (lib_id "tronixio:ONSEMI-NCP5662-ADJ-TO263") (at 129.54 45.72 0) (unit 1)
+  (symbol (lib_id "tronixio:ONSEMI-NCP5662-ADJ-TO263") (at 121.92 43.18 0) (unit 1)
     (in_bom yes) (on_board yes)
-    (property "Reference" "U105" (id 0) (at 129.54 36.83 0)
+    (property "Reference" "U105" (id 0) (at 121.92 34.29 0)
       (effects (font (size 1.15 1.15)))
     )
-    (property "Value" "NCP5662-ADJ" (id 1) (at 129.54 39.37 0)
+    (property "Value" "NCP5662-ADJ" (id 1) (at 121.92 36.83 0)
       (effects (font (size 1.15 1.15)))
     )
@@
       (effects (font (size 1 1)) hide)
     )
-    (property "Tolerance" "10%" (id 5) (at 143.51 63.5 0)
+    (property "Tolerance" "10%" (id 5) (at 142.24 57.15 0)
       (effects (font (size 1.15 1.15)) (justify left) hide)
     )
@@
     )
     (property "Footprint" "" (id 2) (at 167.64 180.34 0)
-      (effects (font (size 1.27 1.27)) hide)
-    )
-    (property "Datasheet" "~" (id 3) (at 167.64 180.34 0)
-      (effects (font (size 1.27 1.27)) hide)
+      (effects (font (size 1 1)) hide)
+    )
+    (property "Datasheet" "" (id 3) (at 167.64 180.34 0)
+      (effects (font (size 1 1)) hide)
     )
     (pin "1")
@@
     )
     (property "Footprint" "" (id 2) (at 175.26 190.5 0)
-      (effects (font (size 1.27 1.27)) hide)
-    )
-    (property "Datasheet" "~" (id 3) (at 175.26 190.5 0)
-      (effects (font (size 1.27 1.27)) hide)
+      (effects (font (size 1 1)) hide)
+    )
+    (property "Datasheet" "" (id 3) (at 175.26 190.5 0)
+      (effects (font (size 1 1)) hide)
     )
     (pin "1")
@@
       (effects (font (size 1.15 1.15)))
     )
-    (property "Footprint" "tronixio:RESISTOR-1016-TH" (id 2) (at 167.64 58.42 0)
+    (property "Footprint" "tronixio:RESISTOR-TH-1016" (id 2) (at 167.64 58.42 0)
       (effects (font (size 1 1)) hide)
     )
@@
       (effects (font (size 1 1)) hide)
     )
-    (property "Tolerance" "5%" (id 4) (at 170.18 44.45 0)
+    (property "Tolerance" "5%" (id 4) (at 170.18 46.99 0)
       (effects (font (size 1.15 1.15)) (justify left) hide)
     )
@@
       (effects (font (size 1.15 1.15)) (justify left))
     )
-    (property "Footprint" "tronixio:LED-05MM-TH" (id 2) (at 157.48 53.34 0)
+    (property "Footprint" "tronixio:LED-TH-05MM" (id 2) (at 157.48 53.34 0)
       (effects (font (size 1 1)) hide)
     )
@@
     )
     (path "/aba47c6d-6a1f-498d-ae98-b277afefcc3f"
-      (reference "LED101") (unit 1) (value "Power") (footprint "tronixio:LED-05MM-TH")
+      (reference "LED101") (unit 1) (value "Power") (footprint "tronixio:LED-TH-05MM")
     )
     (path "/81f75d1b-1f07-400d-98d6-f22aedb6142f/09cf5efb-b260-43b0-87e6-98819bf7d96b"
@@
     )
     (path "/a62b5ec4-70fb-4b70-8887-569d9ace44ad"
-      (reference "R102") (unit 1) (value "4K7") (footprint "tronixio:RESISTOR-1016-TH")
+      (reference "R102") (unit 1) (value "4K7") (footprint "tronixio:RESISTOR-TH-1016")
     )
     (path "/64edc06d-d6ae-4dac-9759-3f1fbed6457d/a9369e84-04c4-4b26-8073-c4fbe88c7f4d"
-      (reference "R201") (unit 1) (value "10K") (footprint "tronixio:RESISTOR-1016-TH")
+      (reference "R201") (unit 1) (value "10K") (footprint "tronixio:RESISTOR-TH-1016")
     )
     (path "/64edc06d-d6ae-4dac-9759-3f1fbed6457d/78883502-61df-41cc-8136-60a362ad2eda"
-      (reference "R202") (unit 1) (value "1K") (footprint "tronixio:RESISTOR-1016-TH")
+      (reference "R202") (unit 1) (value "1K") (footprint "tronixio:RESISTOR-TH-1016")
     )
     (path "/64edc06d-d6ae-4dac-9759-3f1fbed6457d/8822b915-443b-4169-9f73-615862607291"
-      (reference "R203") (unit 1) (value "4K7") (footprint "tronixio:RESISTOR-1016-TH")
+      (reference "R203") (unit 1) (value "4K7") (footprint "tronixio:RESISTOR-TH-1016")
     )
     (path "/64edc06d-d6ae-4dac-9759-3f1fbed6457d/99c5437e-dbc3-47a3-aae9-b12482fa0399"
-      (reference "R204") (unit 1) (value "4K7") (footprint "tronixio:RESISTOR-1016-TH")
+      (reference "R204") (unit 1) (value "4K7") (footprint "tronixio:RESISTOR-TH-1016")
     )
     (path "/8cdf8b92-b881-481d-a85a-c0055e9a856b/29843283-7d2c-4c3a-a497-d39e3f3829e5"
-      (reference "R301") (unit 1) (value "200Ω") (footprint "tronixio:RESISTOR-1206")
+      (reference "R301") (unit 1) (value "200Ω") (footprint "tronixio:RESISTOR-SMD-1206")
     )
     (path "/8cdf8b92-b881-481d-a85a-c0055e9a856b/a47366a5-6845-49d8-bd9c-362158ae1421"
-      (reference "R302") (unit 1) (value "200Ω") (footprint "tronixio:RESISTOR-1206")
+      (reference "R302") (unit 1) (value "200Ω") (footprint "tronixio:RESISTOR-SMD-1206")
     )
     (path "/8cdf8b92-b881-481d-a85a-c0055e9a856b/cc0cecc7-0d93-4e54-a910-5492669f5660"
-      (reference "R303") (unit 1) (value "200Ω") (footprint "tronixio:RESISTOR-1206")
+      (reference "R303") (unit 1) (value "200Ω") (footprint "tronixio:RESISTOR-SMD-1206")
     )
     (path "/8cdf8b92-b881-481d-a85a-c0055e9a856b/6383ccd5-e861-465e-8833-5260793caf1b"
-      (reference "R304") (unit 1) (value "200Ω") (footprint "tronixio:RESISTOR-1206")
+      (reference "R304") (unit 1) (value "200Ω") (footprint "tronixio:RESISTOR-SMD-1206")
     )
     (path "/8cdf8b92-b881-481d-a85a-c0055e9a856b/df6627fa-7d96-4c92-8d26-9eca6d38e095"
-      (reference "R305") (unit 1) (value "200Ω") (footprint "tronixio:RESISTOR-1206")
+      (reference "R305") (unit 1) (value "200Ω") (footprint "tronixio:RESISTOR-SMD-1206")
     )
     (path "/8cdf8b92-b881-481d-a85a-c0055e9a856b/d2f5bb66-48e2-4260-8543-a7551b9278b9"
-      (reference "R306") (unit 1) (value "200Ω") (footprint "tronixio:RESISTOR-1206")
+      (reference "R306") (unit 1) (value "200Ω") (footprint "tronixio:RESISTOR-SMD-1206")
     )
     (path "/8cdf8b92-b881-481d-a85a-c0055e9a856b/c70d3f25-354d-4679-874a-e3e7db17c38b"
-      (reference "R307") (unit 1) (value "200Ω") (footprint "tronixio:RESISTOR-1206")
+      (reference "R307") (unit 1) (value "200Ω") (footprint "tronixio:RESISTOR-SMD-1206")
     )
     (path "/8cdf8b92-b881-481d-a85a-c0055e9a856b/2620f5ca-2fb3-4d21-b9ca-b957ac6a47bd"
-      (reference "R308") (unit 1) (value "200Ω") (footprint "tronixio:RESISTOR-1206")
+      (reference "R308") (unit 1) (value "200Ω") (footprint "tronixio:RESISTOR-SMD-1206")
     )
     (path "/8cdf8b92-b881-481d-a85a-c0055e9a856b/61c6c3fe-7d2f-4f10-a100-9fb225285a8c"
-      (reference "R309") (unit 1) (value "200Ω") (footprint "tronixio:RESISTOR-1206")
+      (reference "R309") (unit 1) (value "200Ω") (footprint "tronixio:RESISTOR-SMD-1206")
     )
     (path "/8cdf8b92-b881-481d-a85a-c0055e9a856b/9527870b-e034-4633-9ab3-67b00175c224"
-      (reference "R310") (unit 1) (value "200Ω") (footprint "tronixio:RESISTOR-1206")
+      (reference "R310") (unit 1) (value "200Ω") (footprint "tronixio:RESISTOR-SMD-1206")
     )
     (path "/8cdf8b92-b881-481d-a85a-c0055e9a856b/cf231d88-ae96-4bef-8b65-0ba79008d17c"
-      (reference "R311") (unit 1) (value "200Ω") (footprint "tronixio:RESISTOR-1206")
+      (reference "R311") (unit 1) (value "200Ω") (footprint "tronixio:RESISTOR-SMD-1206")
     )
     (path "/8cdf8b92-b881-481d-a85a-c0055e9a856b/0456bcac-fce7-4aeb-b106-65c9a20075e0"
-      (reference "R312") (unit 1) (value "200Ω") (footprint "tronixio:RESISTOR-1206")
+      (reference "R312") (unit 1) (value "200Ω") (footprint "tronixio:RESISTOR-SMD-1206")
     )
     (path "/8cdf8b92-b881-481d-a85a-c0055e9a856b/95a18207-9dd9-4060-be43-909e4a9c7123"
-      (reference "R313") (unit 1) (value "200Ω") (footprint "tronixio:RESISTOR-1206")
+      (reference "R313") (unit 1) (value "200Ω") (footprint "tronixio:RESISTOR-SMD-1206")
     )
     (path "/8cdf8b92-b881-481d-a85a-c0055e9a856b/41f9509c-3d72-4584-aa38-3cb1fab4fdac"
-      (reference "R314") (unit 1) (value "200Ω") (footprint "tronixio:RESISTOR-1206")
+      (reference "R314") (unit 1) (value "200Ω") (footprint "tronixio:RESISTOR-SMD-1206")
     )
     (path "/8cdf8b92-b881-481d-a85a-c0055e9a856b/f292c6bb-34c9-4e7d-a1ce-a7d4f8be97fb"
-      (reference "R315") (unit 1) (value "200Ω") (footprint "tronixio:RESISTOR-1206")
+      (reference "R315") (unit 1) (value "200Ω") (footprint "tronixio:RESISTOR-SMD-1206")
     )
     (path "/8cdf8b92-b881-481d-a85a-c0055e9a856b/ec48aa52-3382-4ffe-91de-4fedd71fa2ee"
-      (reference "R316") (unit 1) (value "200Ω") (footprint "tronixio:RESISTOR-1206")
+      (reference "R316") (unit 1) (value "200Ω") (footprint "tronixio:RESISTOR-SMD-1206")
     )
     (path "/81f75d1b-1f07-400d-98d6-f22aedb6142f/2e85c6ac-c1f9-4fea-b1c4-5ca3f0666990"
@@
     )
     (path "/81f75d1b-1f07-400d-98d6-f22aedb6142f/b6935720-5273-42ea-89d6-cf37e254287d"
-      (reference "R402") (unit 1) (value "10Ω") (footprint "tronixio:RESISTOR-1016-TH")
+      (reference "R402") (unit 1) (value "10Ω") (footprint "tronixio:RESISTOR-TH-1016")
     )
     (path "/81f75d1b-1f07-400d-98d6-f22aedb6142f/739dbaa7-7e8e-46a0-9a44-d8a4348f60e5"
@@
     )
     (path "/64edc06d-d6ae-4dac-9759-3f1fbed6457d/aefdb178-1c83-4b81-94e9-78aeec5f99e4"
-      (reference "U201") (unit 1) (value "PIC16F/18F") (footprint "tronixio:DIP-28-W762-SOCKET")
+      (reference "U201") (unit 1) (value "PIC16F/18F") (footprint "tronixio:DIP-28-W762")
     )
     (path "/64edc06d-d6ae-4dac-9759-3f1fbed6457d/ce8b6347-20a2-493f-b8f1-2602aeda2d6d"

Commit message: Update
Parts:
- C101, C102: footprint tronixio:CAPACITOR-ELECTROLYTIC-RADIAL-080-115-035 -> tronixio:CAPACITOR-ELECTROLYTIC-RADIAL-080-110-035
Changed lines of the file:
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@@
   (symbol (lib_id "tronixio:CUI-TB006-508-02BE") (at 78.74 55.88 0) (mirror y) (unit 1)
     (in_bom yes) (on_board yes)
-    (property "Reference" "K102" (id 0) (at 78.74 53.34 0)
-      (effects (font (size 1.15 1.15)))
-    )
-    (property "Value" "AC/DC 9-12V" (id 1) (at 78.74 62.23 0)
+    (property "Reference" "K102" (id 0) (at 78.74 52.705 0)
+      (effects (font (size 1.15 1.15)))
+    )
+    (property "Value" "AC/DC 9-12V" (id 1) (at 78.74 61.595 0)
       (effects (font (size 1.15 1.15)))
     )
@@
     (pin "3")
   )
-  (symbol (lib_id "tronixio:NICHICON-UVZ-220U-25V") (at 114.3 55.88 0) (unit 1)
+  (symbol (lib_name "NICHICON-UVZ-220U-25V_1") (lib_id "tronixio:NICHICON-UVZ-220U-25V") (at 114.3 55.88 0) (unit 1)
     (in_bom yes) (on_board yes)
     (property "Reference" "C101" (id 0) (at 113.665 53.34 0)
@@
       (effects (font (size 1.15 1.15)) (justify right))
     )
-    (property "Footprint" "tronixio:CAPACITOR-ELECTROLYTIC-RADIAL-080-115-035" (id 2) (at 114.3 68.58 0)
+    (property "Footprint" "tronixio:CAPACITOR-ELECTROLYTIC-RADIAL-080-110-035" (id 2) (at 114.3 68.58 0)
       (effects (font (size 1 1)) hide)
     )
@@
   (symbol (lib_id "tronixio:ONSEMI-DF01M") (at 104.14 43.18 0) (unit 1)
     (in_bom yes) (on_board yes)
-    (property "Reference" "B101" (id 0) (at 103.505 36.8299 0)
+    (property "Reference" "B101" (id 0) (at 103.505 36.83 0)
       (effects (font (size 1.15 1.15)) (justify right))
     )
-    (property "Value" "DF01M" (id 1) (at 104.775 36.83 0)
-      (effects (font (size 1.15 1.15)) (justify left))
+    (property "Value" "DF01M" (id 1) (at 103.505 49.53 0)
+      (effects (font (size 1.15 1.15)) (justify right))
     )
     (property "Footprint" "tronixio:DF01M" (id 2) (at 104.14 60.96 0)
@@
       (effects (font (size 1.15 1.15)) (justify left))
     )
-    (property "Footprint" "tronixio:CAPACITOR-ELECTROLYTIC-RADIAL-080-115-035" (id 2) (at 152.4 68.58 0)
+    (property "Footprint" "tronixio:CAPACITOR-ELECTROLYTIC-RADIAL-080-110-035" (id 2) (at 152.4 68.58 0)
       (effects (font (size 1 1)) hide)
     )
@@
     )
     (path "/878fc6d0-3e85-4aaa-bd2e-cc5f4362a64f"
-      (reference "C101") (unit 1) (value "220µ/25V") (footprint "tronixio:CAPACITOR-ELECTROLYTIC-RADIAL-080-115-035")
+      (reference "C101") (unit 1) (value "220µ/25V") (footprint "tronixio:CAPACITOR-ELECTROLYTIC-RADIAL-080-110-035")
     )
     (path "/fd661bfe-3682-4b84-8db0-bdca7dd9a40c"
-      (reference "C102") (unit 1) (value "220µ/25V") (footprint "tronixio:CAPACITOR-ELECTROLYTIC-RADIAL-080-115-035")
+      (reference "C102") (unit 1) (value "220µ/25V") (footprint "tronixio:CAPACITOR-ELECTROLYTIC-RADIAL-080-110-035")
     )
     (path "/64edc06d-d6ae-4dac-9759-3f1fbed6457d/8d5531be-425c-471c-8d2f-56f471ef38cc"

Commit message: Update
Changed lines of the file:
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@@
   (symbol (lib_id "tronixio:ONSEMI-NCP5662-ADJ-TO263") (at 121.92 43.18 0) (unit 1)
     (in_bom yes) (on_board yes)
-    (property "Reference" "U105" (id 0) (at 121.92 34.29 0)
+    (property "Reference" "U105" (id 0) (at 129.54 36.83 0)
       (effects (font (size 1.15 1.15)))
     )
-    (property "Value" "NCP5662-ADJ" (id 1) (at 121.92 36.83 0)
+    (property "Value" "NCP5662-ADJ" (id 1) (at 129.54 39.37 0)
       (effects (font (size 1.15 1.15)))
     )
@@
       (reference "U201") (unit 1) (value "PIC16F/18F") (footprint "tronixio:DIP-28-W762")
     )
-    (path "/64edc06d-d6ae-4dac-9759-3f1fbed6457d/ce8b6347-20a2-493f-b8f1-2602aeda2d6d"
-      (reference "X1") (unit 1) (value "XTAL-DIL08") (footprint "tronixio:DIP-08-W762-SOCKET")
-    )
     (path "/f7b23f20-a100-41e1-ac8c-691c439ad031"
       (reference "X101") (unit 1) (value "3M-SJ5376") (footprint "tronixio:3M-SJ5376")
@@
       (reference "X105") (unit 1) (value "3M-SJ5376") (footprint "tronixio:3M-SJ5376")
     )
-  )
+    (path "/64edc06d-d6ae-4dac-9759-3f1fbed6457d/ce8b6347-20a2-493f-b8f1-2602aeda2d6d"
+      (reference "X201") (unit 1) (value "XTAL-DIL08") (footprint "tronixio:DIP-08-W762-SOCKET")
+    )
+  )

Commit message: Update pic8bit trainer
Parts:
- B101: Name ONSEMI-DF01M -> (none)
- C101, C102: Name NICHICON-UVZ-220U-25V -> (none)
- K101: Name CUI-PJ-102AH-TH -> (none)
- K102: Name CUI-TB006-508-02BE -> (none)
- LED101: Name KINGBRIGHT-LED-05MM-TH -> (none)
- R101: Name VISHAY-5K-64W -> (none)
- R102: Name RESISTOR-1016TH-4K7 -> (none)
- S101: Name CK-1101M2 -> (none)
- TP101, TP102, TP103: Name KEYSTONE-5006 -> (none)
- TP104: Name KEYSTONE-2000-3 -> (none)
- U105: Name ONSEMI-NCP5662-ADJ-TO263 -> (none)

Commit message: Up
Other:
- title: Power -> Root & Power
Changed lines of the file:
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@@
   (paper "A4")
   (title_block
-    (title "Power")
+    (title "Root & Power")
     (date "01/2022")
     (rev "A")
