File: Kicad/trainer/pic8bit.kicad_sch (KiCad schematic)
At the start: 31 parts, among them K101 AC/DC 9-12V, K102 AC/DC 9-12V, K103 PE-450-4X6X-BLACK, U101 KEYSTONE-24283, U102 KEYSTONE-24283, U103 KEYSTONE-24283, U104 KEYSTONE-24283, U105 NCP5662-ADJ, X101 3M-SJ5376, X102 3M-SJ5376, X103 3M-SJ5376, X104 3M-SJ5376, X105 3M-SJ5376

Commit message: Update
Parts:
- C101, C102: value 220µ/25V -> 220µ; footprint tronixio:CAPACITOR-ELECTROLYTIC-RADIAL-080-110-035 -> tronixio:CAPACITOR-ELECTROLYTIC-RADIAL-080-115-035
Changed lines of the file:
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@@
       (effects (font (size 1.15 1.15)) (justify right))
     )
-    (property "Value" "220µ/25V" (at 113.665 58.42 0)
+    (property "Value" "220µ" (at 113.665 58.42 0) (do_not_autoplace)
       (effects (font (size 1.15 1.15)) (justify right))
     )
-    (property "Footprint" "tronixio:CAPACITOR-ELECTROLYTIC-RADIAL-080-110-035" (at 114.3 66.04 0)
-      (effects (font (size 1 1)) hide)
-    )
-    (property "Datasheet" "http://www.nichicon.co.jp/english/products/pdfs/e-uvz.pdf" (at 114.3 68.58 0)
-      (effects (font (size 1 1)) hide)
-    )
-    (property "Voltage" "25V" (at 115.57 60.96 0)
+    (property "Footprint" "tronixio:CAPACITOR-ELECTROLYTIC-RADIAL-080-115-035" (at 114.3 66.04 0) (do_not_autoplace)
+      (effects (font (size 1 1)) hide)
+    )
+    (property "Datasheet" "http://www.nichicon.co.jp/english/products/pdfs/e-uvz.pdf" (at 114.3 68.58 0) (do_not_autoplace)
+      (effects (font (size 1 1)) hide)
+    )
+    (property "Voltage" "25V" (at 113.665 60.96 0) (do_not_autoplace)
+      (effects (font (size 1.15 1.15)) (justify right))
+    )
+    (property "Tolerance" "20%" (at 119.38 60.96 0) (do_not_autoplace)
       (effects (font (size 1.15 1.15)) (justify left) hide)
     )
-    (property "Tolerance" "20%" (at 119.38 60.96 0)
-      (effects (font (size 1.15 1.15)) (justify left) hide)
-    )
-    (property "Mouser" "647-UVZ1E221MPD" (at 114.3 71.12 0)
+    (property "Mouser" "647-UVZ1E221MPD" (at 114.3 71.12 0) (do_not_autoplace)
       (effects (font (size 1 1)) hide)
     )
@@
       (effects (font (size 1.15 1.15)) (justify left))
     )
-    (property "Value" "220µ/25V" (at 153.035 58.42 0)
+    (property "Value" "220µ" (at 153.035 58.42 0) (do_not_autoplace)
       (effects (font (size 1.15 1.15)) (justify left))
     )
-    (property "Footprint" "tronixio:CAPACITOR-ELECTROLYTIC-RADIAL-080-110-035" (at 152.4 66.04 0)
-      (effects (font (size 1 1)) hide)
-    )
-    (property "Datasheet" "http://www.nichicon.co.jp/english/products/pdfs/e-uvz.pdf" (at 152.4 68.58 0)
-      (effects (font (size 1 1)) hide)
-    )
-    (property "Voltage" "25V" (at 153.67 60.96 0)
+    (property "Footprint" "tronixio:CAPACITOR-ELECTROLYTIC-RADIAL-080-115-035" (at 152.4 66.04 0) (do_not_autoplace)
+      (effects (font (size 1 1)) hide)
+    )
+    (property "Datasheet" "http://www.nichicon.co.jp/english/products/pdfs/e-uvz.pdf" (at 152.4 68.58 0) (do_not_autoplace)
+      (effects (font (size 1 1)) hide)
+    )
+    (property "Voltage" "25V" (at 153.035 60.96 0) (do_not_autoplace)
+      (effects (font (size 1.15 1.15)) (justify left))
+    )
+    (property "Tolerance" "20%" (at 157.48 60.96 0) (do_not_autoplace)
       (effects (font (size 1.15 1.15)) (justify left) hide)
     )
-    (property "Tolerance" "20%" (at 157.48 60.96 0)
-      (effects (font (size 1.15 1.15)) (justify left) hide)
-    )
-    (property "Mouser" "647-UVZ1E221MPD" (at 152.4 71.12 0)
-      (effects (font (size 1 1)) hide)
-    )
+    (property "Mouser" "647-UVZ1E221MPD" (at 152.4 71.12 0) (do_not_autoplace)
+      (effects (font (size 1 1)) hide)
+    )

Commit message: Up
Parts:
- C101, C102: Life (none) -> 1000H; Serie (none) -> UVZ
- R102: symbol tronixio:RESISTOR-1016TH-4K7 -> tronixio:RESISTOR-1016TH-4K7-5P
Connections:
- net VDD renamed +VDD
- net VIN renamed +VIN

Commit message: Up
Changed lines of the file:
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@@
     )
     (property "Voltage" "25V" (at 113.665 60.96 0) (do_not_autoplace)
-      (effects (font (size 1.15 1.15)) (justify left))
+      (effects (font (size 1.15 1.15)) (justify right))
     )
     (property "Tolerance" "20%" (at 119.38 60.96 0) (do_not_autoplace)

Commit message: Update
Parts:
- R101: symbol tronixio:VISHAY-5K-64W -> tronixio:TRIMMER-64W-5K
Changed lines of the file:
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@@
     )
   )
-  (symbol (lib_id "tronixio:VISHAY-5K-64W") (at 144.78 55.88 0) (mirror y) (unit 1)
+  (symbol (lib_id "tronixio:TRIMMER-64W-5K") (at 144.78 55.88 0) (mirror y) (unit 1)
     (in_bom yes) (on_board yes) (dnp no)
     (property "Reference" "R101" (at 145.415 51.435 0)
@@
       (effects (font (size 1 1)) hide)
     )
-    (property "Datasheet" "https://www.onsemi.com/products/discretes-drivers/diodes-rectifiers/rectifiers/df01m" (at 104.14 60.96 0) (do_not_autoplace)
-      (effects (font (size 1 1)) hide)
-    )
+    (property "Datasheet" "https://www.onsemi.com/products/discrete-power-modules/rectifiers/DF01M" (at 104.14 60.96 0) (do_not_autoplace)
+      (effects (font (size 1 1)) hide)
+    )

Commit message: Update Trainer Kicad 8
Parts:
- LED101: footprint tronixio:LED-TH-05MM -> tronixio:LED-TH-ROUND-05MM; symbol tronixio:KINGBRIGHT-LED-05MM-TH -> tronixio:KINGBRIGHT-LED-05MM-RED
Connections:
- net +VDD renamed POWER-VDD
- net +VIN renamed POWER-VIN
- net GND renamed POWER-GND

Commit message: Update Trainer
Changed lines of the file:
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@@
 	)
 	(junction
+		(at 116.84 43.18)
+		(diameter 0)
+		(color 0 0 0 0)
+	)
+	(junction
 		(at 91.44 55.88)
 		(diameter 0)
@@
 		(color 0 0 0 0)
 	)
+	(junction
+		(at 96.52 43.18)
+		(diameter 0)
+		(color 0 0 0 0)
+	)
 	(no_connect
 		(at 93.98 33.02)
@@
 	(wire
 		(pts
-			(xy 175.26 180.34) (xy 175.26 190.5)
-		)
-		(stroke
-			(width 0)
-			(type default)
-		)
-	)
-	(wire
-		(pts
 			(xy 114.3 58.42) (xy 114.3 60.96)
 		)
@@
 	(wire
 		(pts
-			(xy 167.64 180.34) (xy 167.64 190.5)
-		)
-		(stroke
-			(width 0)
-			(type default)
-		)
-	)
-	(wire
-		(pts
 			(xy 83.82 43.18) (xy 91.44 43.18)
 		)
@@
 	(wire
 		(pts
-			(xy 114.3 43.18) (xy 121.92 43.18)
+			(xy 114.3 43.18) (xy 116.84 43.18)
+		)
+		(stroke
+			(width 0)
+			(type default)
+		)
+	)
+	(wire
+		(pts
+			(xy 116.84 43.18) (xy 121.92 43.18)
 		)
 		(stroke
@@
 	)
 	(symbol
+		(lib_id "tronixio:POWER-FLAG")
+		(at 96.52 43.18 0)
+		(unit 1)
+		(exclude_from_sim no)
+		(in_bom yes)
+		(on_board yes)
+		(dnp no)
+		(fields_autoplaced yes)
+		(property "Reference" "#FLG01"
+			(at 96.52 45.085 0)
+			(effects
+				(font
+					(size 1.27 1.27)
+				)
+				(hide yes)
+			)
+		)
+		(property "Value" "POWER-FLAG"
+			(at 96.52 46.99 0)
+			(effects
+				(font
+					(size 1.27 1.27)
+				)
+				(hide yes)
+			)
+		)
+		(property "Footprint" ""
+			(at 96.52 43.18 0)
+			(effects
+				(font
+					(size 1 1)
+				)
+				(hide yes)
+			)
+		)
+		(property "Datasheet" ""
+			(at 96.52 43.18 0)
+			(effects
+				(font
+					(size 1 1)
+				)
+				(hide yes)
+			)
+		)
+		(property "Description" "Special symbol for telling ERC where power comes from"
+			(at 96.52 43.18 0)
+			(effects
+				(font
+					(size 1.27 1.27)
+				)
+				(hide yes)
+			)
+		)
+		(pin "1"
+		)
+		(instances
+			(project "pic8bit"
+				(path "/d431d485-8cd8-4e00-afcd-f39218d614ca"
+					(reference "#FLG01")
+					(unit 1)
+				)
+			)
+		)
+	)
+	(symbol
 		(lib_id "tronixio:TRIMMER-64W-5K")
 		(at 144.78 55.88 0)
@@
 	)
 	(symbol
-		(lib_id "tronixio:POWER-FLAG")
-		(at 167.64 180.34 0)
-		(unit 1)
-		(exclude_from_sim no)
-		(in_bom yes)
-		(on_board yes)
-		(dnp no)
-		(fields_autoplaced yes)
-		(property "Reference" "#FLG0101"
-			(at 167.64 182.245 0)
-			(effects
-				(font
-					(size 1.27 1.27)
-				)
-				(hide yes)
-			)
-		)
-		(property "Value" "POWER-FLAG"
-			(at 167.64 184.15 0)
-			(effects
-				(font
-					(size 1.27 1.27)
-				)
-				(hide yes)
-			)
-		)
-		(property "Footprint" ""
-			(at 167.64 180.34 0)
-			(effects
-				(font
-					(size 1 1)
-				)
-				(hide yes)
-			)
-		)
-		(property "Datasheet" ""
-			(at 167.64 180.34 0)
-			(effects
-				(font
-					(size 1 1)
-				)
-				(hide yes)
-			)
-		)
-		(property "Description" "Special symbol for telling ERC where power comes from"
-			(at 167.64 180.34 0)
-			(effects
-				(font
-					(size 1.27 1.27)
-				)
-				(hide yes)
-			)
-		)
-		(pin "1"
-		)
-		(instances
-			(project "pic8bit"
-				(path "/d431d485-8cd8-4e00-afcd-f39218d614ca"
-					(reference "#FLG0101")
-					(unit 1)
-				)
-			)
-		)
-	)
-	(symbol
 		(lib_id "tronixio:POWER-GND")
 		(at 96.52 60.96 0)
@@
 	)
 	(symbol
-		(lib_id "tronixio:POWER-+VIN")
-		(at 175.26 180.34 0)
-		(unit 1)
-		(exclude_from_sim no)
-		(in_bom yes)
-		(on_board yes)
-		(dnp no)
-		(property "Reference" "#PWR0111"
-			(at 175.26 190.5 0)
-			(effects
-				(font
-					(size 1 1)
-				)
-				(hide yes)
-			)
-		)
-		(property "Value" "POWER-VIN"
-			(at 175.26 193.04 0)
-			(effects
-				(font
-					(size 1 1)
-				)
-				(hide yes)
-			)
-		)
-		(property "Footprint" ""
-			(at 175.26 180.34 0)
-			(effects
-				(font
-					(size 1 1)
-				)
-				(hide yes)
-			)
-		)
-		(property "Datasheet" ""
-			(at 175.26 180.34 0)
-			(effects
-				(font
-					(size 1 1)
-				)
-				(hide yes)
-			)
-		)
-		(property "Description" ""
-			(at 175.26 180.34 0)
-			(effects
-				(font
-					(size 1.27 1.27)
-				)
-				(hide yes)
-			)
-		)
-		(property "Name" "VIN"
-			(at 175.26 175.26 0)
-			(do_not_autoplace yes)
-			(effects
-				(font
-					(size 1.15 1.15)
-				)
-			)
-		)
-		(pin "1"
-		)
-		(instances
-			(project "pic8bit"
-				(path "/d431d485-8cd8-4e00-afcd-f39218d614ca"
-					(reference "#PWR0111")
-					(unit 1)
-				)
-			)
-		)
-	)
-	(symbol
-		(lib_id "tronixio:POWER-GND")
-		(at 167.64 190.5 0)
-		(unit 1)
-		(exclude_from_sim no)
-		(in_bom yes)
-		(on_board yes)
-		(dnp no)
-		(fields_autoplaced yes)
-		(property "Reference" "#PWR0110"
-			(at 167.64 195.58 0)
-			(effects
-				(font
-					(size 1 1)
-				)
-				(hide yes)
-			)
-		)
-		(property "Value" "POWER-GND"
-			(at 167.64 198.12 0)
-			(effects
-				(font
-					(size 1 1)
-				)
-				(hide yes)
-			)
-		)
-		(property "Footprint" ""
-			(at 167.64 190.5 0)
-			(effects
-				(font
-					(size 1 1)
-				)
-				(hide yes)
-			)
-		)
-		(property "Datasheet" ""
-			(at 167.64 190.5 0)
-			(effects
-				(font
-					(size 1 1)
-				)
-				(hide yes)
-			)
-		)
-		(property "Description" ""
-			(at 167.64 190.5 0)
-			(effects
-				(font
-					(size 1.27 1.27)
-				)
-				(hide yes)
-			)
-		)
-		(pin "1"
-		)
-		(instances
-			(project "pic8bit"
-				(path "/d431d485-8cd8-4e00-afcd-f39218d614ca"
-					(reference "#PWR0110")
-					(unit 1)
-				)
-			)
-		)
-	)
-	(symbol
 		(lib_id "tronixio:HARWIN-JUMPER-0254-06MM-RED")
 		(at 200.66 172.72 0)
@@
 	(symbol
 		(lib_id "tronixio:POWER-FLAG")
-		(at 175.26 190.5 180)
+		(at 116.84 43.18 0)
 		(unit 1)
 		(exclude_from_sim no)
@@
 		(fields_autoplaced yes)
 		(property "Reference" "#FLG0102"
-			(at 175.26 188.595 0)
+			(at 116.84 45.085 0)
 			(effects
 				(font
@@
 		)
 		(property "Value" "POWER-FLAG"
-			(at 175.26 186.69 0)
+			(at 116.84 46.99 0)
 			(effects
 				(font
@@
 		)
 		(property "Footprint" ""
-			(at 175.26 190.5 0)
+			(at 116.84 43.18 0)
 			(effects
 				(font
@@
 		)
 		(property "Datasheet" ""
-			(at 175.26 190.5 0)
+			(at 116.84 43.18 0)
 			(effects
 				(font
@@
 		)
 		(property "Description" "Special symbol for telling ERC where power comes from"
-			(at 175.26 190.5 0)
+			(at 116.84 43.18 0)
 			(effects
 				(font
@@
 		(on_board yes)
 		(dnp no)
-		(fields_autoplaced yes)
 		(property "Reference" "#PWR0108"
 			(at 167.64 45.72 0)
@@
 			)
 		)
-		(property "Description" ""
-			(at 167.64 35.56 0)
-			(effects
-				(font
-					(size 1.27 1.27)
-				)
-				(hide yes)
-			)
-		)
-		(property "Name" "VDD"
+		(property "Description" "VDD"
 			(at 167.64 30.48 0)
-			(do_not_autoplace yes)
 			(effects
 				(font
-					(size 1.15 1.15)
+					(size 1.27 1.27)
 				)
 			)
@@
 			)
 		)
-		(property "Description" ""
-			(at 114.3 35.56 0)
-			(effects
-				(font
-					(size 1.27 1.27)
-				)
-				(hide yes)
-			)
-		)
-		(property "Name" "VIN"
+		(property "Description" "VIN"
 			(at 114.3 30.48 0)
-			(do_not_autoplace yes)
 			(effects
 				(font
-					(size 1.15 1.15)
+					(size 1.27 1.27)
 				)
 			)
@@
 		(on_board yes)
 		(dnp no)
-		(fields_autoplaced yes)
 		(property "Reference" "#PWR0106"
 			(at 152.4 45.72 0)
@@
 			)
 		)
-		(property "Description" ""
-			(at 152.4 35.56 0)
-			(effects
-				(font
-					(size 1.27 1.27)
-				)
-				(hide yes)
-			)
-		)
-		(property "Name" "VDD"
+		(property "Description" "VDD"
 			(at 152.4 30.48 0)
-			(do_not_autoplace yes)
 			(effects
 				(font
-					(size 1.15 1.15)
+					(size 1.27 1.27)
 				)
 			)

Commit message: Up
Parts:
- U105: footprint tronixio:TO-263-5 -> tronixio:TO-263-5-TABPIN3
Changed lines of the file:
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@@
 			)
 		)
-		(property "Footprint" "tronixio:TO-263-5"
+		(property "Footprint" "tronixio:TO-263-5-TABPIN3"
 			(at 129.54 55.88 0)
 			(effects

Commit message: Up
Parts:
- K101: footprint tronixio:CUI-PJ-102AH -> tronixio:SSD-PJ-102AH; symbol tronixio:CUI-PJ-102AH-TH -> tronixio:SSD-PJ-102AH-TH
Changed lines of the file:
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@@
 		(property "Reference" "K102"
 			(at 78.74 52.705 0)
+			(do_not_autoplace yes)
 			(effects
 				(font
@@
 		(property "Value" "AC/DC 9-12V"
 			(at 78.74 61.595 0)
+			(do_not_autoplace yes)
 			(effects
 				(font
@@
 		)
 		(property "Description" "2~24 Poles, Screw Type, Horizontal, 5.08 Pitch, 26~14 (AWG), Terminal Block Connector"
-			(at 78.74 55.88 0)
-			(effects
-				(font
-					(size 1.27 1.27)
+			(at 78.74 71.12 0)
+			(do_not_autoplace yes)
+			(effects
+				(font
+					(size 1 1)
 				)
 				(hide yes)
@@
 		)
 		(property "Mouser" "490-TB006-508-02BE"
-			(at 78.74 71.12 0)
+			(at 78.74 73.66 0)
 			(do_not_autoplace yes)
 			(effects
@@
 	)
 	(symbol
-		(lib_id "tronixio:CUI-PJ-102AH-TH")
+		(lib_id "tronixio:SSD-PJ-102AH-TH")
 		(at 78.74 43.18 0)
 		(unit 1)
@@
 			)
 		)
-		(property "Footprint" "tronixio:CUI-PJ-102AH"
+		(property "Footprint" "tronixio:SSD-PJ-102AH"
 			(at 78.74 50.8 0)
 			(do_not_autoplace yes)
@@
 			)
 		)
-		(property "Datasheet" "https://www.cuidevices.com/product/interconnect/connectors/dc-power-connectors/jacks/pj-102ah"
+		(property "Datasheet" "https://www.sameskydevices.com/product/interconnect/connectors/dc-power-connectors/jacks/pj-102ah"
 			(at 78.74 53.34 0)
 			(do_not_autoplace yes)
