File: Kicad/trainer/pic8bit-mcu.kicad_sch (KiCad schematic)
At the start: 16 parts, among them IC201 MICROCHIP-PIC16F1778-ISP, K201 MCU 1, K202 MCU 2, K203 ICSP

Commit message: Update
Parts:
- *X1: MOUSER 575-144308 -> (none); Mouser (none) -> 575-144308
- C203: value 100n -> C-0805
- IC201: MOUSER 579-PIC16F1778-I/SP -> (none); Mouser (none) -> 579-PIC16F1778-I/SP
- JP201, JP202, JP203: MOUSER 855-M20-999024 -> (none); Mouser (none) -> 855-M20-999024
- K201, K202: MOUSER 855-M20-782144 -> (none); Mouser (none) -> 855-M20-782144
- K203: MOUSER 200-SSW10602TSRA -> (none); Mouser (none) -> 200-SSW10602TSRA
- S201: MOUSER 611-KSA0M911LFT -> (none); Mouser (none) -> 611-KSA0M911LFT
Connections:
- no-connect marks 1 -> 0
Changed lines of the file:
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@@
   (junction (at 101.6 45.72) (diameter 0.9144) (color 0 0 0 0)
   )
-  (no_connect (at 208.28 144.78))
   (wire (pts (xy 170.18 71.12) (xy 203.2 71.12))
     (stroke (width 0) (type solid) (color 0 0 0 0))
@@
     (effects (font (size 1 1)) (justify left bottom))
   )
-  (hierarchical_label "RC5{slash}MOSI" (shape input) (at 210.82 116.84 0)
+  (hierarchical_label "RC5{slash}MOSI" (shape output) (at 210.82 116.84 0)
     (effects (font (size 1.15 1.15)) (justify left))
   )
@@
     (effects (font (size 1.15 1.15)) (justify right))
   )
-  (hierarchical_label "RC2{slash}I2C_RESET" (shape input) (at 76.2 121.92 180)
+  (hierarchical_label "RC2{slash}I2C_RESET" (shape output) (at 76.2 121.92 180)
     (effects (font (size 1.15 1.15)) (justify right))
   )
-  (hierarchical_label "RB5{slash}UCTS" (shape input) (at 210.82 106.68 0)
+  (hierarchical_label "RB5{slash}UCTS" (shape output) (at 210.82 106.68 0)
     (effects (font (size 1.15 1.15)) (justify left))
   )
@@
     (effects (font (size 1.15 1.15)) (justify right))
   )
-  (hierarchical_label "RA2{slash}SPI_RESET" (shape input) (at 76.2 111.76 180)
+  (hierarchical_label "RA2{slash}SPI_RESET" (shape output) (at 76.2 111.76 180)
     (effects (font (size 1.15 1.15)) (justify right))
   )
-  (hierarchical_label "RA5{slash}SPI_CS" (shape input) (at 76.2 116.84 180)
+  (hierarchical_label "RA5{slash}SPI_CS" (shape output) (at 76.2 116.84 180)
     (effects (font (size 1.15 1.15)) (justify right))
   )
-  (hierarchical_label "RA1{slash}SPI_CS2" (shape input) (at 76.2 109.22 180)
+  (hierarchical_label "RA1{slash}SPI_CS2" (shape output) (at 76.2 109.22 180)
     (effects (font (size 1.15 1.15)) (justify right))
   )
-  (hierarchical_label "RA0{slash}SPI_SC3" (shape input) (at 76.2 106.68 180)
+  (hierarchical_label "RA0{slash}SPI_SC3" (shape output) (at 76.2 106.68 180)
     (effects (font (size 1.15 1.15)) (justify right))
   )
-  (hierarchical_label "RC3{slash}SCL{slash}SCK" (shape input) (at 76.2 124.46 180)
+  (hierarchical_label "RC3{slash}SCL{slash}SCK" (shape output) (at 76.2 124.46 180)
     (effects (font (size 1.15 1.15)) (justify right))
   )
@@
     (effects (font (size 1.15 1.15)) (justify left))
   )
-  (hierarchical_label "RC6{slash}UTX" (shape input) (at 210.82 114.3 0)
+  (hierarchical_label "RC6{slash}UTX" (shape output) (at 210.82 114.3 0)
     (effects (font (size 1.15 1.15)) (justify left))
   )
@@
       (effects (font (size 1 1)) hide)
     )
-    (property "MOUSER" "855-M20-999024" (id 4) (at 121.92 119.38 0)
+    (property "Mouser" "855-M20-999024" (id 4) (at 121.92 119.38 0)
       (effects (font (size 1 1)) hide)
     )
@@
       (effects (font (size 1 1)) hide)
     )
-    (property "MOUSER" "855-M20-782144" (id 4) (at 76.2 106.68 0)
+    (property "Mouser" "855-M20-782144" (id 4) (at 76.2 106.68 0)
       (effects (font (size 1 1)) hide)
     )
@@
       (effects (font (size 1.15 1.15)) (justify left))
     )
-    (property "Value" "100n" (id 1) (at 178.435 114.3 0)
+    (property "Value" "C-0805" (id 1) (at 178.435 114.3 0)
       (effects (font (size 1.15 1.15)) (justify left))
     )
@@
       (effects (font (size 1 1)) hide)
     )
-    (property "MOUSER" "855-M20-999024" (id 4) (at 182.88 71.12 0)
+    (property "Mouser" "855-M20-999024" (id 4) (at 182.88 71.12 0)
       (effects (font (size 1 1)) hide)
     )
@@
       (effects (font (size 1 1)) hide)
     )
-    (property "MOUSER" "200-SSW10602TSRA" (id 4) (at 210.82 157.48 0)
-      (effects (font (size 1 1)) hide)
-    )
     (property "Name" "ICSP" (id 5) (at 210.82 147.32 0)
       (effects (font (size 1.15 1.15)))
+    )
+    (property "Mouser" "200-SSW10602TSRA" (id 6) (at 210.82 157.48 0)
+      (effects (font (size 1 1)) hide)
     )
     (pin "1")
@@
       (effects (font (size 1 1)) hide)
     )
-    (property "Datasheet" "https://www.microchip.com/en-us/product/PIC18F27Q43" (id 3) (at 154.94 105.41 0)
-      (effects (font (size 1 1)) hide)
-    )
-    (property "MOUSER" "579-PIC16F1778-I/SP" (id 4) (at 154.94 107.95 0)
+    (property "Datasheet" "https://www.microchip.com/en-us/product/PIC16F1778" (id 3) (at 154.94 105.41 0)
       (effects (font (size 1 1)) hide)
     )
     (property "Name" "PIC16F1778-ISP" (id 5) (at 167.64 59.69 0)
       (effects (font (size 1.15 1.15)) (justify right))
+    )
+    (property "Mouser" "579-PIC16F1778-I/SP" (id 6) (at 154.94 107.95 0)
+      (effects (font (size 1 1)) hide)
     )
     (pin "1")
@@
       (effects (font (size 1 1)) hide)
     )
-    (property "MOUSER" "855-M20-999024" (id 4) (at 132.08 71.12 0)
+    (property "Mouser" "855-M20-999024" (id 4) (at 132.08 71.12 0)
       (effects (font (size 1 1)) hide)
     )
@@
       (effects (font (size 1 1)) hide)
     )
-    (property "MOUSER" "611-KSA0M911LFT" (id 4) (at 106.68 50.8 0)
+    (property "Mouser" "611-KSA0M911LFT" (id 4) (at 106.68 50.8 0)
       (effects (font (size 1 1)) hide)
     )
@@
       (effects (font (size 1 1)) hide)
     )
-    (property "MOUSER" "575-144308" (id 4) (at 109.22 127 0)
+    (property "Mouser" "575-144308" (id 4) (at 109.22 124.46 0)
       (effects (font (size 1 1)) hide)
     )
@@
       (effects (font (size 1 1)) hide)
     )
-    (property "MOUSER" "855-M20-782144" (id 4) (at 210.82 106.68 0)
-      (effects (font (size 1 1)) hide)
-    )
+    (property "Mouser" "855-M20-782144" (id 4) (at 210.82 106.68 0)
+      (effects (font (size 1 1)) hide)
+    )

Commit message: Up
Parts:
- C203: value C-0805 -> 100n
- K201, K202: footprint tronixio:zzHARWIN-M20-782144x -> tronixio:HARWIN-M20-782144x
- U201: renamed from IC201; Name PIC16F1778-ISP -> PIC16F/PIC18F
- renumbered *X1 to X1
Other:
- note added: "*"
- moved on the sheet: C201, C202, C203, JP201, JP202, JP203, K201, K202, K203, R201, R202, R203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

Commit message: Update
Parts:
- added K204: VIN, tronixio:zzHARWIN-M20-782044x, symbol tronixio:HARWIN-254-F-1X04-VERTICAL
- added K205: VIN, tronixio:HARWIN-M20-999044x, symbol tronixio:HARWIN-254-M-1X04-VERTICAL
- added K206: VDD, tronixio:zzHARWIN-M20-782044x, symbol tronixio:HARWIN-254-F-1X04-VERTICAL
- added K207: GND, tronixio:zzHARWIN-M20-782044x, symbol tronixio:HARWIN-254-F-1X04-VERTICAL
- added K208: VDD, tronixio:HARWIN-M20-999044x, symbol tronixio:HARWIN-254-M-1X04-VERTICAL
- added K209: GND, tronixio:HARWIN-M20-999044x, symbol tronixio:HARWIN-254-M-1X04-VERTICAL
- added K210: SYMBOL-HEADER-F-1X10, tronixio:zzHARWIN-M20-782104x, symbol tronixio:SYMBOL-HEADER-F-1X10
Connections:
- net GND: now also K207.1, K207.2, K207.3, K207.4, K209.1, K209.2, K209.3, K209.4, K210.10 (Pin_10), K210.6 (Pin_6), K210.7 (Pin_7), K210.8 (Pin_8), K210.9 (Pin_9)
- net VCC: now also K206.1, K206.2, K206.3, K206.4, K208.1, K208.2, K208.3, K208.4, K210.1 (Pin_1), K210.2 (Pin_2), K210.3 (Pin_3), K210.4 (Pin_4), K210.5 (Pin_5)
- new net VIN: K204.1, K204.2, K204.3, K204.4, K205.1, K205.2, K205.3, K205.4

Commit message: Update
Parts:
- removed K210: SYMBOL-HEADER-F-1X10, tronixio:zzHARWIN-M20-782104x, symbol tronixio:SYMBOL-HEADER-F-1X10
- added K210: HARWIN-254-F-1X10-VERTICAL, tronixio:HARWIN-M20-782104x, symbol tronixio:HARWIN-254-F-1X10-VERTICAL
- C201, C203: footprint tronixio:zzzKEMET-C315 -> tronixio:KEMET-C315; symbol tronixio:C-0805 -> tronixio:CAPACITOR; Tolerance (none) -> 20%; Voltage (none) -> 50V
- C202: symbol tronixio:C-0805 -> tronixio:CAPACITOR; Tolerance (none) -> 20%; Voltage (none) -> 50V
- JP201: footprint tronixio:HARWIN-M20-975024x -> tronixio:HARWIN-M20-999024x; Name (none) -> HARWIN-254-M-1X02-JUMPER-VERTICAL
- JP202, JP203: Name (none) -> HARWIN-254-M-1X02-JUMPER-VERTICAL
- K201, K202: Name (none) -> HARWIN-254-F-1X14-VERTICAL
- K204, K206, K207: footprint tronixio:zzHARWIN-M20-782044x -> tronixio:HARWIN-M20-782044x; Name (none) -> HARWIN-254-F-1X04-VERTICAL
- K205, K208, K209: Name (none) -> HARWIN-254-M-1X04-VERTICAL
- R201, R202, R203, R204: symbol tronixio:R-0805 -> tronixio:RESISTOR; Tolerance (none) -> 5%
- S201: Name (none) -> CK-KSA
Connections:
- net GND: now also K210.10 (Pin_10), K210.6 (Pin_6), K210.7 (Pin_7), K210.8 (Pin_8), K210.9 (Pin_9)
- net VCC renamed VDD
- net VDD: now also K210.1 (Pin_1), K210.2 (Pin_2), K210.3 (Pin_3), K210.4 (Pin_4), K210.5 (Pin_5)

Commit message: Update
Parts:
- C201, C203: symbol tronixio:CAPACITOR -> tronixio:KEMET-C315-100N-254; Mouser (none) -> 80-C315C104M5U; Name (none) -> KEMET-C315-100N-254; Voltage 50V -> (none)
- C202: symbol tronixio:CAPACITOR -> tronixio:KEMET-C322-10U-508; Mouser (none) -> 80-C322C106K3R; Name (none) -> KEMET-C32210U-508; Tolerance 20% -> 10%; Voltage 50V -> (none)
- JP201: footprint tronixio:HARWIN-M20-999024x -> tronixio:HARWIN-M20-975024x; symbol tronixio:HARWIN-254-M-1X02-JUMPER-VERTICAL -> tronixio:HARWIN-254-M-1X02-JUMPER-HORIZONTAL; Mouser 855-M20-999024 -> 855-M20-975024
- K203: Name ICSP -> MICROCHIP-ICSP-F-1X06
- R201: symbol tronixio:RESISTOR -> tronixio:RESISTOR-1016TH-10K; Mouser (none) -> 594-SFR2500001002JA5; Name (none) -> RESISTOR-1016TH-10K
- R202: symbol tronixio:RESISTOR -> tronixio:RESISTOR-1016TH-1K; Mouser (none) -> 594-SFR2500001001JR5; Name (none) -> RESISTOR-1016TH-1K
- R203, R204: symbol tronixio:RESISTOR -> tronixio:RESISTOR-1016TH-4K7; Mouser (none) -> 594-SFR2500004701JR5; Name (none) -> RESISTOR-1016TH-4K7
- U201: value MICROCHIP-PIC16F1778-ISP -> PIC16F/18F; Name PIC16F/PIC18F -> MICROCHIP-PIC16F1778-ISP

Commit message: Update
Parts:
- X1: Name (none) -> XTAL-DIL08
Changed lines of the file:
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@@
   (junction (at 83.82 73.66) (diameter 0) (color 0 0 0 0)
   )
-  (junction (at 88.9 55.88) (diameter 0.9144) (color 0 0 0 0)
-  )
   (junction (at 121.92 175.26) (diameter 0) (color 0 0 0 0)
   )
   (junction (at 200.66 68.58) (diameter 0) (color 0 0 0 0)
   )
+  (junction (at 88.9 45.72) (diameter 0) (color 0 0 0 0)
+  )
   (junction (at 137.16 177.8) (diameter 0) (color 0 0 0 0)
   )
@@
   (junction (at 106.68 157.48) (diameter 0) (color 0 0 0 0)
   )
-  (junction (at 88.9 45.72) (diameter 0.9144) (color 0 0 0 0)
-  )
   (junction (at 167.64 86.36) (diameter 0) (color 0 0 0 0)
   )
@@
   (junction (at 185.42 63.5) (diameter 0) (color 0 0 0 0)
   )
+  (junction (at 91.44 45.72) (diameter 0) (color 0 0 0 0)
+  )
   (junction (at 121.92 157.48) (diameter 0) (color 0 0 0 0)
   )
@@
   (junction (at 76.2 154.94) (diameter 0) (color 0 0 0 0)
   )
+  (junction (at 88.9 55.88) (diameter 0) (color 0 0 0 0)
+  )
   (junction (at 76.2 160.02) (diameter 0) (color 0 0 0 0)
   )
-  (junction (at 91.44 45.72) (diameter 0.9144) (color 0 0 0 0)
-  )
   (junction (at 109.22 86.36) (diameter 0) (color 0 0 0 0)
   )
@@
     (stroke (width 0) (type default) (color 0 0 0 0))
   )
-  (wire (pts (xy 91.44 54.61) (xy 91.44 55.88))
-    (stroke (width 0) (type solid) (color 0 0 0 0))
-  )
   (wire (pts (xy 106.68 172.72) (xy 106.68 175.26))
     (stroke (width 0) (type default) (color 0 0 0 0))
@@
     (stroke (width 0) (type solid) (color 0 0 0 0))
   )
-  (wire (pts (xy 88.9 45.72) (xy 88.9 46.99))
-    (stroke (width 0) (type solid) (color 0 0 0 0))
-  )
   (wire (pts (xy 71.12 106.68) (xy 76.2 106.68))
     (stroke (width 0) (type default) (color 0 0 0 0))
@@
     (stroke (width 0) (type default) (color 0 0 0 0))
   )
+  (wire (pts (xy 88.9 55.88) (xy 91.44 55.88))
+    (stroke (width 0) (type default) (color 0 0 0 0))
+  )
   (wire (pts (xy 86.36 78.74) (xy 134.62 78.74))
     (stroke (width 0) (type default) (color 0 0 0 0))
@@
     (stroke (width 0) (type solid) (color 0 0 0 0))
   )
+  (wire (pts (xy 88.9 45.72) (xy 91.44 45.72))
+    (stroke (width 0) (type default) (color 0 0 0 0))
+  )
   (wire (pts (xy 185.42 139.7) (xy 203.2 139.7))
     (stroke (width 0) (type default) (color 0 0 0 0))
@@
     (stroke (width 0) (type solid) (color 0 0 0 0))
   )
-  (wire (pts (xy 88.9 57.15) (xy 88.9 55.88))
-    (stroke (width 0) (type solid) (color 0 0 0 0))
-  )
   (wire (pts (xy 165.1 91.44) (xy 193.04 91.44))
     (stroke (width 0) (type solid) (color 0 0 0 0))
@@
     (stroke (width 0) (type default) (color 0 0 0 0))
   )
+  (wire (pts (xy 88.9 55.88) (xy 88.9 57.15))
+    (stroke (width 0) (type default) (color 0 0 0 0))
+  )
   (wire (pts (xy 76.2 162.56) (xy 76.2 160.02))
     (stroke (width 0) (type default) (color 0 0 0 0))
@@
     (stroke (width 0) (type default) (color 0 0 0 0))
   )
-  (wire (pts (xy 91.44 45.72) (xy 88.9 45.72))
-    (stroke (width 0) (type solid) (color 0 0 0 0))
-  )
   (wire (pts (xy 91.44 154.94) (xy 91.44 152.4))
     (stroke (width 0) (type default) (color 0 0 0 0))
@@
     (stroke (width 0) (type default) (color 0 0 0 0))
   )
-  (wire (pts (xy 91.44 45.72) (xy 91.44 46.99))
-    (stroke (width 0) (type solid) (color 0 0 0 0))
-  )
   (wire (pts (xy 73.66 96.52) (xy 93.98 96.52))
     (stroke (width 0) (type default) (color 0 0 0 0))
@@
     (stroke (width 0) (type default) (color 0 0 0 0))
   )
-  (wire (pts (xy 88.9 54.61) (xy 88.9 55.88))
-    (stroke (width 0) (type solid) (color 0 0 0 0))
-  )
   (wire (pts (xy 116.84 114.3) (xy 116.84 119.38))
     (stroke (width 0) (type solid) (color 0 0 0 0))
@@
   )
   (wire (pts (xy 187.96 96.52) (xy 203.2 96.52))
-    (stroke (width 0) (type solid) (color 0 0 0 0))
-  )
-  (wire (pts (xy 91.44 55.88) (xy 88.9 55.88))
     (stroke (width 0) (type solid) (color 0 0 0 0))
   )
@@
       (effects (font (size 1 1)) hide)
     )
-    (property "Tolerance" "20%" (id 5) (at 173.355 116.84 0)
+    (property "Tolerance" "20%" (id 5) (at 173.99 116.84 0)
       (effects (font (size 1.15 1.15)) (justify left) hide)
     )
@@
     )
     (property "Name" "KEMET-C315-100N-254" (id 7) (at 172.72 121.92 0)
-      (effects (font (size 1 1)))
+      (effects (font (size 1 1)) hide)
     )
     (pin "1")
@@
     (pin "1")
   )
-  (symbol (lib_name "RESISTOR-1016TH-4K7_1") (lib_id "tronixio:RESISTOR-1016TH-4K7") (at 127 43.18 0) (unit 1)
+  (symbol (lib_id "tronixio:RESISTOR-1016TH-4K7") (at 127 43.18 0) (unit 1)
     (in_bom yes) (on_board yes)
     (property "Reference" "R203" (id 0) (at 126.365 39.37 0)
@@
       (effects (font (size 1 1)) hide)
     )
-    (property "Tolerance" "20%" (id 5) (at 97.155 55.88 0)
+    (property "Tolerance" "20%" (id 5) (at 97.79 55.88 0)
       (effects (font (size 1.15 1.15)) (justify left) hide)
     )
@@
     )
     (property "Name" "KEMET-C315-100N-254" (id 7) (at 96.52 60.96 0)
-      (effects (font (size 1 1)))
+      (effects (font (size 1 1)) hide)
     )
     (pin "1")
@@
       (effects (font (size 1.15 1.15)))
     )
-    (property "Value" "ICSP" (id 1) (at 205.74 149.86 0)
+    (property "Value" "ICSP" (id 1) (at 205.74 147.32 0)
       (effects (font (size 1.15 1.15)))
     )
@@
       (effects (font (size 1.15 1.15)) (justify right))
     )
-    (property "Footprint" "tronixio:DIP-28-W762-SOCKET" (id 2) (at 149.86 104.14 0)
-      (effects (font (size 1 1)) hide)
-    )
-    (property "Datasheet" "https://www.microchip.com/en-us/product/PIC16F1778" (id 3) (at 149.86 106.68 0)
-      (effects (font (size 1 1)) hide)
-    )
-    (property "Name" "MICROCHIP-PIC16F1778-ISP" (id 5) (at 149.86 59.69 0)
-      (effects (font (size 1 1)) hide)
-    )
-    (property "Mouser" "579-PIC16F1778-I/SP" (id 6) (at 149.86 109.22 0)
+    (property "Footprint" "tronixio:DIP-28-W762-SOCKET" (id 2) (at 134.62 106.68 0)
+      (effects (font (size 1 1)) hide)
+    )
+    (property "Datasheet" "https://www.microchip.com/en-us/product/PIC16F1778" (id 3) (at 134.62 109.22 0)
+      (effects (font (size 1 1)) hide)
+    )
+    (property "Name" "MICROCHIP-PIC16F1778-ISP" (id 5) (at 134.62 104.14 0)
+      (effects (font (size 1 1)) hide)
+    )
+    (property "Mouser" "579-PIC16F1778-I/SP" (id 6) (at 134.62 111.76 0)
       (effects (font (size 1 1)) hide)
     )
@@
       (effects (font (size 1 1)) hide)
     )
-    (property "Tolerance" "10%" (id 5) (at 117.475 116.84 0)
+    (property "Tolerance" "10%" (id 5) (at 118.11 116.84 0)
       (effects (font (size 1.15 1.15)) (justify left) hide)
     )
@@
       (effects (font (size 1.15 1.15)) (justify right))
     )
-    (property "Footprint" "tronixio:CK-KSA-TH" (id 2) (at 99.06 50.8 0)
-      (effects (font (size 1 1)) hide)
-    )
-    (property "Datasheet" "http://www.ckswitches.com/products/switches/product-details/Tactile/KSA/" (id 3) (at 101.6 50.8 0)
-      (effects (font (size 1 1)) hide)
-    )
-    (property "Mouser" "611-KSA0M911LFT" (id 4) (at 104.14 50.8 0)
-      (effects (font (size 1 1)) hide)
-    )
-    (property "Name" "CK-KSA" (id 5) (at 96.52 50.8 0)
+    (property "Footprint" "tronixio:CK-KSA-TH" (id 2) (at 96.52 50.8 0)
+      (effects (font (size 1 1)) hide)
+    )
+    (property "Datasheet" "http://www.ckswitches.com/products/switches/product-details/Tactile/KSA/" (id 3) (at 99.06 50.8 0)
+      (effects (font (size 1 1)) hide)
+    )
+    (property "Mouser" "611-KSA0M911LFT" (id 4) (at 101.6 50.8 0)
+      (effects (font (size 1 1)) hide)
+    )
+    (property "Name" "CK-KSA" (id 5) (at 93.98 50.8 0)
       (effects (font (size 1 1)) hide)
     )
@@
       (effects (font (size 1.15 1.15)) hide)
     )
-    (property "Footprint" "tronixio:DIP-08-W762-SOCKET" (id 2) (at 104.14 121.92 0)
+    (property "Footprint" "tronixio:DIP-08-W762-SOCKET" (id 2) (at 104.14 123.19 0)
       (effects (font (size 1 1)) hide)
     )
@@
       (effects (font (size 1 1)) hide)
     )
-    (property "Mouser" "575-144308" (id 4) (at 104.14 124.46 0)
-      (effects (font (size 1 1)) hide)
-    )
+    (property "Mouser" "575-144308" (id 4) (at 104.14 125.73 0)
+      (effects (font (size 1 1)) hide)
+    )
+    (property "Name" "XTAL-DIL08" (id 5) (at 104.14 120.65 0)
+      (effects (font (size 1 1)) hide)
+    )

Commit message: Update
Parts:
- R201, R202, R203, R204: footprint tronixio:RESISTOR-1016-TH -> tronixio:RESISTOR-TH-1016
- U201: footprint tronixio:DIP-28-W762-SOCKET -> tronixio:DIP-28-W762
Changed lines of the file:
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@@
       (effects (font (size 1.15 1.15)))
     )
-    (property "Footprint" "tronixio:RESISTOR-1016-TH" (id 2) (at 88.9 45.72 0)
+    (property "Footprint" "tronixio:RESISTOR-TH-1016" (id 2) (at 88.9 45.72 0)
       (effects (font (size 1 1)) hide)
     )
@@
       (effects (font (size 1 1)) hide)
     )
-    (property "Tolerance" "5%" (id 4) (at 102.87 48.26 0)
+    (property "Tolerance" "5%" (id 4) (at 100.33 48.26 0)
       (effects (font (size 1.15 1.15)) (justify left) hide)
     )
@@
       (effects (font (size 1.15 1.15)))
     )
-    (property "Footprint" "tronixio:RESISTOR-1016-TH" (id 2) (at 127 58.42 0)
+    (property "Footprint" "tronixio:RESISTOR-TH-1016" (id 2) (at 127 58.42 0)
       (effects (font (size 1 1)) hide)
     )
@@
       (effects (font (size 1 1)) hide)
     )
-    (property "Tolerance" "5%" (id 4) (at 129.54 44.45 0)
+    (property "Tolerance" "5%" (id 4) (at 129.54 46.99 0)
       (effects (font (size 1.15 1.15)) (justify left) hide)
     )
@@
     (pin "4")
   )
-  (symbol (lib_id "tronixio:RESISTOR-1016TH-4K7") (at 177.8 43.18 0) (unit 1)
+  (symbol (lib_name "RESISTOR-1016TH-4K7_1") (lib_id "tronixio:RESISTOR-1016TH-4K7") (at 177.8 43.18 0) (unit 1)
     (in_bom yes) (on_board yes)
     (property "Reference" "R204" (id 0) (at 178.435 39.37 0)
@@
       (effects (font (size 1.15 1.15)))
     )
-    (property "Footprint" "tronixio:RESISTOR-1016-TH" (id 2) (at 177.8 58.42 0)
+    (property "Footprint" "tronixio:RESISTOR-TH-1016" (id 2) (at 177.8 58.42 0)
       (effects (font (size 1 1)) hide)
     )
@@
       (effects (font (size 1 1)) hide)
     )
-    (property "Tolerance" "5%" (id 4) (at 180.34 44.45 0)
+    (property "Tolerance" "5%" (id 4) (at 180.34 46.99 0)
       (effects (font (size 1.15 1.15)) (justify left) hide)
     )
@@
       (effects (font (size 1.15 1.15)))
     )
-    (property "Footprint" "tronixio:RESISTOR-1016-TH" (id 2) (at 88.9 55.88 0)
+    (property "Footprint" "tronixio:RESISTOR-TH-1016" (id 2) (at 88.9 55.88 0)
       (effects (font (size 1 1)) hide)
     )
@@
       (effects (font (size 1 1)) hide)
     )
-    (property "Tolerance" "5%" (id 4) (at 86.36 41.91 0)
+    (property "Tolerance" "5%" (id 4) (at 86.36 44.45 0)
       (effects (font (size 1.15 1.15)) (justify left) hide)
     )
@@
       (effects (font (size 1.15 1.15)) (justify right))
     )
-    (property "Footprint" "tronixio:DIP-28-W762-SOCKET" (id 2) (at 134.62 106.68 0)
-      (effects (font (size 1 1)) hide)
-    )
-    (property "Datasheet" "https://www.microchip.com/en-us/product/PIC16F1778" (id 3) (at 134.62 109.22 0)
-      (effects (font (size 1 1)) hide)
-    )
-    (property "Name" "MICROCHIP-PIC16F1778-ISP" (id 5) (at 134.62 104.14 0)
-      (effects (font (size 1 1)) hide)
-    )
-    (property "Mouser" "579-PIC16F1778-I/SP" (id 6) (at 134.62 111.76 0)
-      (effects (font (size 1 1)) hide)
-    )
+    (property "Footprint" "tronixio:DIP-28-W762" (id 2) (at 149.86 106.68 0)
+      (effects (font (size 1 1)) hide)
+    )
+    (property "Datasheet" "https://www.microchip.com/en-us/product/PIC16F1778" (id 3) (at 149.86 109.22 0)
+      (effects (font (size 1 1)) hide)
+    )
+    (property "Name" "MICROCHIP-PIC16F1778-ISP" (id 5) (at 149.86 104.14 0)
+      (effects (font (size 1 1)) hide)
+    )
+    (property "Mouser" "579-PIC16F1778-I/SP" (id 6) (at 149.86 111.76 0)
+      (effects (font (size 1 1)) hide)
+    )

Commit message: Update
Other:
- moved on the sheet: C201, C202, C203, JP201, JP202, JP203, K201, K202, K203, K204, K205, K206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
