File: Kicad/trainer/pic8bit-mcu.kicad_sch (KiCad schematic)
At the start: 23 parts, among them K201 MCU 1, K202 MCU 2, K203 ICSP, K204 VIN, K205 VIN, K206 VDD, K207 GND, K208 VDD, K209 GND, K210 HARWIN-254-F-1X10-VERTICAL, U201 PIC16F/18F, X1 XTAL-DIL08

Commit message: Update
Parts:
- renumbered X1 to X201
Connections:
- net PGC: no longer names the net of K202.2 (Pin_2), K203.2, U201.27 (PGC/RB6)
- net PGD: no longer names the net of K202.1 (Pin_1), K203.3, U201.28 (PGD/RB7)
- net ~{MCLR}: no longer names the net of K201.1 (Pin_1), K203.6, R202.1, U201.1 (RE3/~{MCLR})
Other:
- moved on the sheet: C201, C202, C203, JP201, JP202, JP203, K201, K202, K203, K204, K205, K206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

Commit message: Update pic8bit trainer
Parts:
- C201, C203: symbol tronixio:KEMET-C315-100N-254 -> tronixio:KEMET-C315-0254-100N-50V-20P; Name KEMET-C315-100N-254 -> (none); Voltage (none) -> 50V
- C202: symbol tronixio:KEMET-C322-10U-508 -> tronixio:KEMET-C322-0508-10U-25V-10P; Name KEMET-C32210U-508 -> (none); Voltage (none) -> 25V
- JP201, JP202, JP203: Name HARWIN-254-M-1X02-JUMPER-VERTICAL -> (none)
- K201, K202: Name HARWIN-254-F-1X14-VERTICAL -> (none)
- K203: Name MICROCHIP-ICSP-F-1X06 -> (none)
- K204, K206, K207: Name HARWIN-254-F-1X04-VERTICAL -> (none)
- K205, K208, K209: Name HARWIN-254-M-1X04-VERTICAL -> (none)
- K210: Name HARWIN-254-F-1X10-VERTICAL -> (none)
- R201: Name RESISTOR-1016TH-10K -> (none)
- R202: Name RESISTOR-1016TH-1K -> (none)
- R203, R204: Name RESISTOR-1016TH-4K7 -> (none)
- S201: Name CK-KSA -> (none)
- U201: Name MICROCHIP-PIC16F1778-ISP -> (none)
- X201: Name XTAL-DIL08 -> (none)
Other:
- moved on the sheet: JP201, JP202, JP203

Commit message: Update
Parts:
- U201: footprint tronixio:DIP-28-W762 -> tronixio:DIP-28-W762-SOCKET
Changed lines of the file:
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@@
       (effects (font (size 1.15 1.15)) (justify right))
     )
-    (property "Footprint" "tronixio:DIP-28-W762" (at 157.48 104.14 0)
+    (property "Footprint" "tronixio:DIP-28-W762-SOCKET" (at 157.48 104.14 0)
       (effects (font (size 1 1)) hide)
     )

Commit message: Up
Parts:
- K203: symbol tronixio:MICROCHIP-ICSP-F-1X06 -> tronixio:MICROCHIP-ICSP-F-RIGHT-ANGLE-TH
- R201: symbol tronixio:RESISTOR-1016TH-10K -> tronixio:RESISTOR-1016TH-10K-5P
- R202: symbol tronixio:RESISTOR-1016TH-1K -> tronixio:RESISTOR-1016TH-1K-5P
- R203, R204: symbol tronixio:RESISTOR-1016TH-4K7 -> tronixio:RESISTOR-1016TH-4K7-5P
- U201: footprint tronixio:DIP-28-W762-SOCKET -> tronixio:DIP-28-W762
Connections:
- net VDD renamed +VDD
- net VIN renamed +VIN

Commit message: Up
Other:
- note added: "*X201: Optional mounted on DIL08"
- note removed: "*X1: Optional mounted on DIL08"
Changed lines of the file:
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@@
     (effects (font (size 1.15 1.15)) (justify left bottom))
   )
-  (text "*X1: Optional mounted on DIL08" (at 180.34 173.99 0)
+  (text "*X201: Optional mounted on DIL08" (at 180.34 173.99 0)
     (effects (font (size 1.27 1.27)) (justify left bottom))
   )

Commit message: Update
Connections:
- net GND: no longer X201.2, X201.7, X201.8
- net at K201.10 (Pin_10), U201.10 (RA6/CLKO), X201.5: no longer X201.6
- net at K201.9 (Pin_9), U201.9 (RA7/CLKI), X201.3: no longer X201.4
