File: Kicad/trainer/pic8bit-mcu.kicad_sch (KiCad schematic)
At the start: 23 parts, among them K201 MCU 1, K202 MCU 2, K203 ICSP, K204 VIN, K205 VIN, K206 VDD, K207 GND, K208 VDD, K209 GND, K210 HARWIN-254-F-1X10-VERTICAL, U201 PIC16F/18F, X201 XTAL-DIL08

Commit message: Update Trainer Kicad 8
Connections:
- net +VDD renamed POWER-VDD
- net +VIN renamed POWER-VIN
- net GND renamed POWER-GND

Commit message: Update Trainer
Connections:
- net POWER-GND: now also X201.2, X201.7, X201.8
- net at K201.10 (Pin_10), U201.10 (RA6/CLKO), X201.5: now also X201.6
- net at K201.9 (Pin_9), U201.9 (RA7/CLKI), X201.3: now also X201.4
Changed lines of the file:
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@@
 		(on_board yes)
 		(dnp no)
-		(fields_autoplaced yes)
 		(property "Reference" "#PWR0209"
 			(at 180.34 45.72 0)
@@
 			)
 		)
-		(property "Description" ""
-			(at 180.34 35.56 0)
-			(effects
-				(font
-					(size 1.27 1.27)
-				)
-				(hide yes)
-			)
-		)
-		(property "Name" "VDD"
+		(property "Description" "VDD"
 			(at 180.34 30.48 0)
-			(do_not_autoplace yes)
 			(effects
 				(font
-					(size 1.15 1.15)
+					(size 1.27 1.27)
 				)
 			)
@@
 			)
 		)
-		(property "Description" ""
-			(at 210.82 127 0)
-			(effects
-				(font
-					(size 1.27 1.27)
-				)
-				(hide yes)
-			)
-		)
-		(property "Name" "VDD"
+		(property "Description" "VDD"
 			(at 210.82 121.92 0)
-			(do_not_autoplace yes)
 			(effects
 				(font
-					(size 1.15 1.15)
+					(size 1.27 1.27)
 				)
 			)
@@
 			)
 		)
-		(property "Description" ""
-			(at 124.46 160.02 0)
-			(effects
-				(font
-					(size 1.27 1.27)
-				)
-				(hide yes)
-			)
-		)
-		(property "Name" "VDD"
+		(property "Description" "VDD"
 			(at 124.46 154.94 0)
-			(do_not_autoplace yes)
 			(effects
 				(font
-					(size 1.15 1.15)
+					(size 1.27 1.27)
 				)
 			)
@@
 			)
 		)
-		(property "Description" ""
-			(at 134.62 35.56 0)
-			(effects
-				(font
-					(size 1.27 1.27)
-				)
-				(hide yes)
-			)
-		)
-		(property "Name" "VDD"
+		(property "Description" "VDD"
 			(at 134.62 30.48 0)
-			(do_not_autoplace yes)
 			(effects
 				(font
-					(size 1.15 1.15)
+					(size 1.27 1.27)
 				)
 			)
@@
 			)
 		)
-		(property "Description" ""
-			(at 93.98 160.02 0)
-			(effects
-				(font
-					(size 1.27 1.27)
-				)
-				(hide yes)
-			)
-		)
-		(property "Name" "VIN"
+		(property "Description" "VIN"
 			(at 93.98 154.94 0)
-			(do_not_autoplace yes)
 			(effects
 				(font
-					(size 1.15 1.15)
+					(size 1.27 1.27)
 				)
 			)
@@
 		(on_board yes)
 		(dnp no)
-		(fields_autoplaced yes)
 		(property "Reference" "#PWR0201"
 			(at 96.52 45.72 0)
@@
 			)
 		)
-		(property "Description" ""
-			(at 96.52 35.56 0)
-			(effects
-				(font
-					(size 1.27 1.27)
-				)
-				(hide yes)
-			)
-		)
-		(property "Name" "VDD"
+		(property "Description" "VDD"
 			(at 96.52 30.48 0)
-			(do_not_autoplace yes)
 			(effects
 				(font
-					(size 1.15 1.15)
+					(size 1.27 1.27)
 				)
 			)
@@
 			)
 		)
-		(property "Description" ""
-			(at 78.74 160.02 0)
-			(effects
-				(font
-					(size 1.27 1.27)
-				)
-				(hide yes)
-			)
-		)
-		(property "Name" "VIN"
+		(property "Description" "VIN"
 			(at 78.74 154.94 0)
-			(do_not_autoplace yes)
 			(effects
 				(font
-					(size 1.15 1.15)
+					(size 1.27 1.27)
 				)
 			)
@@
 			)
 		)
-		(property "Description" ""
-			(at 139.7 160.02 0)
-			(effects
-				(font
-					(size 1.27 1.27)
-				)
-				(hide yes)
-			)
-		)
-		(property "Name" "VDD"
+		(property "Description" "VDD"
 			(at 139.7 154.94 0)
-			(do_not_autoplace yes)
 			(effects
 				(font
-					(size 1.15 1.15)
+					(size 1.27 1.27)
 				)
 			)
@@
 		(on_board yes)
 		(dnp no)
-		(fields_autoplaced yes)
 		(property "Reference" "#PWR0211"
 			(at 185.42 45.72 0)
@@
 			)
 		)
-		(property "Description" ""
-			(at 185.42 35.56 0)
-			(effects
-				(font
-					(size 1.27 1.27)
-				)
-				(hide yes)
-			)
-		)
-		(property "Name" "VDD"
+		(property "Description" "VDD"
 			(at 185.42 30.48 0)
-			(do_not_autoplace yes)
 			(effects
 				(font
-					(size 1.15 1.15)
+					(size 1.27 1.27)
 				)
 			)
@@
 			)
 		)
-		(property "Description" ""
-			(at 109.22 160.02 0)
-			(effects
-				(font
-					(size 1.27 1.27)
-				)
-				(hide yes)
-			)
-		)
-		(property "Name" "VDD"
+		(property "Description" "VDD"
 			(at 109.22 154.94 0)
-			(do_not_autoplace yes)
 			(effects
 				(font
-					(size 1.15 1.15)
+					(size 1.27 1.27)
 				)
 			)

Commit message: Update
Parts:
- U201: footprint tronixio:DIP-28-W762 -> tronixio:DIP-28-W762-SOCKET
Changed lines of the file:
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@@
 		(property "Reference" "U201"
 			(at 144.78 59.69 0)
+			(do_not_autoplace yes)
 			(effects
 				(font
@@
 		(property "Value" "PIC16F/18F"
 			(at 170.18 59.69 0)
+			(do_not_autoplace yes)
 			(effects
 				(font
@@
 			)
 		)
-		(property "Footprint" "tronixio:DIP-28-W762"
+		(property "Footprint" "tronixio:DIP-28-W762-SOCKET"
+			(at 157.48 101.6 0)
+			(do_not_autoplace yes)
+			(effects
+				(font
+					(size 1 1)
+				)
+				(hide yes)
+			)
+		)
+		(property "Datasheet" "https://www.microchip.com/en-us/product/PIC16F1778"
 			(at 157.48 104.14 0)
 			(do_not_autoplace yes)
@@
 			)
 		)
-		(property "Datasheet" "https://www.microchip.com/en-us/product/PIC16F1778"
-			(at 157.48 106.68 0)
+		(property "Description" "28/40/44-Pin, 8-Bit Flash Microcontroller"
+			(at 157.48 109.22 0)
 			(do_not_autoplace yes)
 			(effects
@@
 			)
 		)
-		(property "Description" "28/40/44-Pin, 8-Bit Flash Microcontroller"
-			(at 142.24 63.5 0)
-			(effects
-				(font
-					(size 1.27 1.27)
-				)
-				(hide yes)
-			)
-		)
 		(property "Mouser" "579-PIC16F1778-I/SP"
-			(at 157.48 109.22 0)
+			(at 157.48 106.68 0)
 			(do_not_autoplace yes)
 			(effects

Commit message: Up
Parts:
- U201: footprint tronixio:DIP-28-W762-SOCKET -> tronixio:DIP-28-W762
Changed lines of the file:
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@@
 			)
 		)
-		(property "Footprint" "tronixio:DIP-28-W762-SOCKET"
+		(property "Footprint" "tronixio:DIP-28-W762"
 			(at 157.48 101.6 0)
 			(do_not_autoplace yes)

Commit message: Up
Parts:
- K210: value HARWIN-254-F-1X10-VERTICAL -> VDD & GND
Changed lines of the file:
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@@
 			)
 		)
-		(property "Value" "HARWIN-254-F-1X10-VERTICAL"
+		(property "Value" "VDD & GND"
 			(at 134.62 158.75 0)
 			(effects
