File: Kicad/nano/pic8bit.kicad_sch (KiCad schematic)
At the start: 32 parts, among them IC3 ROHM-BU33SD5WG-500-SOT, K1 MCU 1, K2 MCU 2, K3 ICSP, K4 POWER & UART

Commit message: Update Nano
Parts:
- *IC1: value PIC16F/PIC18F -> (none)
- *IC2: value MCP2221A -> (none); symbol tronixio:MCP2221A-IST -> tronixio:MICROCHIP-MCP2221A-IST; MOUSER 579-MCP2221A-I/ST -> (none); Mouser (none) -> 579-MCP2221A-I/ST; Name (none) -> MCP2221A-IST
- *JP1, *JP2: MOUSER 855-M22-25102 -> (none); Mouser (none) -> 855-M22-25102
- *LED2, *LED3: MOUSER 604-APT2012LSECKJ4RV -> (none); Mouser (none) -> 604-APT2012LSECKJ4RV
- *MEMS1: MOUSER 998-1001CI2-024.5760 -> (none); Mouser (none) -> 998-1001CI2-024.5760
- F1: MOUSER 652-MF-NSMF050-2 -> (none); Mouser (none) -> 652-MF-NSMF050-2; Name (none) -> 500mA
- H1, H2: MOUSER 855-M22-19000 -> (none); Mouser (none) -> 855-M22-19000
- IC3: MOUSER 755-BU33SD5WG-TR -> (none); Mouser (none) -> 755-BU33SD5WG-TR
- K1, K2: MOUSER 200-TSW12022TS -> (none); Mouser (none) -> 200-TSW12022TS
- K3: MOUSER 855-M20-9980346 -> (none); Mouser (none) -> 855-M20-9980346; Name (none) -> ICSP
- K4: MOUSER 649-10118193-0001LF -> (none); Mouser (none) -> 649-10118193-0001LF
- LED1: MOUSER 604-APT2012LVBCD -> (none); Mouser (none) -> 604-APT2012LVBCD
- S1: MOUSER 688-SKRPACE010 -> (none); Mouser (none) -> 688-SKRPACE010
Changed lines of the file:
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@@
-    (stroke (width 0) (type solid) (color 0 0 0 0))
-  )
-  (bus (pts (xy 160.02 33.02) (xy 162.56 33.02))
     (stroke (width 0) (type solid) (color 0 0 0 0))
   )
@@
     (stroke (width 0) (type solid) (color 0 0 0 0))
   )
-  (bus (pts (xy 157.48 33.02) (xy 160.02 33.02))
-    (stroke (width 0) (type solid) (color 0 0 0 0))
-  )
   (wire (pts (xy 226.06 142.24) (xy 228.6 142.24))
     (stroke (width 0) (type solid) (color 0 0 0 0))
@@
     (stroke (width 0) (type solid) (color 0 0 0 0))
   )
-  (bus (pts (xy 66.04 33.02) (xy 157.48 33.02))
-    (stroke (width 0) (type solid) (color 0 0 0 0))
-  )
   (wire (pts (xy 53.34 152.4) (xy 63.5 152.4))
     (stroke (width 0) (type solid) (color 0 0 0 0))
@@
     (stroke (width 0) (type solid) (color 0 0 0 0))
   )
-  (bus (pts (xy 162.56 33.02) (xy 165.1 33.02))
+  (bus (pts (xy 66.04 33.02) (xy 185.42 33.02))
     (stroke (width 0) (type solid) (color 0 0 0 0))
   )
@@
   )
   (wire (pts (xy 165.1 60.96) (xy 175.26 60.96))
-    (stroke (width 0) (type solid) (color 0 0 0 0))
-  )
-  (bus (pts (xy 165.1 33.02) (xy 185.42 33.02))
     (stroke (width 0) (type solid) (color 0 0 0 0))
   )
@@
       (effects (font (size 1 1)) hide)
     )
-    (property "MOUSER" "855-M22-25102" (id 4) (at 180.34 137.16 0)
-      (effects (font (size 1 1)) hide)
-    )
-    (pin "1")
-    (pin "2")
-  )
-  (symbol (lib_id "tronixio:MCP2221A-IST") (at 127 142.24 0) (unit 1)
+    (property "Mouser" "855-M22-25102" (id 4) (at 180.34 137.16 0)
+      (effects (font (size 1 1)) hide)
+    )
+    (pin "1")
+    (pin "2")
+  )
+  (symbol (lib_id "tronixio:MICROCHIP-MCP2221A-IST") (at 127 142.24 0) (unit 1)
     (in_bom yes) (on_board yes)
     (property "Reference" "*IC2" (id 0) (at 119.38 128.27 0)
       (effects (font (size 1.15 1.15)) (justify left))
     )
-    (property "Value" "MCP2221A" (id 1) (at 134.62 128.27 0)
-      (effects (font (size 1.15 1.15)) (justify right))
-    )
-    (property "Footprint" "tronixio:TSSOP-14" (id 2) (at 127 157.48 0)
-      (effects (font (size 1 1)) hide)
-    )
-    (property "Datasheet" "https://www.microchip.com/wwwproducts/en/MCP2221A" (id 3) (at 127 157.48 0)
-      (effects (font (size 1 1)) hide)
-    )
-    (property "MOUSER" "579-MCP2221A-I/ST" (id 4) (at 127 160.02 0)
+    (property "Value" "" (id 1) (at 134.62 128.27 0)
+      (effects (font (size 1 1)) (justify right) hide)
+    )
+    (property "Footprint" "tronixio:TSSOP-14" (id 2) (at 127 162.56 0)
+      (effects (font (size 1 1)) hide)
+    )
+    (property "Datasheet" "https://www.microchip.com/wwwproducts/en/MCP2221A" (id 3) (at 127 165.1 0)
+      (effects (font (size 1 1)) hide)
+    )
+    (property "Name" "MCP2221A-IST" (id 5) (at 127 156.21 0)
+      (effects (font (size 1.15 1.15)))
+    )
+    (property "Mouser" "579-MCP2221A-I/ST" (id 6) (at 127 167.64 0)
       (effects (font (size 1 1)) hide)
     )
@@
       (effects (font (size 1 1)) hide)
     )
-    (property "MOUSER" "604-APT2012LSECKJ4RV" (id 4) (at 137.16 144.78 0)
+    (property "Mouser" "604-APT2012LSECKJ4RV" (id 4) (at 137.16 144.78 0)
       (effects (font (size 1 1)) hide)
     )
@@
       (effects (font (size 1 1)) hide)
     )
-    (property "MOUSER" "855-M22-19000" (id 4) (at 271.78 187.96 0)
+    (property "Mouser" "855-M22-19000" (id 4) (at 271.78 187.96 0)
       (effects (font (size 1 1)) hide)
     )
@@
       (effects (font (size 1 1)) hide)
     )
-    (property "MOUSER" "604-APT2012LSECKJ4RV" (id 4) (at 142.24 144.78 0)
+    (property "Mouser" "604-APT2012LSECKJ4RV" (id 4) (at 142.24 144.78 0)
       (effects (font (size 1 1)) hide)
     )
@@
       (effects (font (size 1 1)) hide)
     )
-    (property "MOUSER" "649-10118193-0001LF" (id 4) (at 88.9 167.64 0)
+    (property "Mouser" "649-10118193-0001LF" (id 4) (at 88.9 167.64 0)
       (effects (font (size 1 1)) hide)
     )
@@
       (effects (font (size 1 1)) hide)
     )
-    (property "MOUSER" "998-1001CI2-024.5760" (id 4) (at 246.38 82.55 0)
-      (effects (font (size 1 1)) hide)
-    )
     (property "Name" "24.5760MHz" (id 5) (at 246.38 72.39 0)
-      (effects (font (size 1.15 1.15)) hide)
+      (effects (font (size 1.15 1.15)))
+    )
+    (property "Mouser" "998-1001CI2-024.5760" (id 5) (at 246.38 82.55 0)
+      (effects (font (size 1 1)) hide)
     )
     (pin "1")
@@
       (effects (font (size 1 1)) hide)
     )
-    (property "MOUSER" "855-M22-25102" (id 4) (at 180.34 139.7 0)
+    (property "Mouser" "855-M22-25102" (id 4) (at 180.34 139.7 0)
       (effects (font (size 1 1)) hide)
     )
@@
       (effects (font (size 1.15 1.15)))
     )
-    (property "Footprint" "tronixio:HARWIN-M20-998034x" (id 2) (at 246.38 104.14 0)
-      (effects (font (size 1 1)) hide)
-    )
-    (property "Datasheet" "https://ww1.microchip.com/downloads/en/DeviceDoc/30277d.pdf" (id 3) (at 247.65 104.14 0)
-      (effects (font (size 1 1)) hide)
-    )
-    (property "MOUSER" "855-M20-9980346" (id 4) (at 247.65 106.68 0)
+    (property "Footprint" "tronixio:HARWIN-M20-998034x" (id 2) (at 247.65 104.14 0)
+      (effects (font (size 1 1)) hide)
+    )
+    (property "Datasheet" "https://ww1.microchip.com/downloads/en/DeviceDoc/30277d.pdf" (id 3) (at 247.65 106.68 0)
+      (effects (font (size 1 1)) hide)
+    )
+    (property "Name" "ICSP" (id 4) (at 247.65 99.06 0)
+      (effects (font (size 1.15 1.15)))
+    )
+    (property "Mouser" "855-M20-9980346" (id 5) (at 247.65 109.22 0)
       (effects (font (size 1 1)) hide)
     )
@@
       (effects (font (size 1 1)) hide)
     )
-    (property "MOUSER" "604-APT2012LVBCD" (id 4) (at 228.6 147.32 0)
+    (property "Mouser" "604-APT2012LVBCD" (id 4) (at 228.6 147.32 0)
       (effects (font (size 1 1)) hide)
     )
@@
       (effects (font (size 1.15 1.15)))
     )
-    (property "Footprint" "tronixio:FUSE-0805" (id 2) (at 99.06 144.78 0)
-      (effects (font (size 1 1)) hide)
-    )
-    (property "Datasheet" "https://www.bourns.com/pdfs/mfnsmf.pdf" (id 3) (at 99.06 147.32 0)
-      (effects (font (size 1 1)) hide)
-    )
-    (property "MOUSER" "652-MF-NSMF050-2" (id 4) (at 99.06 149.86 0)
+    (property "Footprint" "tronixio:FUSE-0805" (id 2) (at 99.06 147.32 0)
+      (effects (font (size 1 1)) hide)
+    )
+    (property "Datasheet" "https://www.bourns.com/pdfs/mfnsmf.pdf" (id 3) (at 99.06 149.86 0)
+      (effects (font (size 1 1)) hide)
+    )
+    (property "Name" "500mA" (id 4) (at 99.06 142.24 0)
+      (effects (font (size 1.15 1.15)))
+    )
+    (property "Mouser" "652-MF-NSMF050-2" (id 5) (at 99.06 152.4 0)
       (effects (font (size 1 1)) hide)
     )
@@
       (effects (font (size 1 1)) hide)
     )
-    (property "MOUSER" "855-M22-19000" (id 4) (at 276.86 187.96 0)
+    (property "Mouser" "855-M22-19000" (id 4) (at 276.86 187.96 0)
       (effects (font (size 1 1)) hide)
     )
@@
       (effects (font (size 1 1)) hide)
     )
-    (property "MOUSER" "200-TSW12022TS" (id 4) (at 50.8 170.18 0)
+    (property "Mouser" "200-TSW12022TS" (id 4) (at 50.8 170.18 0)
       (effects (font (size 1 1)) hide)
     )
@@
       (effects (font (size 1 1)) hide)
     )
-    (property "MOUSER" "688-SKRPACE010" (id 4) (at 246.38 43.18 0)
+    (property "Mouser" "688-SKRPACE010" (id 4) (at 246.38 43.18 0)
       (effects (font (size 1 1)) hide)
     )
@@
       (effects (font (size 1 1)) hide)
     )
-    (property "MOUSER" "200-TSW12022TS" (id 4) (at 50.8 101.6 0)
+    (property "Mouser" "200-TSW12022TS" (id 4) (at 50.8 101.6 0)
       (effects (font (size 1 1)) hide)
     )
@@
       (effects (font (size 1.15 1.15)))
     )
-    (property "Value" "PIC16F/PIC18F" (id 1) (at 195.58 68.58 0)
-      (effects (font (size 1.15 1.15)))
-    )
-    (property "Footprint" "tronixio:TQFP-44" (id 2) (at 198.12 86.36 0)
+    (property "Value" "" (id 1) (at 195.58 68.58 0)
+      (effects (font (size 1.15 1.15)))
+    )
+    (property "Footprint" "tronixio:TQFP-44" (id 2) (at 195.58 96.52 0)
       (effects (font (size 1 1)) hide)
     )
@@
       (effects (font (size 1 1)) hide)
     )
-    (property "MOUSER" "755-BU33SD5WG-TR" (id 4) (at 218.44 157.48 0)
-      (effects (font (size 1 1)) hide)
-    )
     (property "Name" "BU33SD5WG" (id 5) (at 218.44 135.89 0)
       (effects (font (size 1.15 1.15)))
     )
-    (pin "1")
+    (property "Mouser" "755-BU33SD5WG-TR" (id 5) (at 218.44 157.48 0)
+      (effects (font (size 1 1)) hide)
+    )
+    (pin "1")

Commit message: Upadte
Parts:
- *IC1: value (none) -> PIC16F/PIC18F
- *IC2: value (none) -> MCP2221A
Other:
- moved on the sheet: *C2, *C5, *IC1, *IC2, *JP1, *JP2, *LED2, *LED3, *MEMS1, *R3, *R4, *R5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

Commit message: Up
Parts:
- renumbered *IC1 to U1, *IC2 to U2, IC3 to U3
Other:
- note added: "*U1: Check the pinout for the desired MCU family."
- note removed: "*IC1: Check the pinout for the desired MCU family."
Changed lines of the file:
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@@
     (effects (font (size 1.27 1.27)) (justify right bottom))
   )
-  (text "*IC1: Check the pinout for the desired MCU family."
-    (at 180.34 168.91 0)
+  (text "*U1: Check the pinout for the desired MCU family." (at 180.34 168.91 0)
     (effects (font (size 1.27 1.27)) (justify left bottom))
   )
@@
   (symbol (lib_id "tronixio:MICROCHIP-MCP2221A-IST") (at 121.92 142.24 0) (unit 1)
     (in_bom yes) (on_board yes)
-    (property "Reference" "*IC2" (id 0) (at 114.3 128.27 0)
+    (property "Reference" "U2" (id 0) (at 114.3 128.27 0)
       (effects (font (size 1.15 1.15)) (justify left))
     )
@@
   (symbol (lib_id "tronixio:SYMBOL-PIC8BIT-TQFP-44") (at 190.5 66.04 0) (unit 1)
     (in_bom yes) (on_board yes)
-    (property "Reference" "*IC1" (id 0) (at 190.5 63.5 0)
+    (property "Reference" "U1" (id 0) (at 190.5 63.5 0)
       (effects (font (size 1.15 1.15)))
     )
@@
   (symbol (lib_id "tronixio:ROHM-BU33SD5WG-500-SOT") (at 213.36 142.24 0) (unit 1)
     (in_bom yes) (on_board yes)
-    (property "Reference" "IC3" (id 0) (at 213.36 133.35 0)
+    (property "Reference" "U3" (id 0) (at 213.36 133.35 0)
       (effects (font (size 1.15 1.15)))
     )
@@
       (reference "*C5") (unit 1) (value "10µ") (footprint "tronixio:CAPACITOR-0805")
     )
-    (path "/db1cc9a9-8b98-44a9-9739-971dd0953aad"
-      (reference "*IC1") (unit 1) (value "PIC16F/PIC18F") (footprint "tronixio:TQFP-44")
-    )
-    (path "/15b76320-9a6e-4ed9-be26-15ea028b6641"
-      (reference "*IC2") (unit 1) (value "MCP2221A") (footprint "tronixio:TSSOP-14")
-    )
     (path "/11fdfe8d-ab60-4c39-986c-736a762545a1"
       (reference "*JP1") (unit 1) (value "SCL") (footprint "tronixio:HARWIN-M22-25102xx")
@@
       (reference "H2") (unit 1) (value "HARWIN-JUMPER-0200-03MM-BLACK") (footprint "tronixio:HARWIN-M22-190-193")
     )
-    (path "/ef27345a-c7c1-44c7-b4de-dc92b9c6de34"
-      (reference "IC3") (unit 1) (value "ROHM-BU33SD5WG-500-SOT") (footprint "tronixio:SOT-23-5")
-    )
     (path "/b98b70f3-e265-46ac-a952-ea805824e1b9"
       (reference "K1") (unit 1) (value "MCU 1") (footprint "tronixio:SAMTEC-TSW-120-22-T-S")
@@
       (reference "S1") (unit 1) (value "Reset") (footprint "tronixio:ALPS-SKRPAC")
     )
-  )
+    (path "/db1cc9a9-8b98-44a9-9739-971dd0953aad"
+      (reference "U1") (unit 1) (value "PIC16F/PIC18F") (footprint "tronixio:TQFP-44")
+    )
+    (path "/15b76320-9a6e-4ed9-be26-15ea028b6641"
+      (reference "U2") (unit 1) (value "MCP2221A") (footprint "tronixio:TSSOP-14")
+    )
+    (path "/ef27345a-c7c1-44c7-b4de-dc92b9c6de34"
+      (reference "U3") (unit 1) (value "ROHM-BU33SD5WG-500-SOT") (footprint "tronixio:SOT-23-5")
+    )
+  )

Commit message: Update
Parts:
- C1, C3, C4: symbol tronixio:C-0805 -> tronixio:CAPACITOR-0805-100N; Mouser (none) -> 80-C0805C104M5R; Name (none) -> CAPACITOR-0805-100N; Tolerance (none) -> 20%; Voltage (none) -> 50V
- C2: renamed from *C2; symbol tronixio:C-0805 -> tronixio:CAPACITOR-0805-100N; Mouser (none) -> 80-C0805C104M5R; Name (none) -> CAPACITOR-0805-100N; Tolerance (none) -> 20%; Voltage (none) -> 50V
- C5: renamed from *C5; symbol tronixio:C-0805 -> tronixio:CAPACITOR-0805-10U; Mouser (none) -> 80-C0805C106M3P; Name (none) -> CAPACITOR-0805-10U; Tolerance (none) -> 20%; Voltage (none) -> 25V
- C7, C8: symbol tronixio:C-0805 -> tronixio:CAPACITOR-0805-1U; Mouser (none) -> 80-C0805C105M5R; Name (none) -> CAPACITOR-0805-1U; Tolerance (none) -> 20%; Voltage (none) -> 50V
- F1: value F050 -> 500mA; Name 500mA -> BOURNS-FUSE-MF-NSMF050
- JP1: renamed from *JP1; Name (none) -> HARWIN-200-M-1X02-JUMPER-TH-VERTICAL
- JP2: renamed from *JP2; Name (none) -> HARWIN-200-M-1X02-JUMPER-TH-VERTICAL
- K1, K2: Name (none) -> SAMTEC-254-M-TSW-1X20-22-T-S
- K3: symbol tronixio:MICROCHIP-ICSP-M-2x03 -> tronixio:MICROCHIP-ICSP-M-2X03; Name ICSP -> MICROCHIP-ICSP-M-2X03
- K4: Name (none) -> FCI-USB-TYPE-B-MICRO-THT
- LED1: symbol tronixio:LED-0805-BLUE -> tronixio:KINGBRIGHT-LED-0805-BLUE; Name (none) -> KINGBRIGHT-LED-0805-BLUE
- LED2: renamed from *LED2; symbol tronixio:LED-0805-ORANGE -> tronixio:KINGBRIGHT-LED-0805-BLUE; Mouser 604-APT2012LSECKJ4RV -> 604-APT2012LVBCD; Name (none) -> KINGBRIGHT-LED-0805-BLUE
- LED3: renamed from *LED3; symbol tronixio:LED-0805-ORANGE -> tronixio:KINGBRIGHT-LED-0805-BLUE; Mouser 604-APT2012LSECKJ4RV -> 604-APT2012LVBCD; Name (none) -> KINGBRIGHT-LED-0805-BLUE
- MEMS1: renamed from *MEMS1; value MICROCHIP-DSC1001C-245760-CDFN -> DSC1001C; Name 24.5760MHz -> MICROCHIP-DSC1001C-245760-CDFN
- R1: value 10K -> 4K7; symbol tronixio:R-0805 -> tronixio:RESISTOR-0805-10K; Mouser (none) -> 660-RK73B2ATTDD103J; Name (none) -> RESISTOR-0805-10K; Tolerance (none) -> 5%
- R2: symbol tronixio:R-0805 -> tronixio:RESISTOR-0805-1K; Mouser (none) -> 660-RK73B2ATTDD102J; Name (none) -> RESISTOR-0805-1K; Tolerance (none) -> 5%
- R3: renamed from *R3; symbol tronixio:R-0805 -> tronixio:RESISTOR-0805-10K; Mouser (none) -> 660-RK73B2ATTDD103J; Name (none) -> RESISTOR-0805-10K; Tolerance (none) -> 5%
- R4: renamed from *R4; symbol tronixio:R-0805 -> tronixio:RESISTOR-0805-4K7; Mouser (none) -> 660-RK73B2ATTDD472J; Name (none) -> RESISTOR-0805-4K7; Tolerance (none) -> 5%
- R5: renamed from *R5; symbol tronixio:R-0805 -> tronixio:RESISTOR-0805-4K7; Mouser (none) -> 660-RK73B2ATTDD472J; Name (none) -> RESISTOR-0805-4K7; Tolerance (none) -> 5%
- R6: renamed from *R6; symbol tronixio:R-0805 -> tronixio:RESISTOR-0805-4K7; Mouser (none) -> 660-RK73B2ATTDD472J; Name (none) -> RESISTOR-0805-4K7; Tolerance (none) -> 5%
- R7: renamed from *R7; symbol tronixio:R-0805 -> tronixio:RESISTOR-0805-4K7; Mouser (none) -> 660-RK73B2ATTDD472J; Name (none) -> RESISTOR-0805-4K7; Tolerance (none) -> 5%
- R8: symbol tronixio:R-0805 -> tronixio:RESISTOR-0805-4K7; Mouser (none) -> 660-RK73B2ATTDD472J; Name (none) -> RESISTOR-0805-4K7; Tolerance (none) -> 5%
- S1: Name (none) -> ALPS-SKRPAC
- U1: symbol tronixio:SYMBOL-PIC8BIT-TQFP-44 -> tronixio:MICROCHIP-PIC16F1779-IPT; Mouser (none) -> 579-PIC16F1779-I/PT; Name (none) -> MICROCHIP-PIC16F1779-IPT
- U2: value MCP2221A -> MCP2221A-IST; Name MCP2221A-IST -> MICROCHIP-MCP2221A-IST
- U3: value ROHM-BU33SD5WG-500-SOT -> BU33SD5WG; Name BU33SD5WG -> ROHM-BU33SD5WG-500-SOT
Other:
- note added: "*"
- note added: "*R3/*R6/*R7/*LED2/*LED3/*U2: EUSART Optional components."
- note removed: "*R3/*R6/*R7/*LED2/*LED3/*IC2: EUSART Optional components."

Commit message: Update
Parts:
- K1, K2: Name SAMTEC-254-M-TSW-1X20-22-T-S -> SAMTEC-254-M-TSW-1X20-22-T-S_1
- U3: symbol tronixio:ROHM-BU33SD5WG-500-SOT -> tronixio:ROHM-BU33SD5WG-500-SOT-23; Name ROHM-BU33SD5WG-500-SOT -> ROHM-BU33SD5WG-500-SOT-23

Commit message: Update
Parts:
- F1: symbol tronixio:BOURNS-FUSE-MF-NSMF050 -> tronixio:BOURNS-FUSE-MF-PSMF050X; Mouser 652-MF-NSMF050-2 -> 652-MF-PSMF050X-2; Name BOURNS-FUSE-MF-NSMF050 -> BOURNS-FUSE-MF-PSMF050X
Changed lines of the file:
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@@
     (pin "1")
   )
-  (symbol (lib_id "tronixio:BOURNS-FUSE-MF-NSMF050") (at 93.98 139.7 0) (unit 1)
+  (symbol (lib_id "tronixio:BOURNS-FUSE-MF-PSMF050X") (at 93.98 139.7 0) (unit 1)
     (in_bom yes) (on_board yes)
     (property "Reference" "F1" (id 0) (at 93.98 135.255 0)
@@
       (effects (font (size 1 1)) hide)
     )
-    (property "Name" "BOURNS-FUSE-MF-NSMF050" (id 4) (at 93.98 144.78 0)
+    (property "Name" "BOURNS-FUSE-MF-PSMF050X" (id 4) (at 93.98 144.78 0)
       (effects (font (size 1 1)) hide)
     )
-    (property "Mouser" "652-MF-NSMF050-2" (id 5) (at 93.98 152.4 0)
+    (property "Mouser" "652-MF-PSMF050X-2" (id 5) (at 93.98 152.4 0)
       (effects (font (size 1 1)) hide)
     )

Commit message: Update
Parts:
- C1, C2, C3, C4, C5, C7, C8: footprint tronixio:CAPACITOR-0805 -> tronixio:CAPACITOR-SMD-0805
- F1: footprint tronixio:FUSE-0805 -> tronixio:FUSE-SMD-0805
- LED1, LED2, LED3: footprint tronixio:LED-0805 -> tronixio:LED-SMD-0805
- R1, R2, R3, R4, R5, R6, R7, R8: footprint tronixio:RESISTOR-0805 -> tronixio:RESISTOR-SMD-0805

Commit message: Update
Parts:
- U2: value MCP2221A-IST -> MCP2221A
Other:
- note added: "*U2/*R3/*R6/*R7/*LED2/*LED3: EUSART Optional components."
- note removed: "*R3/*R6/*R7/*LED2/*LED3/*U2: EUSART Optional components."
Changed lines of the file:
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@@
     (effects (font (size 1.27 1.27)) (justify right bottom))
   )
-  (text "*R3/*R6/*R7/*LED2/*LED3/*U2: EUSART Optional components."
+  (text "*U2/*R3/*R6/*R7/*LED2/*LED3: EUSART Optional components."
     (at 180.34 179.07 0)
     (effects (font (size 1.27 1.27)) (justify left bottom))
@@
       (effects (font (size 1.15 1.15)) (justify left))
     )
-    (property "Value" "MCP2221A-IST" (id 1) (at 121.92 156.21 0)
-      (effects (font (size 1.15 1.15)))
+    (property "Value" "MCP2221A" (id 1) (at 129.54 128.27 0)
+      (effects (font (size 1.15 1.15)) (justify right))
     )
     (property "Footprint" "tronixio:TSSOP-14" (id 2) (at 121.92 162.56 0)
@@
     )
     (path "/15b76320-9a6e-4ed9-be26-15ea028b6641"
-      (reference "U2") (unit 1) (value "MCP2221A-IST") (footprint "tronixio:TSSOP-14")
+      (reference "U2") (unit 1) (value "MCP2221A") (footprint "tronixio:TSSOP-14")
     )
     (path "/ef27345a-c7c1-44c7-b4de-dc92b9c6de34"
