File: Kicad/nano/pic8bit.kicad_sch (KiCad schematic)
At the start: 32 parts, among them K1 MCU 1, K2 MCU 2, K3 ICSP, K4 POWER & UART, U1 PIC16F/PIC18F, U2 MCP2221A, U3 BU33SD5WG

Commit message: Up
Parts:
- C1, C2, C3, C4: symbol tronixio:KEMET-X7R-0805-100N-50V-20P -> tronixio:CAPACITOR-0805-100N-20P-X7R
- C5: symbol tronixio:KEMET-X5R-0805-10U-6V3-20P -> tronixio:CAPACITOR-0805-10U-20P-X7R
- C7, C8: symbol tronixio:KEMET-X7R-0805-1U-16V-20P -> tronixio:CAPACITOR-0805-1U-20P-X7R
- R1, R3: symbol tronixio:KOASPEER-RK73B-0805-10K-5P -> tronixio:RESISTOR-0805-10K-5P
- R2: symbol tronixio:KOASPEER-RK73B-0805-1K-5P -> tronixio:RESISTOR-0805-1K-5P
- R4, R5, R6, R7, R8: symbol tronixio:KOASPEER-RK73B-0805-4K7-5P -> tronixio:RESISTOR-0805-4K7-5P
Connections:
- net +3V3: now also U3.5 (VOUT)
Other:
- moved on the sheet: C2, MEMS1

Commit message: Up
Parts:
- C1, C2, C3, C4: symbol tronixio:CAPACITOR-0805-100N-20P-X7R -> tronixio:CAPACITOR-0805-100N-10P-X7R; Mouser 80-C0805C104M5R -> 80-C0805C104K5RAC; Tolerance 20% -> 10%
- C5: symbol tronixio:CAPACITOR-0805-10U-20P-X7R -> tronixio:CAPACITOR-0805-10U-10P-X7R; Mouser 80-C0805C106M9P -> 187-CL21B106KAYQNNE; Tolerance 20% -> 10%; Voltage 6V3 -> 25V
- C7, C8: symbol tronixio:CAPACITOR-0805-1U-20P-X7R -> tronixio:CAPACITOR-0805-1U-10P-X7R; Mouser 80-C0805C105M4R -> 187-CL21B105KBFNNN; Tolerance 20% -> 10%; Voltage 16V -> 50V
- R1, R3: value 10K -> 10k
- R2: value 1K -> 1k
- R4, R5, R6, R7, R8: value 4K7 -> 4k7

Commit message: Up
Parts:
- C1, C2, C3, C4: symbol tronixio:CAPACITOR-0805-100N-10P-X7R -> tronixio:CAPACITOR-0805-100N-50V-5P-X7R; Mouser 80-C0805C104K5RAC -> 80-C0805C104J5; Tolerance 10% -> 5%
- C5: symbol tronixio:CAPACITOR-0805-10U-10P-X7R -> tronixio:CAPACITOR-0805-10U-25V-10P-X7R; Mouser 187-CL21B106KAYQNNE -> 81-GRM21BZ71E106KE5L
- C7, C8: symbol tronixio:CAPACITOR-0805-1U-10P-X7R -> tronixio:CAPACITOR-0805-1U-50V-10P-X7R; Mouser 187-CL21B105KBFNNN -> 187-CL21B105KBFNNNE
- JP1, JP2: symbol tronixio:HARWIN-200-M-1X02-JUMPER-TH-VERTICAL -> tronixio:HARWIN-200-M-1X02-JUMPER-VERTICAL
- K3: Mouser 855-M20-9980346 -> 855-M20-998034
- K4: footprint tronixio:FCI-USB-TYPE-B-MICRO-THT -> tronixio:USB-TYPE-B-MICRO-TH
Connections:
- net GND: now also K4.SH (SHIELD); no longer K4.6 (SHIELD)
- no-connect marks 4 -> 5

Commit message: Up
Parts:
- K4: symbol tronixio:FCI-USB-TYPE-B-MICRO-THT -> tronixio:FCI-USB-TYPE-B-MICRO-TH
Changed lines of the file:
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@@
     (effects (font (size 1 1)) (justify right bottom))
+  )
+  (label "{RA[0..7] RB[0..7] RC[0..7] RD[0..7] RE[0..2] RA4{slash}VCAP RA7{slash}CLKI RB6{slash}PGC RB7{slash}PGD ~{MCLR}}"
+    (at 60.96 33.02 0) (fields_autoplaced)
+    (effects (font (size 1.27 1.27)) (justify left bottom))
   )
   (label "~{MCLR}" (at 193.04 96.52 90) (fields_autoplaced)
@@
     )
   )
-  (symbol (lib_id "tronixio:FCI-USB-TYPE-B-MICRO-THT") (at 83.82 144.78 0) (unit 1)
+  (symbol (lib_id "tronixio:FCI-USB-TYPE-B-MICRO-TH") (at 83.82 144.78 0) (unit 1)
     (in_bom yes) (on_board yes) (dnp no)
     (property "Reference" "K4" (at 83.9105 132.08 0)
