File: Kicad/nano/pic8bit.kicad_sch (KiCad schematic)
At the start: 32 parts, among them K1 MCU 1, K2 MCU 2, K3 ICSP, K4 POWER & UART, U1 PIC16F/PIC18F, U2 MCP2221A, U3 BU33SD5WG

Commit message: Update Nano
Connections:
- net +3V3 renamed POWER-+3V3
- net +5V renamed POWER-+5V
- net GND renamed POWER-GND

Commit message: Update Nano
Connections:
- net POWER-+3V3 renamed +3V3
- net POWER-GND renamed GND
- no-connect marks 5 -> 4
Other:
- moved on the sheet: JP1, JP2

Commit message: Up
Parts:
- K1, K2: symbol tronixio:SAMTEC-254-M-TSW-1X20-22-T-S -> tronixio:SAMTEC-254-M-1X20-VERTICAL
Changed lines of the file:
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@@
 	)
 	(symbol
-		(lib_id "tronixio:SAMTEC-254-M-TSW-1X20-22-T-S")
+		(lib_id "tronixio:SAMTEC-254-M-1X20-VERTICAL")
 		(at 45.72 111.76 0)
 		(mirror y)
@@
 		)
 		(property "Description" "TSW/HTSW Series - 2.54mm Pitch PCB Connector"
-			(at 45.72 111.76 0)
-			(effects
-				(font
-					(size 1.27 1.27)
+			(at 45.72 172.72 0)
+			(do_not_autoplace yes)
+			(effects
+				(font
+					(size 1 1)
 				)
 				(hide yes)
@@
 	)
 	(symbol
-		(lib_id "tronixio:SAMTEC-254-M-TSW-1X20-22-T-S")
+		(lib_id "tronixio:SAMTEC-254-M-1X20-VERTICAL")
 		(at 45.72 43.18 0)
 		(mirror y)
@@
 		)
 		(property "Description" "TSW/HTSW Series - 2.54mm Pitch PCB Connector"
-			(at 45.72 43.18 0)
-			(effects
-				(font
-					(size 1.27 1.27)
-				)
-				(hide yes)
+			(at 45.72 104.14 0)
+			(do_not_autoplace yes)
+			(effects
+				(font
+					(size 1 1)
+				)
+				(hide yes)

Commit message: Up
Parts:
- H1, H2: footprint tronixio:HARWIN-M22-190-193 -> tronixio:HARWIN-M22-190-19X; now left out of the parts list
- MEMS1: value DSC1001C -> 24.5760MHz
Changed lines of the file:
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@@
 	(wire
 		(pts
-			(xy 226.06 66.04) (xy 236.22 66.04)
-		)
-		(stroke
-			(width 0)
-			(type solid)
-		)
-	)
-	(wire
-		(pts
 			(xy 254 60.96) (xy 254 63.5)
 		)
@@
 	(wire
 		(pts
+			(xy 226.06 66.04) (xy 233.68 66.04)
+		)
+		(stroke
+			(width 0)
+			(type default)
+		)
+	)
+	(wire
+		(pts
 			(xy 48.26 66.04) (xy 58.42 66.04)
 		)
@@
 	(text "*"
 		(exclude_from_sim no)
-		(at 238.76 61.595 0)
+		(at 236.855 61.595 0)
 		(effects
 			(font
@@
 	)
 	(label "RA7{slash}CLKI"
-		(at 227.33 66.04 0)
+		(at 226.06 66.04 0)
 		(fields_autoplaced yes)
 		(effects
@@
 		(property "Reference" "C1"
 			(at 245.745 45.72 0)
+			(do_not_autoplace yes)
 			(effects
 				(font
@@
 		(unit 1)
 		(exclude_from_sim no)
-		(in_bom yes)
+		(in_bom no)
 		(on_board yes)
 		(dnp no)
@@
 			)
 		)
-		(property "Footprint" "tronixio:HARWIN-M22-190-193"
+		(property "Footprint" "tronixio:HARWIN-M22-190-19X"
 			(at 269.24 182.88 0)
 			(do_not_autoplace yes)
@@
 		(dnp no)
 		(property "Reference" "MEMS1"
-			(at 238.76 60.96 0)
+			(at 240.03 60.96 0)
+			(do_not_autoplace yes)
 			(effects
 				(font
 					(size 1.15 1.15)
 				)
-				(justify right)
 			)
 		)
-		(property "Value" "DSC1001C"
-			(at 241.3 71.12 0)
+		(property "Value" "24.5760MHz"
+			(at 240.665 71.12 0)
+			(do_not_autoplace yes)
 			(effects
 				(font
@@
 			)
 		)
-		(property "Description" "Resistor"
+		(property "Description" ""
 			(at 104.14 121.92 0)
 			(effects
@@
 		(property "Reference" "K3"
 			(at 242.57 86.995 0)
+			(do_not_autoplace yes)
 			(effects
 				(font
@@
 		(property "Value" "ICSP"
 			(at 242.57 88.9 0)
+			(do_not_autoplace yes)
 			(effects
 				(font
@@
 		(property "Reference" "R1"
 			(at 254.635 29.21 0)
+			(do_not_autoplace yes)
 			(effects
 				(font
@@
 			)
 		)
-		(property "Description" "Resistor"
+		(property "Description" ""
 			(at 254 33.02 0)
 			(effects
@@
 		(property "Reference" "R2"
 			(at 236.22 35.56 90)
+			(do_not_autoplace yes)
 			(effects
 				(font
@@
 		(unit 1)
 		(exclude_from_sim no)
-		(in_bom yes)
+		(in_bom no)
 		(on_board yes)
 		(dnp no)
@@
 			)
 		)
-		(property "Footprint" "tronixio:HARWIN-M22-190-193"
+		(property "Footprint" "tronixio:HARWIN-M22-190-19X"
 			(at 274.32 182.88 0)
 			(do_not_autoplace yes)
@@
 		(property "Reference" "S1"
 			(at 255.27 39.37 90)
+			(do_not_autoplace yes)
 			(effects
 				(font
@@
 		(property "Value" "Reset"
 			(at 255.27 46.99 90)
+			(do_not_autoplace yes)
 			(effects
 				(font
@@
 		(property "Reference" "C2"
 			(at 255.27 66.04 0)
+			(do_not_autoplace yes)
 			(effects
 				(font
