File: Kicad/nano/pic8bit.kicad_pcb (KiCad board)
At the start: 2 copper layers, 21 x 52 mm, 34 parts, among them IC3 ROHM-BU33SD5WG-500-SOT, K1 MCU 1, K2 MCU 2, K3 ICSP, K4 POWER & UART

Commit message: Upadte
Parts:
- added kibuzzard-6288A768: G***, kibuzzard-6288A768, F.Cu at (116.4, 82.9)
- added kibuzzard-6288A773: G***, kibuzzard-6288A773, F.Cu at (116.1, 85.4)
- added kibuzzard-6288A7C8: G***, kibuzzard-6288A7C8, F.Cu at (104.6, 62.5)
- added kibuzzard-6288A7F5: G***, kibuzzard-6288A7F5, F.Cu at (104.9, 65.1)

Commit message: Up
Parts:
- removed *IC1: PIC16F/PIC18F, tronixio:TQFP-44
- removed *IC2: MCP2221A, tronixio:TSSOP-14
- removed IC3: ROHM-BU33SD5WG-500-SOT, tronixio:SOT-23-5
- added U1: PIC16F/PIC18F, tronixio:TQFP-44, F.Cu at (110.5, 75.2)
- added U2: MCP2221A, tronixio:TSSOP-14, B.Cu at (110.5, 59.5)
- added U3: ROHM-BU33SD5WG-500-SOT, tronixio:SOT-23-5, B.Cu at (110.5, 50.1)

Commit message: Update
Parts:
- F1: value F050 -> 500mA
- MEMS1: renamed from *MEMS1; value MICROCHIP-DSC1001C-245760-CDFN -> DSC1001C
- R1: value 10K -> 4K7
- U2: value MCP2221A -> MCP2221A-IST
- U3: value ROHM-BU33SD5WG-500-SOT -> BU33SD5WG
- renumbered *C2 to C2, *C5 to C5, *JP1 to JP1, *JP2 to JP2, *LED2 to LED2, *LED3 to LED3, *R3 to R3, *R4 to R4, *R5 to R5, *R6 to R6, *R7 to R7

Commit message: Update
Parts:
- C1, C2, C3, C4, C5, C7, C8: footprint tronixio:CAPACITOR-0805 -> tronixio:CAPACITOR-SMD-0805
- F1: footprint tronixio:FUSE-0805 -> tronixio:FUSE-SMD-0805
- LED1, LED2, LED3: footprint tronixio:LED-0805 -> tronixio:LED-SMD-0805
- R1, R2, R3, R4, R5, R6, R7, R8: footprint tronixio:RESISTOR-0805 -> tronixio:RESISTOR-SMD-0805

Commit message: Update Nano
Parts:
- R1: value 4K7 -> 10K
- U2: value MCP2221A-IST -> MCP2221A
