File: Kicad/nano/pic8bit.kicad_pcb (KiCad board)
At the start: 2 copper layers, 21 x 52 mm, 42 parts, among them K1 MCU 1, K2 MCU 2, K3 ICSP, K4 POWER & UART, U1 PIC16F/PIC18F, U2 MCP2221A, U3 BU33SD5WG

Commit message: Up
Parts:
- K4: footprint tronixio:FCI-USB-TYPE-B-MICRO-THT -> tronixio:USB-TYPE-B-MICRO-TH
- R1, R3: value 10K -> 10k
- R2: value 1K -> 1k
- R4, R5, R6, R7, R8: value 4K7 -> 4k7

Commit message: Up
Changed lines of the file:
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@@
     (fp_line (start 1 2.75) (end 1 1.25)
       (stroke (width 0.1) (type solid)) (layer "F.Fab"))
-    (pad "1" thru_hole circle (at 0 0 90) (size 1.4 1.4) (drill 0.8) (layers "*.Cu" "*.Mask")
+    (pad "1" thru_hole roundrect (at 0 0 90) (size 1.4 1.4) (drill 0.8) (layers "*.Cu" "*.Mask") (roundrect_rratio 0.25)
       (net 42 "Net-(U2-SDA)") (pintype "passive"))
-    (pad "2" thru_hole circle (at 0 2 90) (size 1.4 1.4) (drill 0.8) (layers "*.Cu" "*.Mask")
+    (pad "2" thru_hole roundrect (at 0 2 90) (size 1.4 1.4) (drill 0.8) (layers "*.Cu" "*.Mask") (roundrect_rratio 0.25)
       (net 15 "RC4{slash}SDA") (pintype "passive"))
     (model "${KICAD_USER_3DMODEL_DIR}/Misc/HARWIN-M22-25102xx.step"
@@
     (fp_line (start 3.81 6.0325) (end 3.81 4.1275)
       (stroke (width 0.1) (type solid)) (layer "F.Fab"))
-    (pad "1" thru_hole circle (at 0 0 90) (size 1.8 1.8) (drill 0.8) (layers "*.Cu" "*.Mask")
+    (pad "1" thru_hole roundrect (at 0 0 90) (size 1.6 1.6) (drill 0.8) (layers "*.Cu" "*.Mask") (roundrect_rratio 0.1)
       (net 20 "/~{MCLR}") (pinfunction "1") (pintype "passive"))
-    (pad "2" thru_hole circle (at 2.54 0 90) (size 1.8 1.8) (drill 0.8) (layers "*.Cu" "*.Mask")
+    (pad "2" thru_hole roundrect (at 2.54 0 90) (size 1.6 1.6) (drill 0.8) (layers "*.Cu" "*.Mask") (roundrect_rratio 0.1)
       (net 1 "+3V3") (pinfunction "2") (pintype "passive"))
-    (pad "3" thru_hole circle (at 0 2.54 90) (size 1.8 1.8) (drill 0.8) (layers "*.Cu" "*.Mask")
+    (pad "3" thru_hole roundrect (at 0 2.54 90) (size 1.6 1.6) (drill 0.8) (layers "*.Cu" "*.Mask") (roundrect_rratio 0.1)
       (net 2 "GND") (pinfunction "3") (pintype "passive"))
-    (pad "4" thru_hole circle (at 2.54 2.54 90) (size 1.8 1.8) (drill 0.8) (layers "*.Cu" "*.Mask")
+    (pad "4" thru_hole roundrect (at 2.54 2.54 90) (size 1.6 1.6) (drill 0.8) (layers "*.Cu" "*.Mask") (roundrect_rratio 0.1)
       (net 19 "/RB7{slash}PGD") (pinfunction "4") (pintype "passive"))
-    (pad "5" thru_hole circle (at 0 5.08 90) (size 1.8 1.8) (drill 0.8) (layers "*.Cu" "*.Mask")
+    (pad "5" thru_hole roundrect (at 0 5.08 90) (size 1.6 1.6) (drill 0.8) (layers "*.Cu" "*.Mask") (roundrect_rratio 0.1)
       (net 18 "/RB6{slash}PGC") (pinfunction "5") (pintype "passive"))
-    (pad "6" thru_hole circle (at 2.54 5.08 90) (size 1.8 1.8) (drill 0.8) (layers "*.Cu" "*.Mask")
+    (pad "6" thru_hole roundrect (at 2.54 5.08 90) (size 1.6 1.6) (drill 0.8) (layers "*.Cu" "*.Mask") (roundrect_rratio 0.1)
       (net 43 "unconnected-(K3-Pad6)") (pinfunction "6") (pintype "passive+no_connect"))
     (model "${KICAD_USER_3DMODEL_DIR}/Header/HARWIN-M20-998034x.wrl"
@@
     (fp_line (start 1 2.75) (end 1 1.25)
       (stroke (width 0.1) (type solid)) (layer "F.Fab"))
-    (pad "1" thru_hole circle (at 0 0 90) (size 1.4 1.4) (drill 0.8) (layers "*.Cu" "*.Mask")
+    (pad "1" thru_hole roundrect (at 0 0 90) (size 1.4 1.4) (drill 0.8) (layers "*.Cu" "*.Mask") (roundrect_rratio 0.25)
       (net 41 "Net-(U2-SCL)") (pintype "passive"))
-    (pad "2" thru_hole circle (at 0 2 90) (size 1.4 1.4) (drill 0.8) (layers "*.Cu" "*.Mask")
+    (pad "2" thru_hole roundrect (at 0 2 90) (size 1.4 1.4) (drill 0.8) (layers "*.Cu" "*.Mask") (roundrect_rratio 0.25)
       (net 34 "RC3{slash}SCL") (pintype "passive"))
     (model "${KICAD_USER_3DMODEL_DIR}/Misc/HARWIN-M22-25102xx.step"
@@
   (gr_circle (center 150.5 76.75) (end 150.7 76.75)
     (stroke (width 0.1) (type solid)) (fill solid) (layer "B.SilkS"))
-  (gr_circle (center 149.1 52) (end 149.35 52)
-    (stroke (width 0.1) (type solid)) (fill solid) (layer "B.SilkS"))
   (gr_circle (center 153.5 56.75) (end 153.75 56.75)
     (stroke (width 0.1) (type solid)) (fill solid) (layer "B.SilkS"))
@@
     )
     (stroke (width 0.1) (type solid)) (fill solid) (layer "B.SilkS"))
+  (gr_circle (center 151.5 67.5) (end 151.25 67.5)
+    (stroke (width 0.1) (type solid)) (fill solid) (layer "F.SilkS"))
   (gr_poly
     (pts
@@
   (segment (start 153.75 77.353629) (end 153.75 75.4) (width 0.4) (layer "F.Cu") (net 2))
   (segment (start 147.2 50.1) (end 148.35 50.1) (width 0.4) (layer "F.Cu") (net 2))
-  (segment (start 153.75 97.25) (end 154.75 96.25) (width 0.3) (layer "F.Cu") (net 2))
+  (segment (start 151.75 97.25) (end 154.25 97.25) (width 0.3) (layer "F.Cu") (net 2))
   (segment (start 159.251371 82.855) (end 155.096194 78.699823) (width 0.3) (layer "F.Cu") (net 2))
   (segment (start 141.61 62.535) (end 144.5 65.425) (width 0.3) (layer "F.Cu") (net 2))
@@
   (segment (start 148.35 50.1) (end 149.2 50.95) (width 0.4) (layer "F.Cu") (net 2))
   (segment (start 155.096194 78.699823) (end 153.75 77.353629) (width 0.4) (layer "F.Cu") (net 2))
+  (segment (start 154.75 96.75) (end 154.75 96.25) (width 0.3) (layer "F.Cu") (net 2))
   (segment (start 144.5 65.425) (end 144.5 69.235) (width 0.3) (layer "F.Cu") (net 2))
-  (segment (start 151.75 97.25) (end 153.75 97.25) (width 0.3) (layer "F.Cu") (net 2))
+  (segment (start 154.25 97.25) (end 154.75 96.75) (width 0.3) (layer "F.Cu") (net 2))
   (segment (start 147.5 72.25) (end 148 72.25) (width 0.4) (layer "F.Cu") (net 2))
   (segment (start 144.5 69.235) (end 146.469491 71.204491) (width 0.3) (layer "F.Cu") (net 2))
-  (segment (start 150.5 98.5) (end 151.75 97.25) (width 0.3) (layer "F.Cu") (net 2))
   (segment (start 146.469491 71.219491) (end 147.5 72.25) (width 0.4) (layer "F.Cu") (net 2))
   (segment (start 149.2 50.95) (end 149.2 52.9) (width 0.4) (layer "F.Cu") (net 2))
+  (segment (start 150.5 98.5) (end 151.75 97.25) (width 0.3) (layer "F.Cu") (net 2))
   (segment (start 148.4 89.65) (end 150.5 89.65) (width 0.4) (layer "F.Cu") (net 2))
   (segment (start 153.8 50.1) (end 153.8 52.4) (width 0.5) (layer "F.Cu") (net 2))
@@
   (segment (start 157.106613 72.0225) (end 157.5225 72.0225) (width 0.3) (layer "F.Cu") (net 33))
   (segment (start 155.664138 72.335862) (end 158 70) (width 0.3) (layer "F.Cu") (net 34))
-  (segment (start 150.5 69.5) (end 154.25 73.25) (width 0.3) (layer "F.Cu") (net 34))
-  (segment (start 150.5 64.75) (end 150.5 64.25) (width 0.3) (layer "F.Cu") (net 34))
-  (segment (start 158 70) (end 158 69.005) (width 0.3) (layer "F.Cu") (net 34))
-  (segment (start 150.5 65.75) (end 150.5 69.5) (width 0.3) (layer "F.Cu") (net 34))
   (segment (start 154.75 73.25) (end 155.66188 72.33812) (width 0.3) (layer "F.Cu") (net 34))
+  (segment (start 158 70) (end 158 69.005) (width 0.3) (layer "F.Cu") (net 34))
+  (segment (start 150.5 66) (end 150.5 69.5) (width 0.3) (layer "F.Cu") (net 34))
   (segment (start 158 69.005) (end 159.39 67.615) (width 0.3) (layer "F.Cu") (net 34))
-  (segment (start 150.5 65.75) (end 150.5 64.75) (width 0.2) (layer "F.Cu") (net 34))
+  (segment (start 150.5 64.5) (end 150.5 64.25) (width 0.3) (layer "F.Cu") (net 34))
+  (segment (start 150.5 66) (end 150.5 64.5) (width 0.2) (layer "F.Cu") (net 34))
+  (segment (start 150.5 69.5) (end 154.25 73.25) (width 0.3) (layer "F.Cu") (net 34))
   (segment (start 150.5 64.25) (end 151.5 63.25) (width 0.3) (layer "F.Cu") (net 34))
   (segment (start 154.25 73.25) (end 154.75 73.25) (width 0.3) (layer "F.Cu") (net 34))
@@
   (segment (start 149.5 63.25) (end 149.5 60.75) (width 0.3) (layer "F.Cu") (net 41))
   (via (at 149.25 60.5) (size 0.8) (drill 0.4) (layers "F.Cu" "B.Cu") (net 41))
-  (segment (start 150.5 67) (end 150.5 65.75) (width 0.3) (layer "B.Cu") (net 41))
-  (segment (start 151.75 67.5) (end 151 67.5) (width 0.3) (layer "B.Cu") (net 41))
-  (segment (start 151 67.5) (end 150.5 67) (width 0.3) (layer "B.Cu") (net 41))
   (segment (start 148.9 60.15) (end 149.25 60.5) (width 0.3) (layer "B.Cu") (net 41))
-  (segment (start 150.5 64.25) (end 150.5 64.75) (width 0.3) (layer "B.Cu") (net 41))
+  (segment (start 150.5 66) (end 150.5 64.5) (width 0.2) (layer "B.Cu") (net 41))
+  (segment (start 150.5 67) (end 151 67.5) (width 0.3) (layer "B.Cu") (net 41))
+  (segment (start 150.5 64.5) (end 150.5 64.25) (width 0.3) (layer "B.Cu") (net 41))
   (segment (start 150.5 64.25) (end 149.5 63.25) (width 0.3) (layer "B.Cu") (net 41))
-  (segment (start 150.5 65.75) (end 150.5 64.75) (width 0.2) (layer "B.Cu") (net 41))
+  (segment (start 151 67.5) (end 151.75 67.5) (width 0.3) (layer "B.Cu") (net 41))
   (segment (start 147.5 60.15) (end 148.9 60.15) (width 0.3) (layer "B.Cu") (net 41))
+  (segment (start 150.5 66) (end 150.5 67) (width 0.3) (layer "B.Cu") (net 41))
   (segment (start 149.25 66.5) (end 149.5 66.25) (width 0.3) (layer "B.Cu") (net 42))
   (segment (start 146.25 63.5) (end 146.25 61.25) (width 0.3) (layer "B.Cu") (net 42))
